Commit message: Repaired .stl files loading, working gazebo model loading fixed trunk in the air

File: description/RobotElements/LeftLegElems/Lankle.xacro (robot description, xacro)
@@ -12,5 +12,5 @@
         <origin xyz="0 0 0" rpy="0 0 0"/>
         <geometry>
-          <mesh filename="package://ros2_humanoid_virtual_twin/STLe/Left-Ankle.stl"/>
+          <mesh filename="file://$(find ros2_humanoid_virtual_twin)/STLe/Left-Ankle.stl"/>
         </geometry>
         <material name="grey"/>
@@ -19,5 +19,5 @@
         <origin xyz="0 0 0" rpy="0 0 0"/>
         <geometry>
-            <mesh filename="package://ros2_humanoid_virtual_twin/STLe/Left-Ankle-Collision.stl"/>
+            <mesh filename="file://$(find ros2_humanoid_virtual_twin)/STLe/Left-Ankle-Collision.stl"/>
         </geometry>
       </collision>

File: description/RobotElements/LeftLegElems/Lfoot.xacro (robot description, xacro)
@@ -12,5 +12,5 @@
         <origin xyz="0 0 0" rpy="0 0 0"/>
         <geometry>
-          <mesh filename="package://ros2_humanoid_virtual_twin/STLe/Left-Foot.stl"/>
+          <mesh filename="file://$(find ros2_humanoid_virtual_twin)/STLe/Left-Foot.stl"/>
         </geometry>
         <material name="grey"/>
@@ -19,5 +19,5 @@
         <origin xyz="0 0 0" rpy="0 0 0"/>
         <geometry>
-			<mesh filename="package://ros2_humanoid_virtual_twin/STLe/Left-Foot-collision.stl"/>
+			<mesh filename="file://$(find ros2_humanoid_virtual_twin)/STLe/Left-Foot-collision.stl"/>
         </geometry>
       </collision>

File: description/RobotElements/LeftLegElems/Lhip.xacro (robot description, xacro)
@@ -13,5 +13,5 @@
         <origin xyz="0 0 0" rpy="0 0 0"/>
         <geometry>
-          <mesh filename="package://ros2_humanoid_virtual_twin/STLe/Left-Hip.stl"/>
+          <mesh filename="file://$(find ros2_humanoid_virtual_twin)/STLe/Left-Hip.stl"/>
         </geometry>
         <material name="grey"/>
@@ -20,5 +20,5 @@
         <origin xyz="0 0 0" rpy="0 0 0"/>
         <geometry>
-            <mesh filename="package://ros2_humanoid_virtual_twin/STLe/Right-Hip-Collision.stl"/>
+            <mesh filename="file://$(find ros2_humanoid_virtual_twin)/STLe/Right-Hip-Collision.stl"/>
         </geometry>
       </collision>

File: description/RobotElements/LeftLegElems/Lhipmount.xacro (robot description, xacro)
@@ -14,5 +14,5 @@
       <origin xyz="0 0 0" rpy="0 0 0"/>
       <geometry>
-        <mesh filename="package://ros2_humanoid_virtual_twin/STLe/Left-HipMount.stl"/>
+        <mesh filename="file://$(find ros2_humanoid_virtual_twin)/STLe/Left-HipMount.stl"/>
       </geometry>
       <material name="grey"/>
@@ -21,5 +21,5 @@
       <origin xyz="0 0 0" rpy="0 0 0"/>
       <geometry>
-        <mesh filename="package://ros2_humanoid_virtual_twin/STLe/Rgiht-HipMount-Collision.stl"/>
+        <mesh filename="file://$(find ros2_humanoid_virtual_twin)/STLe/Rgiht-HipMount-Collision.stl"/>
       </geometry>
     </collision>

File: description/RobotElements/LeftLegElems/Lshank.xacro (robot description, xacro)
@@ -12,5 +12,5 @@
         <origin xyz="0 0 0" rpy="0 0 0"/>
         <geometry>
-          <mesh filename="package://ros2_humanoid_virtual_twin/STLe/Left-Shank.stl"/>
+          <mesh filename="file://$(find ros2_humanoid_virtual_twin)/STLe/Left-Shank.stl"/>
         </geometry>
         <material name="grey"/>
@@ -19,5 +19,5 @@
         <origin xyz="0 0 0" rpy="0 0 0"/>
         <geometry>
-            <mesh filename="package://ros2_humanoid_virtual_twin/STLe/Right-Shank-Collision.stl"/>
+            <mesh filename="file://$(find ros2_humanoid_virtual_twin)/STLe/Right-Shank-Collision.stl"/>
         </geometry>
       </collision>

File: description/RobotElements/LeftLegElems/Lthigh.xacro (robot description, xacro)
@@ -12,5 +12,5 @@
         <origin xyz="0 0 0" rpy="0 0 0"/>
         <geometry>
-          <mesh filename="package://ros2_humanoid_virtual_twin/STLe/Left-Thigh.stl"/>
+          <mesh filename="file://$(find ros2_humanoid_virtual_twin)/STLe/Left-Thigh.stl"/>
         </geometry>
         <material name="grey"/>
@@ -19,5 +19,5 @@
         <origin xyz="0 0 0" rpy="0 0 0"/>
         <geometry>
-            <mesh filename="package://ros2_humanoid_virtual_twin/STLe/Right-Thigh-Collision.stl"/>
+            <mesh filename="file://$(find ros2_humanoid_virtual_twin)/STLe/Right-Thigh-Collision.stl"/>
         </geometry>
       </collision>

File: description/RobotElements/Trunk.xacro (robot description, xacro)
@@ -13,5 +13,5 @@
       <origin xyz="0 0 0" rpy="0 0 0"/>
       <geometry>
-        <mesh filename="package://ros2_humanoid_virtual_twin/STLe/Trunk.stl"/>
+        <mesh filename="file://$(find ros2_humanoid_virtual_twin)/STLe/Trunk.stl"/>
       </geometry>
       <material name="grey"/>
@@ -25,10 +25,10 @@
       <origin xyz="0 0 0" rpy="0 0 0"/>
       <geometry>
-        <mesh filename="package://ros2_humanoid_virtual_twin/STLe/Trunk-Collision.stl"/>
+        <mesh filename="file://$(find ros2_humanoid_virtual_twin)/STLe/Trunk-Collision.stl"/>
       </geometry>
     </collision>
   </link>
   <gazebo reference="Trunk">
-      <material>Gazebo/Black</material>
+      <material>Gazebo/Grey</material>
   </gazebo>
 </robot>

File: description/robot.urdf.xacro (robot description, xacro)
@@ -3,4 +3,10 @@
     <!-- Below is a file which initiates geometry of robot and inertial, dynamic, collision parameters -->
     <xacro:include filename="robot_core.xacro" />
+    <!-- If you want the Trunk to be immovable and static at a certain height uncomment lines below -->
+    <link name="world"/>
+    <joint name="world-base_link-fixed" type="fixed">
+        <parent link="world"/>
+        <child link="base_link"/>
+    </joint>
     <!-- Below is a file which contains parameters controlling movements of a robot -->
 </robot>

Commit message: Changed name of the file containing .stl files, and repaired color visualisation

File: description/RobotElements/LeftLegElems/Lankle.xacro (robot description, xacro)
@@ -12,5 +12,5 @@
         <origin xyz="0 0 0" rpy="0 0 0"/>
         <geometry>
-          <mesh filename="file://$(find ros2_humanoid_virtual_twin)/STLe/Left-Ankle.stl"/>
+          <mesh filename="file://$(find ros2_humanoid_virtual_twin)/meshes/Left-Ankle.stl"/>
         </geometry>
         <material name="grey"/>
@@ -19,5 +19,5 @@
         <origin xyz="0 0 0" rpy="0 0 0"/>
         <geometry>
-            <mesh filename="file://$(find ros2_humanoid_virtual_twin)/STLe/Left-Ankle-Collision.stl"/>
+            <mesh filename="file://$(find ros2_humanoid_virtual_twin)/meshes/Left-Ankle-Collision.stl"/>
         </geometry>
       </collision>
@@ -28,3 +28,6 @@
       </inertial>
     </link>
+    <gazebo reference="Left_Ankle">
+      <material>Gazebo/Grey</material>
+    </gazebo>
 </robot>

File: description/RobotElements/LeftLegElems/Lfoot.xacro (robot description, xacro)
@@ -12,5 +12,5 @@
         <origin xyz="0 0 0" rpy="0 0 0"/>
         <geometry>
-          <mesh filename="file://$(find ros2_humanoid_virtual_twin)/STLe/Left-Foot.stl"/>
+          <mesh filename="file://$(find ros2_humanoid_virtual_twin)/meshes/Left-Foot.stl"/>
         </geometry>
         <material name="grey"/>
@@ -19,5 +19,5 @@
         <origin xyz="0 0 0" rpy="0 0 0"/>
         <geometry>
-			<mesh filename="file://$(find ros2_humanoid_virtual_twin)/STLe/Left-Foot-collision.stl"/>
+			<mesh filename="file://$(find ros2_humanoid_virtual_twin)/meshes/Left-Foot-collision.stl"/>
         </geometry>
       </collision>
@@ -28,3 +28,6 @@
       </inertial>
     </link>
+    <gazebo reference="Left_Foot">
+      <material>Gazebo/Grey</material>
+    </gazebo>
 </robot>

File: description/RobotElements/LeftLegElems/Lhip.xacro (robot description, xacro)
@@ -13,5 +13,5 @@
         <origin xyz="0 0 0" rpy="0 0 0"/>
         <geometry>
-          <mesh filename="file://$(find ros2_humanoid_virtual_twin)/STLe/Left-Hip.stl"/>
+          <mesh filename="file://$(find ros2_humanoid_virtual_twin)/meshes/Left-Hip.stl"/>
         </geometry>
         <material name="grey"/>
@@ -20,5 +20,5 @@
         <origin xyz="0 0 0" rpy="0 0 0"/>
         <geometry>
-            <mesh filename="file://$(find ros2_humanoid_virtual_twin)/STLe/Right-Hip-Collision.stl"/>
+            <mesh filename="file://$(find ros2_humanoid_virtual_twin)/meshes/Right-Hip-Collision.stl"/>
         </geometry>
       </collision>
@@ -29,3 +29,6 @@
       </inertial>
     </link>
+    <gazebo reference="Left_Hip">
+      <material>Gazebo/Grey</material>
+    </gazebo>
 </robot>

File: description/RobotElements/LeftLegElems/Lhipmount.xacro (robot description, xacro)
@@ -14,5 +14,5 @@
       <origin xyz="0 0 0" rpy="0 0 0"/>
       <geometry>
-        <mesh filename="file://$(find ros2_humanoid_virtual_twin)/STLe/Left-HipMount.stl"/>
+        <mesh filename="file://$(find ros2_humanoid_virtual_twin)/meshes/Left-HipMount.stl"/>
       </geometry>
       <material name="grey"/>
@@ -21,5 +21,5 @@
       <origin xyz="0 0 0" rpy="0 0 0"/>
       <geometry>
-        <mesh filename="file://$(find ros2_humanoid_virtual_twin)/STLe/Rgiht-HipMount-Collision.stl"/>
+        <mesh filename="file://$(find ros2_humanoid_virtual_twin)/meshes/Rgiht-HipMount-Collision.stl"/>
       </geometry>
     </collision>
@@ -31,5 +31,5 @@
   </link>
   <gazebo reference="Left_HipMount">
-      <material>Gazebo/Black</material>
+      <material>Gazebo/Grey</material>
   </gazebo>
 </robot>

File: description/RobotElements/LeftLegElems/Lshank.xacro (robot description, xacro)
@@ -12,5 +12,5 @@
         <origin xyz="0 0 0" rpy="0 0 0"/>
         <geometry>
-          <mesh filename="file://$(find ros2_humanoid_virtual_twin)/STLe/Left-Shank.stl"/>
+          <mesh filename="file://$(find ros2_humanoid_virtual_twin)/meshes/Left-Shank.stl"/>
         </geometry>
         <material name="grey"/>
@@ -19,5 +19,5 @@
         <origin xyz="0 0 0" rpy="0 0 0"/>
         <geometry>
-            <mesh filename="file://$(find ros2_humanoid_virtual_twin)/STLe/Right-Shank-Collision.stl"/>
+            <mesh filename="file://$(find ros2_humanoid_virtual_twin)/meshes/Right-Shank-Collision.stl"/>
         </geometry>
       </collision>
@@ -28,3 +28,6 @@
       </inertial>
     </link>
+    <gazebo reference="Left_Shank">
+      <material>Gazebo/Grey</material>
+    </gazebo>
 </robot>

File: description/RobotElements/LeftLegElems/Lthigh.xacro (robot description, xacro)
@@ -12,5 +12,5 @@
         <origin xyz="0 0 0" rpy="0 0 0"/>
         <geometry>
-          <mesh filename="file://$(find ros2_humanoid_virtual_twin)/STLe/Left-Thigh.stl"/>
+          <mesh filename="file://$(find ros2_humanoid_virtual_twin)/meshes/Left-Thigh.stl"/>
         </geometry>
         <material name="grey"/>
@@ -19,5 +19,5 @@
         <origin xyz="0 0 0" rpy="0 0 0"/>
         <geometry>
-            <mesh filename="file://$(find ros2_humanoid_virtual_twin)/STLe/Right-Thigh-Collision.stl"/>
+            <mesh filename="file://$(find ros2_humanoid_virtual_twin)/meshes/Right-Thigh-Collision.stl"/>
         </geometry>
       </collision>
@@ -28,3 +28,6 @@
       </inertial>
     </link>
+    <gazebo reference="Left_Thigh">
+      <material>Gazebo/Grey</material>
+    </gazebo>
 </robot>

File: description/RobotElements/Trunk.xacro (robot description, xacro)
@@ -13,5 +13,5 @@
       <origin xyz="0 0 0" rpy="0 0 0"/>
       <geometry>
-        <mesh filename="file://$(find ros2_humanoid_virtual_twin)/STLe/Trunk.stl"/>
+        <mesh filename="file://$(find ros2_humanoid_virtual_twin)/meshes/Trunk.stl"/>
       </geometry>
       <material name="grey"/>
@@ -25,5 +25,5 @@
       <origin xyz="0 0 0" rpy="0 0 0"/>
       <geometry>
-        <mesh filename="file://$(find ros2_humanoid_virtual_twin)/STLe/Trunk-Collision.stl"/>
+        <mesh filename="file://$(find ros2_humanoid_virtual_twin)/meshes/Trunk-Collision.stl"/>
       </geometry>
     </collision>
