Commit message: Added right leg, gazebo visually correct and rviz2 too

File: description/RobotElements/LeftLegElems/Lfoot.xacro (robot description, xacro)
@@ -12,5 +12,6 @@
         <origin xyz="0 0 0" rpy="0 0 0"/>
         <geometry>
-          <mesh filename="file://$(find ros2_humanoid_virtual_twin)/meshes/Left-Foot.stl"/>
+          <!-- Right foot .stl is used to describe right foot because visually its better :)-->
+          <mesh filename="file://$(find ros2_humanoid_virtual_twin)/meshes/Right-Foot.stl"/>
         </geometry>
         <material name="grey"/>

File: description/RobotElements/Trunk.xacro (robot description, xacro)
@@ -10,5 +10,5 @@
   <link name="Trunk">
     <visual>
-		  <!--Origin defines geometric center of spawnego object relative to child frame-->
+		  <!--Origin defines geometric center of spawned object relative to child frame-->
       <origin xyz="0 0 0" rpy="0 0 0"/>
       <geometry>

File: description/robot_core.xacro (robot description, xacro)
@@ -10,3 +10,4 @@
   <xacro:include filename="RobotElements/Trunk.xacro"/>
   <xacro:include filename="RobotElements/left_leg.xacro"/>
+  <xacro:include filename="RobotElements/right_leg.xacro"/>
 </robot>
