Commit message: Added Right leg and head visual loading to rviz2 and gazebo

File: description/RobotElements/HeadElems/Headmount.xacro (robot description, xacro)
@@ -1,16 +1,16 @@
 <?xml version="1.0"?>
 <robot xmlns:xacro="http://www.ros.org/wiki/xacro">
-    <joint name="RTz" type="revolute">
-        <origin xyz="0 -40e-03 -150.065e-03" rpy="0 0 0"/>
+    <joint name="Hz" type="revolute">
+        <origin xyz="18.061e-3 0.134e-3 42.5e-3" rpy="0 0 0"/>
         <parent link="Trunk"/>
-        <child link="Right_HipMount"/>
+        <child link="Head_Mounting"/>
         <axis xyz="0 0 1.0"/>
         <limit lower="${-pi/2}" upper="${pi/2}" effort="100" velocity="100"/>
     </joint>
-    <link name="Right_HipMount">
+    <link name="Head_Mounting">
         <visual>
             <origin xyz="0 0 0" rpy="0 0 0"/>
             <geometry>
-                <mesh filename="file://$(find ros2_humanoid_virtual_twin)/meshes/Right-HipMount.stl"/>
+                <mesh filename="file://$(find ros2_humanoid_virtual_twin)/meshes/HeadMounting.stl"/>
             </geometry>
             <material name="grey"/>
@@ -19,14 +19,14 @@
             <origin xyz="0 0 0" rpy="0 0 0"/>
             <geometry>
-                <mesh filename="file://$(find ros2_humanoid_virtual_twin)/meshes/Right-HipMount-Collision.stl"/>
+                <mesh filename="file://$(find ros2_humanoid_virtual_twin)/meshes/Head-Mounting-Collision.stl"/>
             </geometry>
         </collision>
         <inertial>
-            <origin xyz="-14.306e-03 0 24.769e-03" rpy="0 0 0"/>
-            <mass value="0.038"/>
-            <inertia ixx="11.743e-6" iyy="61.298e-6" izz="58.734e-6" ixy="0" ixz="4.429e-6" iyz="0"/>
+            <origin xyz="0 -3.335e-3 -17.703e-3" rpy="0 0 0"/>
+            <mass value="0.011"/>
+            <inertia ixx="4.859e-6" iyy="2.246e-6" izz="3.894e-6" ixy="0" ixz="0"  iyz="0.637e-3"/>
         </inertial>
     </link>
-    <gazebo reference="Right_HipMount">
+    <gazebo reference="Head_Mounting">
         <material>Gazebo/Grey</material>
     </gazebo>

File: description/RobotElements/LeftLegElems/Lankle.xacro (robot description, xacro)
@@ -6,5 +6,5 @@
       <child link="Left_Ankle"/>
       <axis xyz="0 1.0 0"/>
-      <limit lower="${-pi}" upper="${pi}" effort="100" velocity="100"/>
+      <limit lower="${-pi/2}" upper="${pi/2}" effort="100" velocity="100"/>
     </joint>
 	<link name="Left_Ankle">

File: description/RobotElements/LeftLegElems/Lfoot.xacro (robot description, xacro)
@@ -6,5 +6,5 @@
       <child link="Left_Foot"/>
       <axis xyz="1.0 0 0"/>
-      <limit lower="${-pi}" upper="${pi}" effort="100" velocity="100"/>
+      <limit lower="${-pi/2}" upper="${pi/2}" effort="100" velocity="100"/>
     </joint>
     <link name="Left_Foot">

File: description/RobotElements/LeftLegElems/Lhip.xacro (robot description, xacro)
@@ -7,5 +7,5 @@
       <child link="Left_Hip"/>
       <axis xyz="1.0 0 0"/>
-      <limit lower="${-pi}" upper="${pi}" effort="100" velocity="100"/>
+      <limit lower="${-pi/2}" upper="${pi/2}" effort="100" velocity="100"/>
     </joint>
     <link name="Left_Hip">

File: description/RobotElements/LeftLegElems/Lhipmount.xacro (robot description, xacro)
@@ -8,5 +8,5 @@
     <child link="Left_HipMount"/>
     <axis xyz="0 0 1.0"/>
-    <limit lower="${-pi}" upper="${pi}" effort="100" velocity="100"/>
+    <limit lower="${-pi/2}" upper="${pi/2}" effort="100" velocity="100"/>
   </joint>
   <link name="Left_HipMount">

File: description/RobotElements/LeftLegElems/Lshank.xacro (robot description, xacro)
@@ -6,5 +6,5 @@
       <child link="Left_Shank"/>
       <axis xyz="0 1.0 0"/>
-      <limit lower="${-pi}" upper="${pi}" effort="100" velocity="100"/>
+      <limit lower="${-pi/2}" upper="${pi/2}" effort="100" velocity="100"/>
     </joint>
 	<link name="Left_Shank">

File: description/RobotElements/LeftLegElems/Lthigh.xacro (robot description, xacro)
@@ -6,5 +6,5 @@
       <child link="Left_Thigh"/>
       <axis xyz="0 1.0 0"/>
-      <limit lower="${-pi}" upper="${pi}" effort="100" velocity="100"/>
+      <limit lower="${-pi/2}" upper="${pi/2}" effort="100" velocity="100"/>
     </joint>
     <link name="Left_Thigh">

File: description/RobotElements/RightArmElems/Rarm.xacro (robot description, xacro)
@@ -1,12 +1,12 @@
 <?xml version="1.0"?>
 <robot xmlns:xacro="http://www.ros.org/wiki/xacro" >
-    <joint name="LAx" type="revolute">
+    <joint name="RAx" type="revolute">
         <origin xyz="0 0 0" rpy="0 0 0"/>
-        <parent link="Left_ArmMounting"/>
-        <child link="Left_Arm"/>
+        <parent link="Right_ArmMounting"/>
+        <child link="Right_Arm"/>
         <axis xyz="1.0 0 0"/>
         <limit lower="${-pi/2}" upper="${pi/2}" effort="100" velocity="100"/>
     </joint>
-    <link name="Left_Arm">
+    <link name="Right_Arm">
         <visual>
             <origin xyz="0 0 0" rpy="0 0 0"/>
@@ -28,5 +28,5 @@
         </inertial>
     </link>
-    <gazebo reference="Left_Arm">
+    <gazebo reference="Right_Arm">
         <material>Gazebo/Grey</material>
     </gazebo>

File: description/RobotElements/RightArmElems/Rarmmount.xacro (robot description, xacro)
@@ -1,16 +1,16 @@
 <?xml version="1.0"?>
 <robot xmlns:xacro="http://www.ros.org/wiki/xacro" >
-    <joint name="LAy" type="revolute">
-        <origin xyz="0 88.341e-3 0" rpy="0 0 0"/>
+    <joint name="RAy" type="revolute">
+        <origin xyz="0 -88.659e-3 0" rpy="0 0 0"/>
         <parent link="Trunk"/>
-        <child link="Left_ArmMounting"/>
+        <child link="Right_ArmMounting"/>
         <axis xyz="0 1.0 0"/>
         <limit lower="${-pi/2}" upper="${pi/2}" effort="100" velocity="100"/>
     </joint>
-    <link name="Left_ArmMounting">
+    <link name="Right_ArmMounting">
         <visual>
             <origin xyz="0 0 0" rpy="0 0 0"/>
             <geometry>
-                <mesh filename="file://$(find ros2_humanoid_virtual_twin)/meshes/Left-ArmMounting.stl"/>
+                <mesh filename="file://$(find ros2_humanoid_virtual_twin)/meshes/Right-ArmMounting.stl"/>
             </geometry>
             <material name="grey"/>
@@ -19,5 +19,5 @@
             <origin xyz="0 0 0" rpy="0 0 0"/>
             <geometry>
-                <mesh filename="file://$(find ros2_humanoid_virtual_twin)/meshes/Left-ArmMounting-Collision.stl"/>
+                <mesh filename="file://$(find ros2_humanoid_virtual_twin)/meshes/Right-ArmMounting-Collision.stl"/>
             </geometry>
         </collision>
@@ -25,8 +25,8 @@
             <origin xyz="-3.335e-3 -17.703e-3 0" rpy="0 0 0"/>
             <mass value="0.011"/>
-            <inertia ixx="2.246e-6" iyy="3.894e-6" izz="4.859e-6" ixy="0.637e-6" ixz="0"  iyz="0"/>
+            <inertia ixx="2.246e-6" iyy="3.894e-6" izz="4.859e-6" ixy="-0.637e-6" ixz="0"  iyz="0"/>
         </inertial>
     </link>
-    <gazebo reference="Left_ArmMounting">
+    <gazebo reference="Right_ArmMounting">
         <material>Gazebo/Grey</material>
     </gazebo>

File: description/RobotElements/RightArmElems/Rforearm.xacro (robot description, xacro)
@@ -1,16 +1,16 @@
 <?xml version="1.0"?>
 <robot xmlns:xacro="http://www.ros.org/wiki/xacro" >
-    <joint name="LFAy" type="revolute">
+    <joint name="RFAy" type="revolute">
         <origin xyz="0 0 -112.3e-3" rpy="0 0 0"/>
-        <parent link="Left_Arm"/>
-        <child link="Left_Forearm"/>
+        <parent link="Right_Arm"/>
+        <child link="Right_Forearm"/>
         <axis xyz="0 1.0 0"/>
         <limit lower="${-pi/2}" upper="${pi/2}" effort="100" velocity="100"/>
     </joint>
-    <link name="Left_Forearm">
+    <link name="Right_Forearm">
         <visual>
             <origin xyz="0 0 0" rpy="0 0 0"/>
             <geometry>
-                <mesh filename="file://$(find ros2_humanoid_virtual_twin)/meshes/Left_ForeArm.stl" scale="0.001 0.001 0.001"/>
+                <mesh filename="file://$(find ros2_humanoid_virtual_twin)/meshes/Right_Forearm.stl" scale="0.001 0.001 0.001"/>
             </geometry>
             <material name="grey"/>
@@ -28,5 +28,5 @@
         </inertial>
     </link>
-    <gazebo reference="Left_Forearm">
+    <gazebo reference="Right_Forearm">
         <material>Gazebo/Grey</material>
     </gazebo>

File: description/RobotElements/RightLegElems/Rankle.xacro (robot description, xacro)
@@ -6,5 +6,5 @@
         <child link="Right_Ankle"/>
         <axis xyz="0 1.0 0"/>
-        <limit lower="${-pi}" upper="${pi}" effort="100" velocity="100"/>
+        <limit lower="${-pi/2}" upper="${pi/2}" effort="100" velocity="100"/>
     </joint>
     <link name="Right_Ankle">

File: description/RobotElements/RightLegElems/Rfoot.xacro (robot description, xacro)
@@ -6,5 +6,5 @@
         <child link="Right_Foot"/>
         <axis xyz="1.0 0 0"/>
-        <limit lower="${-pi}" upper="${pi}" effort="100" velocity="100"/>
+        <limit lower="${-pi/2}" upper="${pi/2}" effort="100" velocity="100"/>
     </joint>
     <link name="Right_Foot">

File: description/RobotElements/RightLegElems/Rhip.xacro (robot description, xacro)
@@ -6,5 +6,5 @@
         <child link="Right_Hip"/>
         <axis xyz="1.0 0 0"/>
-        <limit lower="${-pi}" upper="${pi}" effort="100" velocity="100"/>
+        <limit lower="${-pi/2}" upper="${pi/2}" effort="100" velocity="100"/>
     </joint>
     <link name="Right_Hip">

File: description/RobotElements/RightLegElems/Rshank.xacro (robot description, xacro)
@@ -6,5 +6,5 @@
       <child link="Right_Shank"/>
       <axis xyz="0 1.0 0"/>
-      <limit lower="${-pi}" upper="${pi}" effort="100" velocity="100"/>
+      <limit lower="${-pi/2}" upper="${pi/2}" effort="100" velocity="100"/>
     </joint>
     <link name="Right_Shank">

File: description/RobotElements/RightLegElems/Rthigh.xacro (robot description, xacro)
@@ -6,5 +6,5 @@
       <child link="Right_Thigh"/>
       <axis xyz="0 1.0 0"/>
-      <limit lower="${-pi}" upper="${pi}" effort="100" velocity="100"/>
+      <limit lower="${-pi/2}" upper="${pi/2}" effort="100" velocity="100"/>
     </joint>
     <link name="Right_Thigh">

File: description/RobotElements/Trunk.xacro (robot description, xacro)
@@ -6,5 +6,5 @@
       <child link="Trunk"/>
       <!--Origin defines translation child frame relative to parent frame. Translation is performed in parent frame.-->
-      <origin xyz="0 0 0.5" rpy="0 0 0"/>
+      <origin xyz="0 0 0.45" rpy="0 0 0"/>
   </joint>
   <link name="Trunk">

File: description/robot.urdf.xacro (robot description, xacro)
@@ -4,9 +4,9 @@
     <xacro:include filename="robot_core.xacro" />
     <!-- If you want the Trunk to be immovable and static at a certain height uncomment lines below -->
-    <link name="world"/>
+    <!-- <link name="world"/>
     <joint name="world-base_link-fixed" type="fixed">
         <parent link="world"/>
         <child link="base_link"/>
-    </joint>
+    </joint> -->
     <!-- Below is a file which contains parameters controlling movements of a robot -->
 </robot>

File: description/robot_core.xacro (robot description, xacro)
@@ -12,3 +12,5 @@
   <xacro:include filename="RobotElements/right_leg.xacro"/>
   <xacro:include filename="RobotElements/left_arm.xacro"/>
+  <xacro:include filename="RobotElements/right_arm.xacro"/>
+  <xacro:include filename="RobotElements/head.xacro"/>
 </robot>
