Commit message: Solved inertia problems

File: description/RobotElements/HeadElems/Head.xacro (robot description, xacro)
@@ -25,5 +25,5 @@
             <origin xyz="0.022e-3 0.28e-3 11.283e-3" rpy="0 0 0"/>
             <mass value="0.077"/>
-            <inertia ixx="22.035e-6" iyy="18.242e-6" izz="13.649e-6" ixy="-0.008e-6" ixz="-0.02e-6"  iyz="0.689e-3"/>
+            <inertia ixx="22.035e-6" iyy="18.242e-6" izz="13.649e-6" ixy="-0.008e-6" ixz="-0.02e-6"  iyz="0.689e-6"/>
         </inertial>
     </link>

File: description/RobotElements/HeadElems/Headmount.xacro (robot description, xacro)
@@ -25,5 +25,5 @@
             <origin xyz="0 -3.335e-3 -17.703e-3" rpy="0 0 0"/>
             <mass value="0.011"/>
-            <inertia ixx="4.859e-6" iyy="2.246e-6" izz="3.894e-6" ixy="0" ixz="0"  iyz="0.637e-3"/>
+            <inertia ixx="4.859e-6" iyy="2.246e-6" izz="3.894e-6" ixy="0" ixz="0"  iyz="0.637e-6"/>
         </inertial>
     </link>

Commit message: Added xacro property names to set physical properties in gazebo for all links. Robot is stable tipping over

File: description/RobotElements/HeadElems/Head.xacro (robot description, xacro)
@@ -30,9 +30,10 @@
     <gazebo reference="Head">
         <material>Gazebo/Grey</material>
-        <mu1 value="200.0"/>
-        <mu2 value="100.0"/>
-        <kp value="10000000.0" />
-        <kd value="1.0" />
-        <selfCollide>true</selfCollide>
+        <mu1 value="${mu1_val}"/>
+        <mu2 value="${mu2_val}"/>
+        <kp value="${kp_val}" />
+        <kd value="${kd_val}" />
+        <maxVel value="${maxVel_val}"/>
+        <selfCollide>${selfCollide_val}</selfCollide>
     </gazebo>
 </robot>

File: description/RobotElements/HeadElems/Headmount.xacro (robot description, xacro)
@@ -30,9 +30,10 @@
     <gazebo reference="Head_Mounting">
         <material>Gazebo/Grey</material>
-        <mu1 value="200.0"/>
-        <mu2 value="100.0"/>
-        <kp value="10000000.0" />
-        <kd value="1.0" />
-        <selfCollide>true</selfCollide>
+        <mu1 value="${mu1_val}"/>
+        <mu2 value="${mu2_val}"/>
+        <kp value="${kp_val}" />
+        <kd value="${kd_val}" />
+        <maxVel value="${maxVel_val}"/>
+        <selfCollide>${selfCollide_val}</selfCollide>
     </gazebo>
 </robot>

File: description/RobotElements/LeftArmElems/Larm.xacro (robot description, xacro)
@@ -30,9 +30,10 @@
     <gazebo reference="Left_Arm">
         <material>Gazebo/Grey</material>
-        <mu1 value="200.0"/>
-        <mu2 value="100.0"/>
-        <kp value="10000000.0" />
-        <kd value="1.0" />
-        <selfCollide>true</selfCollide>
+        <mu1 value="${mu1_val}"/>
+        <mu2 value="${mu2_val}"/>
+        <kp value="${kp_val}" />
+        <kd value="${kd_val}" />
+        <maxVel value="${maxVel_val}"/>
+        <selfCollide>${selfCollide_val}</selfCollide>
     </gazebo>
 </robot>

File: description/RobotElements/LeftArmElems/Larmmount.xacro (robot description, xacro)
@@ -30,9 +30,10 @@
     <gazebo reference="Left_ArmMounting">
         <material>Gazebo/Grey</material>
-        <mu1 value="200.0"/>
-        <mu2 value="100.0"/>
-        <kp value="10000000.0" />
-        <kd value="1.0" />
-        <selfCollide>true</selfCollide>
+        <mu1 value="${mu1_val}"/>
+        <mu2 value="${mu2_val}"/>
+        <kp value="${kp_val}" />
+        <kd value="${kd_val}" />
+        <maxVel value="${maxVel_val}"/>
+        <selfCollide>${selfCollide_val}</selfCollide>
     </gazebo>
 </robot>

File: description/RobotElements/LeftArmElems/Lforearm.xacro (robot description, xacro)
@@ -30,9 +30,10 @@
     <gazebo reference="Left_Forearm">
         <material>Gazebo/Grey</material>
-        <mu1 value="200.0"/>
-        <mu2 value="100.0"/>
-        <kp value="10000000.0" />
-        <kd value="1.0" />
-        <selfCollide>true</selfCollide>
+        <mu1 value="${mu1_val}"/>
+        <mu2 value="${mu2_val}"/>
+        <kp value="${kp_val}" />
+        <kd value="${kd_val}" />
+        <maxVel value="${maxVel_val}"/>
+        <selfCollide>${selfCollide_val}</selfCollide>
     </gazebo>
 </robot>

File: description/RobotElements/LeftLegElems/Lankle.xacro (robot description, xacro)
@@ -29,10 +29,11 @@
     </link>
     <gazebo reference="Left_Ankle">
-      <material>Gazebo/Grey</material>
-        <mu1 value="200.0"/>
-        <mu2 value="100.0"/>
-        <kp value="10000000.0" />
-        <kd value="1.0" />
-        <selfCollide>true</selfCollide>
+        <material>Gazebo/Grey</material>
+        <mu1 value="${mu1_val}"/>
+        <mu2 value="${mu2_val}"/>
+        <kp value="${kp_val}" />
+        <kd value="${kd_val}" />
+        <maxVel value="${maxVel_val}"/>
+        <selfCollide>${selfCollide_val}</selfCollide>
     </gazebo>
 </robot>

File: description/RobotElements/LeftLegElems/Lfoot.xacro (robot description, xacro)
@@ -30,8 +30,11 @@
     </link>
     <gazebo reference="Left_Foot">
-      <material>Gazebo/Grey</material>
-      <mu1 value="0.002"/>
-      <mu2 value="0.003"/>
-      <kp value="100000.0"/>
+        <material>Gazebo/Grey</material>
+        <mu1 value="0.02"/>
+        <mu2 value="0.03"/>
+        <kp value="${kp_val}" />
+        <kd value="${kd_val}" />
+        <maxVel value="${maxVel_val}"/>
+        <selfCollide>${selfCollide_val}</selfCollide>
     </gazebo>
 </robot>

File: description/RobotElements/LeftLegElems/Lhip.xacro (robot description, xacro)
@@ -30,10 +30,11 @@
     </link>
     <gazebo reference="Left_Hip">
-      <material>Gazebo/Grey</material>
-      <mu1 value="200.0"/>
-      <mu2 value="100.0"/>
-      <kp value="10000000.0" />
-      <kd value="1.0" />
-      <selfCollide>true</selfCollide>
+        <material>Gazebo/Grey</material>
+        <mu1 value="${mu1_val}"/>
+        <mu2 value="${mu2_val}"/>
+        <kp value="${kp_val}" />
+        <kd value="${kd_val}" />
+        <maxVel value="${maxVel_val}"/>
+        <selfCollide>${selfCollide_val}</selfCollide>
     </gazebo>
 </robot>

File: description/RobotElements/LeftLegElems/Lhipmount.xacro (robot description, xacro)
@@ -31,10 +31,11 @@
   </link>
   <gazebo reference="Left_HipMount">
-      <material>Gazebo/Grey</material>
-      <mu1 value="200.0"/>
-      <mu2 value="100.0"/>
-      <kp value="10000000.0" />
-      <kd value="1.0" />
-      <selfCollide>true</selfCollide>
+        <material>Gazebo/Grey</material>
+        <mu1 value="${mu1_val}"/>
+        <mu2 value="${mu2_val}"/>
+        <kp value="${kp_val}" />
+        <kd value="${kd_val}" />
+        <maxVel value="${maxVel_val}"/>
+        <selfCollide>${selfCollide_val}</selfCollide>
   </gazebo>
 </robot>

File: description/RobotElements/LeftLegElems/Lshank.xacro (robot description, xacro)
@@ -29,10 +29,11 @@
     </link>
     <gazebo reference="Left_Shank">
-      <material>Gazebo/Grey</material>
-      <mu1 value="200.0"/>
-      <mu2 value="100.0"/>
-      <kp value="10000000.0" />
-      <kd value="1.0" />
-      <selfCollide>true</selfCollide>
+        <material>Gazebo/Grey</material>
+        <mu1 value="${mu1_val}"/>
+        <mu2 value="${mu2_val}"/>
+        <kp value="${kp_val}" />
+        <kd value="${kd_val}" />
+        <maxVel value="${maxVel_val}"/>
+        <selfCollide>${selfCollide_val}</selfCollide>
     </gazebo>
 </robot>

File: description/RobotElements/LeftLegElems/Lthigh.xacro (robot description, xacro)
@@ -29,10 +29,11 @@
     </link>
     <gazebo reference="Left_Thigh">
-      <material>Gazebo/Grey</material>
-      <mu1 value="200.0"/>
-      <mu2 value="100.0"/>
-      <kp value="10000000.0" />
-      <kd value="1.0" />
-      <selfCollide>true</selfCollide>
+        <material>Gazebo/Grey</material>
+        <mu1 value="${mu1_val}"/>
+        <mu2 value="${mu2_val}"/>
+        <kp value="${kp_val}" />
+        <kd value="${kd_val}" />
+        <maxVel value="${maxVel_val}"/>
+        <selfCollide>${selfCollide_val}</selfCollide>
     </gazebo>
 </robot>

File: description/RobotElements/RightArmElems/Rarm.xacro (robot description, xacro)
@@ -30,9 +30,10 @@
     <gazebo reference="Right_Arm">
         <material>Gazebo/Grey</material>
-        <mu1 value="200.0"/>
-        <mu2 value="100.0"/>
-        <kp value="10000000.0" />
-        <kd value="1.0" />
-        <selfCollide>true</selfCollide>
+        <mu1 value="${mu1_val}"/>
+        <mu2 value="${mu2_val}"/>
+        <kp value="${kp_val}" />
+        <kd value="${kd_val}" />
+        <maxVel value="${maxVel_val}"/>
+        <selfCollide>${selfCollide_val}</selfCollide>
     </gazebo>
 </robot>

File: description/RobotElements/RightArmElems/Rarmmount.xacro (robot description, xacro)
@@ -30,9 +30,10 @@
     <gazebo reference="Right_ArmMounting">
         <material>Gazebo/Grey</material>
-        <mu1 value="200.0"/>
-        <mu2 value="100.0"/>
-        <kp value="10000000.0" />
-        <kd value="1.0" />
-        <selfCollide>true</selfCollide>
+        <mu1 value="${mu1_val}"/>
+        <mu2 value="${mu2_val}"/>
+        <kp value="${kp_val}" />
+        <kd value="${kd_val}" />
+        <maxVel value="${maxVel_val}"/>
+        <selfCollide>${selfCollide_val}</selfCollide>
     </gazebo>
 </robot>

File: description/RobotElements/RightArmElems/Rforearm.xacro (robot description, xacro)
@@ -30,9 +30,10 @@
     <gazebo reference="Right_Forearm">
         <material>Gazebo/Grey</material>
-        <mu1 value="200.0"/>
-        <mu2 value="100.0"/>
-        <kp value="10000000.0" />
-        <kd value="1.0" />
-        <selfCollide>true</selfCollide>
+        <mu1 value="${mu1_val}"/>
+        <mu2 value="${mu2_val}"/>
+        <kp value="${kp_val}" />
+        <kd value="${kd_val}" />
+        <maxVel value="${maxVel_val}"/>
+        <selfCollide>${selfCollide_val}</selfCollide>
     </gazebo>
 </robot>

File: description/RobotElements/RightLegElems/Rankle.xacro (robot description, xacro)
@@ -32,9 +32,10 @@
     <gazebo reference="Right_Ankle">
         <material>Gazebo/Grey</material>
-        <mu1 value="200.0"/>
-        <mu2 value="100.0"/>
-        <kp value="10000000.0" />
-        <kd value="1.0" />
-        <selfCollide>true</selfCollide>
+        <mu1 value="${mu1_val}"/>
+        <mu2 value="${mu2_val}"/>
+        <kp value="${kp_val}" />
+        <kd value="${kd_val}" />
+        <maxVel value="${maxVel_val}"/>
+        <selfCollide>${selfCollide_val}</selfCollide>
     </gazebo>
 </robot>

File: description/RobotElements/RightLegElems/Rfoot.xacro (robot description, xacro)
@@ -30,7 +30,10 @@
     <gazebo reference="Right_Foot">
         <material>Gazebo/Grey</material>
-        <mu1 value="0.002"/>
-        <mu2 value="0.003"/>
-        <kp value="100000.0"/>
+        <mu1 value="0.02"/>
+        <mu2 value="0.03"/>
+        <kp value="${kp_val}" />
+        <kd value="${kd_val}" />
+        <maxVel value="${maxVel_val}"/>
+        <selfCollide>${selfCollide_val}</selfCollide>
     </gazebo>
 </robot>

File: description/RobotElements/RightLegElems/Rhip.xacro (robot description, xacro)
@@ -30,9 +30,10 @@
     <gazebo reference="Right_Hip">
         <material>Gazebo/Grey</material>
-        <mu1 value="200.0"/>
-        <mu2 value="100.0"/>
-        <kp value="10000000.0" />
-        <kd value="1.0" />
-        <selfCollide>true</selfCollide>
+        <mu1 value="${mu1_val}"/>
+        <mu2 value="${mu2_val}"/>
+        <kp value="${kp_val}" />
+        <kd value="${kd_val}" />
+        <maxVel value="${maxVel_val}"/>
+        <selfCollide>${selfCollide_val}</selfCollide>
     </gazebo>
 </robot>

File: description/RobotElements/RightLegElems/Rhipmount.xacro (robot description, xacro)
@@ -30,9 +30,10 @@
     <gazebo reference="Right_HipMount">
         <material>Gazebo/Grey</material>
-        <mu1 value="200.0"/>
-        <mu2 value="100.0"/>
-        <kp value="10000000.0" />
-        <kd value="1.0" />
-        <selfCollide>true</selfCollide>
+        <mu1 value="${mu1_val}"/>
+        <mu2 value="${mu2_val}"/>
+        <kp value="${kp_val}" />
+        <kd value="${kd_val}" />
+        <maxVel value="${maxVel_val}"/>
+        <selfCollide>${selfCollide_val}</selfCollide>
     </gazebo>
 </robot>

File: description/RobotElements/RightLegElems/Rshank.xacro (robot description, xacro)
@@ -30,9 +30,10 @@
     <gazebo reference="Right_Shank">
         <material>Gazebo/Grey</material>
-        <mu1 value="200.0"/>
-        <mu2 value="100.0"/>
-        <kp value="10000000.0" />
-        <kd value="1.0" />
-        <selfCollide>true</selfCollide>
+        <mu1 value="${mu1_val}"/>
+        <mu2 value="${mu2_val}"/>
+        <kp value="${kp_val}" />
+        <kd value="${kd_val}" />
+        <maxVel value="${maxVel_val}"/>
+        <selfCollide>${selfCollide_val}</selfCollide>
     </gazebo>
  </robot>

File: description/RobotElements/RightLegElems/Rthigh.xacro (robot description, xacro)
@@ -30,9 +30,10 @@
     <gazebo reference="Right_Thigh">
         <material>Gazebo/Grey</material>
-        <mu1 value="200.0"/>
-        <mu2 value="100.0"/>
-        <kp value="10000000.0" />
-        <kd value="1.0" />
-        <selfCollide>true</selfCollide>
+        <mu1 value="${mu1_val}"/>
+        <mu2 value="${mu2_val}"/>
+        <kp value="${kp_val}" />
+        <kd value="${kd_val}" />
+        <maxVel value="${maxVel_val}"/>
+        <selfCollide>${selfCollide_val}</selfCollide>
     </gazebo>
 </robot>
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