Commit message: Added automatic setting and unsetting GAZEBO joints and links physics coefficients AND URDF joint dynamics automatic setting and unsetting. It is possible now to set also those values for every coefficient from one place

File: description/RobotElements/HeadElems/Head.xacro (robot description, xacro)
@@ -6,5 +6,8 @@
         <child link="Head"/>
         <axis xyz="0 1.0 0"/>
-        <limit lower="${-pi/2}" upper="${pi/2}" effort="1" velocity="1"/>
+        <limit lower="${-pi/2}" upper="${pi/2}" effort="${maxeffort_val}" velocity="${maxVel_val}"/>
+        <xacro:if value="$(arg use_URDF_joint_dynamics_coefficients)">
+            <dynamics damping="${damping_val}" friction="${friction_val}"/>
+        </xacro:if>
     </joint>
     <link name="Head">
@@ -28,4 +31,5 @@
         </inertial>
     </link>
+  <xacro:if value="$(arg use_gazebo_joint_physics_coefficients)">
     <gazebo reference="Hy">
         <implicitSpringDamper>${Damper_val}</implicitSpringDamper>
@@ -35,13 +39,16 @@
         <stopCfm>${stopCfm_val}</stopCfm>
     </gazebo>
+    </xacro:if>
     <gazebo reference="Head">
         <material>Gazebo/Grey</material>
-        <mu1 value="${mu1_val}"/>
-        <mu2 value="${mu2_val}"/>
-        <kp value="${kp_val}" />
-        <kd value="${kd_val}" />
-        <maxVel value="${maxVel_val}"/>
-        <dampingFactor value="${dampigFactor_val}"/>
-        <selfCollide>${selfCollide_val}</selfCollide>
+        <xacro:if value="$(arg use_gazebo_link_physics_coefficients)">
+          <mu1 value="${mu1_val}"/>
+          <mu2 value="${mu2_val}"/>
+          <kp value="${kp_val}" />
+          <kd value="${kd_val}" />
+          <maxVel value="${maxVel_val}"/>
+          <dampingFactor value="${dampigFactor_val}"/>
+          <selfCollide>${selfCollide_val}</selfCollide>
+        </xacro:if>
     </gazebo>
 </robot>

File: description/RobotElements/HeadElems/Headmount.xacro (robot description, xacro)
@@ -6,5 +6,8 @@
         <child link="Head_Mounting"/>
         <axis xyz="0 0 1.0"/>
-        <limit lower="${-pi/2}" upper="${pi/2}" effort="1" velocity="1"/>
+        <limit lower="${-pi/2}" upper="${pi/2}" effort="${maxeffort_val}" velocity="${maxVel_val}"/>
+        <xacro:if value="$(arg use_URDF_joint_dynamics_coefficients)">
+            <dynamics damping="${damping_val}" friction="${friction_val}"/>
+        </xacro:if>
     </joint>
     <link name="Head_Mounting">
@@ -28,20 +31,24 @@
         </inertial>
     </link>
-    <gazebo reference="Hz">
-        <implicitSpringDamper>${Damper_val}</implicitSpringDamper>
-        <springStiffness>${springstiffness_val}</springStiffness>
-        <springReference>${springReference_val}</springReference>
-        <stopErp>${stopErp_val}</stopErp>
-        <stopCfm>${stopCfm_val}</stopCfm>
-    </gazebo>
+    <xacro:if value="$(arg use_gazebo_joint_physics_coefficients)">
+        <gazebo reference="Hz">
+            <implicitSpringDamper>${Damper_val}</implicitSpringDamper>
+            <springStiffness>${springstiffness_val}</springStiffness>
+            <springReference>${springReference_val}</springReference>
+            <stopErp>${stopErp_val}</stopErp>
+            <stopCfm>${stopCfm_val}</stopCfm>
+        </gazebo>
+    </xacro:if>
     <gazebo reference="Head_Mounting">
         <material>Gazebo/Grey</material>
-        <mu1 value="${mu1_val}"/>
-        <mu2 value="${mu2_val}"/>
-        <kp value="${kp_val}" />
-        <kd value="${kd_val}" />
-        <maxVel value="${maxVel_val}"/>
-        <dampingFactor value="${dampigFactor_val}"/>
-        <selfCollide>${selfCollide_val}</selfCollide>
+        <xacro:if value="$(arg use_gazebo_link_physics_coefficients)">
+          <mu1 value="${mu1_val}"/>
+          <mu2 value="${mu2_val}"/>
+          <kp value="${kp_val}" />
+          <kd value="${kd_val}" />
+          <maxVel value="${maxVel_val}"/>
+          <dampingFactor value="${dampigFactor_val}"/>
+          <selfCollide>${selfCollide_val}</selfCollide>
+        </xacro:if>
     </gazebo>
 </robot>

File: description/RobotElements/LeftArmElems/Larm.xacro (robot description, xacro)
@@ -6,5 +6,8 @@
         <child link="Left_Arm"/>
         <axis xyz="1.0 0 0"/>
-        <limit lower="${-pi/2}" upper="${pi/2}" effort="1" velocity="1"/>
+        <limit lower="${-pi/2}" upper="${pi/2}" effort="${maxeffort_val}" velocity="${maxVel_val}"/>
+        <xacro:if value="$(arg use_URDF_joint_dynamics_coefficients)">
+            <dynamics damping="${damping_val}" friction="${friction_val}"/>
+        </xacro:if>
     </joint>
     <link name="Left_Arm">
@@ -28,4 +31,5 @@
         </inertial>
     </link>
+    <xacro:if value="$(arg use_gazebo_joint_physics_coefficients)">
     <gazebo reference="LAx">
         <implicitSpringDamper>${Damper_val}</implicitSpringDamper>
@@ -35,13 +39,16 @@
         <stopCfm>${stopCfm_val}</stopCfm>
     </gazebo>
+    </xacro:if>
     <gazebo reference="Left_Arm">
         <material>Gazebo/Grey</material>
-        <mu1 value="${mu1_val}"/>
-        <mu2 value="${mu2_val}"/>
-        <kp value="${kp_val}" />
-        <kd value="${kd_val}" />
-        <maxVel value="${maxVel_val}"/>
-        <dampingFactor value="${dampigFactor_val}"/>
-        <selfCollide>${selfCollide_val}</selfCollide>
+        <xacro:if value="$(arg use_gazebo_link_physics_coefficients)">
+          <mu1 value="${mu1_val}"/>
+          <mu2 value="${mu2_val}"/>
+          <kp value="${kp_val}" />
+          <kd value="${kd_val}" />
+          <maxVel value="${maxVel_val}"/>
+          <dampingFactor value="${dampigFactor_val}"/>
+          <selfCollide>${selfCollide_val}</selfCollide>
+        </xacro:if>
     </gazebo>
 </robot>

File: description/RobotElements/LeftArmElems/Larmmount.xacro (robot description, xacro)
@@ -6,5 +6,8 @@
         <child link="Left_ArmMounting"/>
         <axis xyz="0 1.0 0"/>
-        <limit lower="${-pi/2}" upper="${pi/2}" effort="1" velocity="1"/>
+        <limit lower="${-pi/2}" upper="${pi/2}" effort="${maxeffort_val}" velocity="${maxVel_val}"/>
+        <xacro:if value="$(arg use_URDF_joint_dynamics_coefficients)">
+            <dynamics damping="${damping_val}" friction="${friction_val}"/>
+        </xacro:if>
     </joint>
     <link name="Left_ArmMounting">
@@ -28,4 +31,5 @@
         </inertial>
     </link>
+    <xacro:if value="$(arg use_gazebo_joint_physics_coefficients)">
     <gazebo reference="LAy">
         <implicitSpringDamper>${Damper_val}</implicitSpringDamper>
@@ -35,13 +39,16 @@
         <stopCfm>${stopCfm_val}</stopCfm>
     </gazebo>
+    </xacro:if>
     <gazebo reference="Left_ArmMounting">
         <material>Gazebo/Grey</material>
-        <mu1 value="${mu1_val}"/>
-        <mu2 value="${mu2_val}"/>
-        <kp value="${kp_val}" />
-        <kd value="${kd_val}" />
-        <maxVel value="${maxVel_val}"/>
-        <dampingFactor value="${dampigFactor_val}"/>
-        <selfCollide>${selfCollide_val}</selfCollide>
+        <xacro:if value="$(arg use_gazebo_link_physics_coefficients)">
+          <mu1 value="${mu1_val}"/>
+          <mu2 value="${mu2_val}"/>
+          <kp value="${kp_val}" />
+          <kd value="${kd_val}" />
+          <maxVel value="${maxVel_val}"/>
+          <dampingFactor value="${dampigFactor_val}"/>
+          <selfCollide>${selfCollide_val}</selfCollide>
+        </xacro:if>
     </gazebo>
 </robot>

File: description/RobotElements/LeftArmElems/Lforearm.xacro (robot description, xacro)
@@ -6,5 +6,8 @@
         <child link="Left_Forearm"/>
         <axis xyz="0 1.0 0"/>
-        <limit lower="${-pi/2}" upper="${pi/2}" effort="1" velocity="1"/>
+        <limit lower="${-pi/2}" upper="${pi/2}" effort="${maxeffort_val}" velocity="${maxVel_val}"/>
+        <xacro:if value="$(arg use_URDF_joint_dynamics_coefficients)">
+            <dynamics damping="${damping_val}" friction="${friction_val}"/>
+        </xacro:if>
     </joint>
     <link name="Left_Forearm">
@@ -28,4 +31,5 @@
         </inertial>
     </link>
+    <xacro:if value="$(arg use_gazebo_joint_physics_coefficients)">
     <gazebo reference="LFAy">
         <implicitSpringDamper>${Damper_val}</implicitSpringDamper>
@@ -35,13 +39,16 @@
         <stopCfm>${stopCfm_val}</stopCfm>
     </gazebo>
+    </xacro:if>
     <gazebo reference="Left_Forearm">
         <material>Gazebo/Grey</material>
-        <!-- <mu1 value="${mu1_val}"/>
-        <mu2 value="${mu2_val}"/>
-        <kp value="${kp_val}" />
-        <kd value="${kd_val}" />
-        <maxVel value="${maxVel_val}"/>
-        <dampingFactor value="${dampigFactor_val}"/>
-        <selfCollide>${selfCollide_val}</selfCollide>   -->
+        <!-- <xacro:if value="$(arg use_gazebo_link_physics_coefficients)">
+          <mu1 value="${mu1_val}"/>
+          <mu2 value="${mu2_val}"/>
+          <kp value="${kp_val}" />
+          <kd value="${kd_val}" />
+          <maxVel value="${maxVel_val}"/>
+          <dampingFactor value="${dampigFactor_val}"/>
+          <selfCollide>${selfCollide_val}</selfCollide>
+        </xacro:if> -->
     </gazebo>
 </robot>

File: description/RobotElements/LeftLegElems/Lankle.xacro (robot description, xacro)
@@ -6,5 +6,8 @@
       <child link="Left_Ankle"/>
       <axis xyz="0 1.0 0"/>
-      <limit lower="${-pi/2}" upper="${pi/2}" effort="1" velocity="1"/>
+      <limit lower="${-pi/2}" upper="${pi/2}" effort="${maxeffort_val}" velocity="${maxVel_val}"/>
+      <xacro:if value="$(arg use_URDF_joint_dynamics_coefficients)">
+          <dynamics damping="${damping_val}" friction="${friction_val}"/>
+      </xacro:if>
     </joint>
 	<link name="Left_Ankle">
@@ -28,4 +31,5 @@
       </inertial>
     </link>
+    <xacro:if value="$(arg use_gazebo_joint_physics_coefficients)">
     <gazebo reference="LFy">
         <implicitSpringDamper>${Damper_val}</implicitSpringDamper>
@@ -35,13 +39,16 @@
         <stopCfm>${stopCfm_val}</stopCfm>
     </gazebo>
+    </xacro:if>
     <gazebo reference="Left_Ankle">
         <material>Gazebo/Grey</material>
-        <mu1 value="${mu1_val}"/>
-        <mu2 value="${mu2_val}"/>
-        <kp value="${kp_val}" />
-        <kd value="${kd_val}" />
-        <maxVel value="${maxVel_val}"/>
-        <dampingFactor value="${dampigFactor_val}"/>
-        <selfCollide>${selfCollide_val}</selfCollide>
+        <xacro:if value="$(arg use_gazebo_link_physics_coefficients)">
+          <mu1 value="${mu1_val}"/>
+          <mu2 value="${mu2_val}"/>
+          <kp value="${kp_val}" />
+          <kd value="${kd_val}" />
+          <maxVel value="${maxVel_val}"/>
+          <dampingFactor value="${dampigFactor_val}"/>
+          <selfCollide>${selfCollide_val}</selfCollide>
+        </xacro:if>
     </gazebo>
 </robot>

File: description/RobotElements/LeftLegElems/Lfoot.xacro (robot description, xacro)
@@ -6,6 +6,8 @@
       <child link="Left_Foot"/>
       <axis xyz="1.0 0 0"/>
-      <limit lower="${-pi/2}" upper="${pi/2}" effort="1" velocity="1"/>
-      <dynamics damping="${damping_val}" friction="${friction_val}"/>
+      <limit lower="${-pi/2}" upper="${pi/2}" effort="${maxeffort_val}" velocity="${maxVel_val}"/>
+      <xacro:if value="$(arg use_URDF_joint_dynamics_coefficients)">
+        <dynamics damping="${damping_val}" friction="${friction_val}"/>
+      </xacro:if>
     </joint>
     <link name="Left_Foot">
@@ -30,20 +32,24 @@
       </inertial>
     </link>
-  <gazebo reference="LFx">
-    <implicitSpringDamper>${Damper_val}</implicitSpringDamper>
-    <springStiffness>${springstiffness_val}</springStiffness>
-    <springReference>${springReference_val}</springReference>
-    <stopErp>${stopErp_val}</stopErp>
-    <stopCfm>${stopCfm_val}</stopCfm>
-  </gazebo>
+  <xacro:if value="$(arg use_gazebo_joint_physics_coefficients)">
+    <gazebo reference="LFx">
+      <implicitSpringDamper>${Damper_val}</implicitSpringDamper>
+      <springStiffness>${springstiffness_val}</springStiffness>
+      <springReference>${springReference_val}</springReference>
+      <stopErp>${stopErp_val}</stopErp>
+      <stopCfm>${stopCfm_val}</stopCfm>
+    </gazebo>
+  </xacro:if>
     <gazebo reference="Left_Foot">
         <material>Gazebo/Grey</material>
-        <mu1 value="${mu1_val}"/>
-        <mu2 value="${mu2_val}"/>
-        <kp value="${kp_val}" />
-        <kd value="${kd_val}" />
-        <maxVel value="${maxVel_val}"/>
-        <dampingFactor value="${dampigFactor_val}"/>
-        <selfCollide>${selfCollide_val}</selfCollide>
+        <xacro:if value="$(arg use_gazebo_link_physics_coefficients)">
+          <mu1 value="${mu1_val}"/>
+          <mu2 value="${mu2_val}"/>
+          <kp value="${kp_val}" />
+          <kd value="${kd_val}" />
+          <maxVel value="${maxVel_val}"/>
+          <dampingFactor value="${dampigFactor_val}"/>
+          <selfCollide>${selfCollide_val}</selfCollide>
+        </xacro:if>
     </gazebo>
 </robot>

File: description/RobotElements/LeftLegElems/Lhip.xacro (robot description, xacro)
@@ -7,5 +7,8 @@
       <child link="Left_Hip"/>
       <axis xyz="1.0 0 0"/>
-      <limit lower="${-pi/2}" upper="${pi/2}" effort="1" velocity="1"/>
+      <limit lower="${-pi/2}" upper="${pi/2}" effort="${maxeffort_val}" velocity="${maxVel_val}"/>
+      <xacro:if value="$(arg use_URDF_joint_dynamics_coefficients)">
+          <dynamics damping="${damping_val}" friction="${friction_val}"/>
+      </xacro:if>
     </joint>
     <link name="Left_Hip">
@@ -29,4 +32,5 @@
       </inertial>
     </link>
+    <xacro:if value="$(arg use_gazebo_joint_physics_coefficients)">
     <gazebo reference="LTx">
         <implicitSpringDamper>${Damper_val}</implicitSpringDamper>
@@ -36,13 +40,16 @@
         <stopCfm>${stopCfm_val}</stopCfm>
     </gazebo>
+    </xacro:if>
     <gazebo reference="Left_Hip">
         <material>Gazebo/Grey</material>
-        <mu1 value="${mu1_val}"/>
-        <mu2 value="${mu2_val}"/>
-        <kp value="${kp_val}" />
-        <kd value="${kd_val}" />
-        <maxVel value="${maxVel_val}"/>
-        <dampingFactor value="${dampigFactor_val}"/>
-        <selfCollide>${selfCollide_val}</selfCollide>
+        <xacro:if value="$(arg use_gazebo_link_physics_coefficients)">
+          <mu1 value="${mu1_val}"/>
+          <mu2 value="${mu2_val}"/>
+          <kp value="${kp_val}" />
+          <kd value="${kd_val}" />
+          <maxVel value="${maxVel_val}"/>
+          <dampingFactor value="${dampigFactor_val}"/>
+          <selfCollide>${selfCollide_val}</selfCollide>
+        </xacro:if>
     </gazebo>
 </robot>

File: description/RobotElements/LeftLegElems/Lhipmount.xacro (robot description, xacro)
@@ -8,5 +8,8 @@
     <child link="Left_HipMount"/>
     <axis xyz="0 0 1.0"/>
-    <limit lower="${-pi/2}" upper="${pi/2}" effort="1" velocity="1"/>
+    <limit lower="${-pi/2}" upper="${pi/2}" effort="${maxeffort_val}" velocity="${maxVel_val}"/>
+    <xacro:if value="$(arg use_URDF_joint_dynamics_coefficients)">
+        <dynamics damping="${damping_val}" friction="${friction_val}"/>
+    </xacro:if>
   </joint>
   <link name="Left_HipMount">
@@ -30,4 +33,5 @@
     </inertial>
   </link>
+  <xacro:if value="$(arg use_gazebo_joint_physics_coefficients)">
   <gazebo reference="LTz">
     <implicitSpringDamper>${Damper_val}</implicitSpringDamper>
@@ -37,13 +41,16 @@
     <stopCfm>${stopCfm_val}</stopCfm>
   </gazebo>
+  </xacro:if>
   <gazebo reference="Left_HipMount">
         <material>Gazebo/Grey</material>
-        <mu1 value="${mu1_val}"/>
-        <mu2 value="${mu2_val}"/>
-        <kp value="${kp_val}" />
-        <kd value="${kd_val}" />
-        <maxVel value="${maxVel_val}"/>
-        <dampingFactor value="${dampigFactor_val}"/>
-        <selfCollide>${selfCollide_val}</selfCollide>
+        <xacro:if value="$(arg use_gazebo_link_physics_coefficients)">
+          <mu1 value="${mu1_val}"/>
+          <mu2 value="${mu2_val}"/>
+          <kp value="${kp_val}" />
+          <kd value="${kd_val}" />
+          <maxVel value="${maxVel_val}"/>
+          <dampingFactor value="${dampigFactor_val}"/>
+          <selfCollide>${selfCollide_val}</selfCollide>
+        </xacro:if>
   </gazebo>
 </robot>

File: description/RobotElements/LeftLegElems/Lshank.xacro (robot description, xacro)
@@ -6,5 +6,8 @@
       <child link="Left_Shank"/>
       <axis xyz="0 1.0 0"/>
-      <limit lower="${-pi/2}" upper="${pi/2}" effort="1" velocity="1"/>
+      <limit lower="${-pi/2}" upper="${pi/2}" effort="${maxeffort_val}" velocity="${maxVel_val}"/>
+      <xacro:if value="$(arg use_URDF_joint_dynamics_coefficients)">
+          <dynamics damping="${damping_val}" friction="${friction_val}"/>
+      </xacro:if>
     </joint>
 	<link name="Left_Shank">
@@ -28,4 +31,5 @@
       </inertial>
     </link>
+    <xacro:if value="$(arg use_gazebo_joint_physics_coefficients)">
     <gazebo reference="LSy">
         <implicitSpringDamper>${Damper_val}</implicitSpringDamper>
@@ -35,13 +39,16 @@
         <stopCfm>${stopCfm_val}</stopCfm>
     </gazebo>
+    </xacro:if>
     <gazebo reference="Left_Shank">
         <material>Gazebo/Grey</material>
-        <mu1 value="${mu1_val}"/>
-        <mu2 value="${mu2_val}"/>
-        <kp value="${kp_val}" />
-        <kd value="${kd_val}" />
-        <maxVel value="${maxVel_val}"/>
-        <dampingFactor value="${dampigFactor_val}"/>
-        <selfCollide>${selfCollide_val}</selfCollide>
+        <xacro:if value="$(arg use_gazebo_link_physics_coefficients)">
+          <mu1 value="${mu1_val}"/>
+          <mu2 value="${mu2_val}"/>
+          <kp value="${kp_val}" />
+          <kd value="${kd_val}" />
+          <maxVel value="${maxVel_val}"/>
+          <dampingFactor value="${dampigFactor_val}"/>
+          <selfCollide>${selfCollide_val}</selfCollide>
+        </xacro:if>
     </gazebo>
 </robot>

File: description/RobotElements/LeftLegElems/Lthigh.xacro (robot description, xacro)
@@ -6,5 +6,8 @@
       <child link="Left_Thigh"/>
       <axis xyz="0 1.0 0"/>
-      <limit lower="${-pi/2}" upper="${pi/2}" effort="1" velocity="1"/>
+      <limit lower="${-pi/2}" upper="${pi/2}" effort="${maxeffort_val}" velocity="${maxVel_val}"/>
+      <xacro:if value="$(arg use_URDF_joint_dynamics_coefficients)">
+          <dynamics damping="${damping_val}" friction="${friction_val}"/>
+      </xacro:if>
     </joint>
     <link name="Left_Thigh">
@@ -28,4 +31,5 @@
       </inertial>
     </link>
+    <xacro:if value="$(arg use_gazebo_joint_physics_coefficients)">
     <gazebo reference="LTy">
         <implicitSpringDamper>${Damper_val}</implicitSpringDamper>
@@ -35,13 +39,16 @@
         <stopCfm>${stopCfm_val}</stopCfm>
     </gazebo>
+    </xacro:if>
     <gazebo reference="Left_Thigh">
         <material>Gazebo/Grey</material>
-        <mu1 value="${mu1_val}"/>
-        <mu2 value="${mu2_val}"/>
-        <kp value="${kp_val}" />
-        <kd value="${kd_val}" />
-        <maxVel value="${maxVel_val}"/>
-        <dampingFactor value="${dampigFactor_val}"/>
-        <selfCollide>${selfCollide_val}</selfCollide>
+        <xacro:if value="$(arg use_gazebo_link_physics_coefficients)">
+          <mu1 value="${mu1_val}"/>
+          <mu2 value="${mu2_val}"/>
+          <kp value="${kp_val}" />
+          <kd value="${kd_val}" />
+          <maxVel value="${maxVel_val}"/>
+          <dampingFactor value="${dampigFactor_val}"/>
+          <selfCollide>${selfCollide_val}</selfCollide>
+        </xacro:if>
     </gazebo>
 </robot>

File: description/RobotElements/RightArmElems/Rarm.xacro (robot description, xacro)
@@ -6,5 +6,8 @@
         <child link="Right_Arm"/>
         <axis xyz="1.0 0 0"/>
-        <limit lower="${-pi/2}" upper="${pi/2}" effort="1" velocity="1"/>
+        <limit lower="${-pi/2}" upper="${pi/2}" effort="${maxeffort_val}" velocity="${maxVel_val}"/>
+        <xacro:if value="$(arg use_URDF_joint_dynamics_coefficients)">
+            <dynamics damping="${damping_val}" friction="${friction_val}"/>
+        </xacro:if>
     </joint>
     <link name="Right_Arm">
@@ -28,4 +31,5 @@
         </inertial>
     </link>
+    <xacro:if value="$(arg use_gazebo_joint_physics_coefficients)">
     <gazebo reference="RAx">
         <implicitSpringDamper>${Damper_val}</implicitSpringDamper>
@@ -35,13 +39,16 @@
         <stopCfm>${stopCfm_val}</stopCfm>
     </gazebo>
+    </xacro:if>
     <gazebo reference="Right_Arm">
         <material>Gazebo/Grey</material>
-        <mu1 value="${mu1_val}"/>
-        <mu2 value="${mu2_val}"/>
-        <kp value="${kp_val}" />
-        <kd value="${kd_val}" />
-        <maxVel value="${maxVel_val}"/>
-        <dampingFactor value="${dampigFactor_val}"/>
-        <selfCollide>${selfCollide_val}</selfCollide>
+        <xacro:if value="$(arg use_gazebo_link_physics_coefficients)">
+          <mu1 value="${mu1_val}"/>
+          <mu2 value="${mu2_val}"/>
+          <kp value="${kp_val}" />
+          <kd value="${kd_val}" />
+          <maxVel value="${maxVel_val}"/>
+          <dampingFactor value="${dampigFactor_val}"/>
+          <selfCollide>${selfCollide_val}</selfCollide>
+        </xacro:if>
     </gazebo>
 </robot>

File: description/RobotElements/RightArmElems/Rarmmount.xacro (robot description, xacro)
@@ -6,5 +6,8 @@
         <child link="Right_ArmMounting"/>
         <axis xyz="0 1.0 0"/>
-        <limit lower="${-pi/2}" upper="${pi/2}" effort="1" velocity="1"/>
+        <limit lower="${-pi/2}" upper="${pi/2}" effort="${maxeffort_val}" velocity="${maxVel_val}"/>
+        <xacro:if value="$(arg use_URDF_joint_dynamics_coefficients)">
+            <dynamics damping="${damping_val}" friction="${friction_val}"/>
+        </xacro:if>
     </joint>
     <link name="Right_ArmMounting">
@@ -28,4 +31,5 @@
         </inertial>
     </link>
+    <xacro:if value="$(arg use_gazebo_joint_physics_coefficients)">
     <gazebo reference="RAy">
         <implicitSpringDamper>${Damper_val}</implicitSpringDamper>
@@ -35,13 +39,16 @@
         <stopCfm>${stopCfm_val}</stopCfm>
     </gazebo>
+    </xacro:if>
     <gazebo reference="Right_ArmMounting">
         <material>Gazebo/Grey</material>
-        <mu1 value="${mu1_val}"/>
-        <mu2 value="${mu2_val}"/>
-        <kp value="${kp_val}" />
-        <kd value="${kd_val}" />
-        <maxVel value="${maxVel_val}"/>
-        <dampingFactor value="${dampigFactor_val}"/>
-        <selfCollide>${selfCollide_val}</selfCollide>
+        <xacro:if value="$(arg use_gazebo_link_physics_coefficients)">
+          <mu1 value="${mu1_val}"/>
+          <mu2 value="${mu2_val}"/>
+          <kp value="${kp_val}" />
+          <kd value="${kd_val}" />
+          <maxVel value="${maxVel_val}"/>
+          <dampingFactor value="${dampigFactor_val}"/>
+          <selfCollide>${selfCollide_val}</selfCollide>
+        </xacro:if>
     </gazebo>
 </robot>
