Commit message: Added automatic setting and unsetting GAZEBO joints and links physics coefficients AND URDF joint dynamics automatic setting and unsetting. It is possible now to set also those values for every coefficient from one place

File: description/RobotElements/RightArmElems/Rforearm.xacro (robot description, xacro)
@@ -6,5 +6,8 @@
         <child link="Right_Forearm"/>
         <axis xyz="0 1.0 0"/>
-        <limit lower="${-pi/2}" upper="${pi/2}" effort="1" velocity="1"/>
+        <limit lower="${-pi/2}" upper="${pi/2}" effort="${maxeffort_val}" velocity="${maxVel_val}"/>
+        <xacro:if value="$(arg use_URDF_joint_dynamics_coefficients)">
+            <dynamics damping="${damping_val}" friction="${friction_val}"/>
+        </xacro:if>
     </joint>
     <link name="Right_Forearm">
@@ -28,4 +31,5 @@
         </inertial>
     </link>
+    <xacro:if value="$(arg use_gazebo_joint_physics_coefficients)">
     <gazebo reference="RFAy">
         <implicitSpringDamper>${Damper_val}</implicitSpringDamper>
@@ -35,13 +39,16 @@
         <stopCfm>${stopCfm_val}</stopCfm>
     </gazebo>
+    </xacro:if>
     <gazebo reference="Right_Forearm">
         <material>Gazebo/Grey</material>
-        <!-- <mu1 value="${mu1_val}"/>
-        <mu2 value="${mu2_val}"/>
-        <kp value="${kp_val}" />
-        <kd value="${kd_val}" />
-        <maxVel value="${maxVel_val}"/>
-        <dampingFactor value="${dampigFactor_val}"/>
-        <selfCollide>${selfCollide_val}</selfCollide>    -->
+        <!-- <xacro:if value="$(arg use_gazebo_link_physics_coefficients)">
+          <mu1 value="${mu1_val}"/>
+          <mu2 value="${mu2_val}"/>
+          <kp value="${kp_val}" />
+          <kd value="${kd_val}" />
+          <maxVel value="${maxVel_val}"/>
+          <dampingFactor value="${dampigFactor_val}"/>
+          <selfCollide>${selfCollide_val}</selfCollide>
+        </xacro:if> -->
     </gazebo>
 </robot>

File: description/RobotElements/RightLegElems/Rankle.xacro (robot description, xacro)
@@ -6,5 +6,8 @@
         <child link="Right_Ankle"/>
         <axis xyz="0 1.0 0"/>
-        <limit lower="${-pi/2}" upper="${pi/2}" effort="1" velocity="1"/>
+        <limit lower="${-pi/2}" upper="${pi/2}" effort="${maxeffort_val}" velocity="${maxVel_val}"/>
+        <xacro:if value="$(arg use_URDF_joint_dynamics_coefficients)">
+            <dynamics damping="${damping_val}" friction="${friction_val}"/>
+        </xacro:if>
     </joint>
     <link name="Right_Ankle">
@@ -30,4 +33,5 @@
         </inertial>
     </link>
+    <xacro:if value="$(arg use_gazebo_joint_physics_coefficients)">
     <gazebo reference="RFy">
         <implicitSpringDamper>${Damper_val}</implicitSpringDamper>
@@ -37,13 +41,16 @@
         <stopCfm>${stopCfm_val}</stopCfm>
     </gazebo>
+    </xacro:if>
     <gazebo reference="Right_Ankle">
         <material>Gazebo/Grey</material>
-        <mu1 value="${mu1_val}"/>
-        <mu2 value="${mu2_val}"/>
-        <kp value="${kp_val}" />
-        <kd value="${kd_val}" />
-        <maxVel value="${maxVel_val}"/>
-        <dampingFactor value="${dampigFactor_val}"/>
-        <selfCollide>${selfCollide_val}</selfCollide>
+        <xacro:if value="$(arg use_gazebo_link_physics_coefficients)">
+          <mu1 value="${mu1_val}"/>
+          <mu2 value="${mu2_val}"/>
+          <kp value="${kp_val}" />
+          <kd value="${kd_val}" />
+          <maxVel value="${maxVel_val}"/>
+          <dampingFactor value="${dampigFactor_val}"/>
+          <selfCollide>${selfCollide_val}</selfCollide>
+        </xacro:if>
     </gazebo>
 </robot>

File: description/RobotElements/RightLegElems/Rfoot.xacro (robot description, xacro)
@@ -6,7 +6,8 @@
         <child link="Right_Foot"/>
         <axis xyz="1.0 0 0"/>
-        <limit lower="${-pi/2}" upper="${pi/2}" effort="1" velocity="1"/>
-        <dynamics damping="0.7" friction="0.5"/>
-        <dynamics damping="${damping_val}" friction="${friction_val}"/>
+        <limit lower="${-pi/2}" upper="${pi/2}" effort="${maxeffort_val}" velocity="${maxVel_val}"/>
+        <xacro:if value="$(arg use_URDF_joint_dynamics_coefficients)">
+            <dynamics damping="${damping_val}" friction="${friction_val}"/>
+        </xacro:if>
     </joint>
     <link name="Right_Foot">
@@ -30,4 +31,5 @@
         </inertial>
     </link>
+    <xacro:if value="$(arg use_gazebo_joint_physics_coefficients)">
     <gazebo reference="RFx">
         <implicitSpringDamper>${Damper_val}</implicitSpringDamper>
@@ -37,13 +39,16 @@
         <stopCfm>${stopCfm_val}</stopCfm>
     </gazebo>
+    </xacro:if>
     <gazebo reference="Right_Foot">
         <material>Gazebo/Grey</material>
-        <mu1 value="${mu1_val}"/>
-        <mu2 value="${mu2_val}"/>
-        <kp value="${kp_val}" />
-        <kd value="${kd_val}" />
-        <maxVel value="${maxVel_val}"/>
-        <dampingFactor value="${dampigFactor_val}"/>
-        <selfCollide>${selfCollide_val}</selfCollide>
+        <xacro:if value="$(arg use_gazebo_link_physics_coefficients)">
+          <mu1 value="${mu1_val}"/>
+          <mu2 value="${mu2_val}"/>
+          <kp value="${kp_val}" />
+          <kd value="${kd_val}" />
+          <maxVel value="${maxVel_val}"/>
+          <dampingFactor value="${dampigFactor_val}"/>
+          <selfCollide>${selfCollide_val}</selfCollide>
+        </xacro:if>
     </gazebo>
 </robot>

File: description/RobotElements/RightLegElems/Rhip.xacro (robot description, xacro)
@@ -6,5 +6,8 @@
         <child link="Right_Hip"/>
         <axis xyz="1.0 0 0"/>
-        <limit lower="${-pi/2}" upper="${pi/2}" effort="1" velocity="1"/>
+        <limit lower="${-pi/2}" upper="${pi/2}" effort="${maxeffort_val}" velocity="${maxVel_val}"/>
+        <xacro:if value="$(arg use_URDF_joint_dynamics_coefficients)">
+            <dynamics damping="${damping_val}" friction="${friction_val}"/>
+        </xacro:if>
     </joint>
     <link name="Right_Hip">
@@ -28,4 +31,5 @@
         </inertial>
     </link>
+    <xacro:if value="$(arg use_gazebo_joint_physics_coefficients)">
     <gazebo reference="RTx">
         <implicitSpringDamper>${Damper_val}</implicitSpringDamper>
@@ -35,13 +39,16 @@
         <stopCfm>${stopCfm_val}</stopCfm>
     </gazebo>
+    </xacro:if>
     <gazebo reference="Right_Hip">
         <material>Gazebo/Grey</material>
-        <mu1 value="${mu1_val}"/>
-        <mu2 value="${mu2_val}"/>
-        <kp value="${kp_val}" />
-        <kd value="${kd_val}" />
-        <maxVel value="${maxVel_val}"/>
-        <dampingFactor value="${dampigFactor_val}"/>
-        <selfCollide>${selfCollide_val}</selfCollide>
+        <xacro:if value="$(arg use_gazebo_link_physics_coefficients)">
+          <mu1 value="${mu1_val}"/>
+          <mu2 value="${mu2_val}"/>
+          <kp value="${kp_val}" />
+          <kd value="${kd_val}" />
+          <maxVel value="${maxVel_val}"/>
+          <dampingFactor value="${dampigFactor_val}"/>
+          <selfCollide>${selfCollide_val}</selfCollide>
+        </xacro:if>
     </gazebo>
 </robot>

File: description/RobotElements/RightLegElems/Rhipmount.xacro (robot description, xacro)
@@ -6,5 +6,8 @@
         <child link="Right_HipMount"/>
         <axis xyz="0 0 1.0"/>
-        <limit lower="${-pi/2}" upper="${pi/2}" effort="1" velocity="1"/>
+        <limit lower="${-pi/2}" upper="${pi/2}" effort="${maxeffort_val}" velocity="${maxVel_val}"/>
+        <xacro:if value="$(arg use_URDF_joint_dynamics_coefficients)">
+            <dynamics damping="${damping_val}" friction="${friction_val}"/>
+        </xacro:if>
     </joint>
     <link name="Right_HipMount">
@@ -28,4 +31,5 @@
         </inertial>
     </link>
+    <xacro:if value="$(arg use_gazebo_joint_physics_coefficients)">
     <gazebo reference="RTz">
         <implicitSpringDamper>${Damper_val}</implicitSpringDamper>
@@ -35,13 +39,16 @@
         <stopCfm>${stopCfm_val}</stopCfm>
     </gazebo>
+    </xacro:if>
     <gazebo reference="Right_HipMount">
         <material>Gazebo/Grey</material>
-        <mu1 value="${mu1_val}"/>
-        <mu2 value="${mu2_val}"/>
-        <kp value="${kp_val}" />
-        <kd value="${kd_val}" />
-        <maxVel value="${maxVel_val}"/>
-        <dampingFactor value="${dampigFactor_val}"/>
-        <selfCollide>${selfCollide_val}</selfCollide>
+        <xacro:if value="$(arg use_gazebo_link_physics_coefficients)">
+          <mu1 value="${mu1_val}"/>
+          <mu2 value="${mu2_val}"/>
+          <kp value="${kp_val}" />
+          <kd value="${kd_val}" />
+          <maxVel value="${maxVel_val}"/>
+          <dampingFactor value="${dampigFactor_val}"/>
+          <selfCollide>${selfCollide_val}</selfCollide>
+        </xacro:if>
     </gazebo>
 </robot>

File: description/RobotElements/RightLegElems/Rshank.xacro (robot description, xacro)
@@ -6,5 +6,8 @@
       <child link="Right_Shank"/>
       <axis xyz="0 1.0 0"/>
-      <limit lower="${-pi/2}" upper="${pi/2}" effort="1" velocity="1"/>
+        <limit lower="${-pi/2}" upper="${pi/2}" effort="${maxeffort_val}" velocity="${maxVel_val}"/>
+        <xacro:if value="$(arg use_URDF_joint_dynamics_coefficients)">
+            <dynamics damping="${damping_val}" friction="${friction_val}"/>
+        </xacro:if>
     </joint>
     <link name="Right_Shank">
@@ -28,4 +31,5 @@
         </inertial>
     </link>
+    <xacro:if value="$(arg use_gazebo_joint_physics_coefficients)">
     <gazebo reference="RSy">
         <implicitSpringDamper>${Damper_val}</implicitSpringDamper>
@@ -35,13 +39,16 @@
         <stopCfm>${stopCfm_val}</stopCfm>
     </gazebo>
+    </xacro:if>
     <gazebo reference="Right_Shank">
         <material>Gazebo/Grey</material>
-        <mu1 value="${mu1_val}"/>
-        <mu2 value="${mu2_val}"/>
-        <kp value="${kp_val}" />
-        <kd value="${kd_val}" />
-        <maxVel value="${maxVel_val}"/>
-        <dampingFactor value="${dampigFactor_val}"/>
-        <selfCollide>${selfCollide_val}</selfCollide>
+        <xacro:if value="$(arg use_gazebo_link_physics_coefficients)">
+          <mu1 value="${mu1_val}"/>
+          <mu2 value="${mu2_val}"/>
+          <kp value="${kp_val}" />
+          <kd value="${kd_val}" />
+          <maxVel value="${maxVel_val}"/>
+          <dampingFactor value="${dampigFactor_val}"/>
+          <selfCollide>${selfCollide_val}</selfCollide>
+        </xacro:if>
     </gazebo>
  </robot>

File: description/RobotElements/RightLegElems/Rthigh.xacro (robot description, xacro)
@@ -6,5 +6,8 @@
       <child link="Right_Thigh"/>
       <axis xyz="0 1.0 0"/>
-      <limit lower="${-pi/2}" upper="${pi/2}" effort="1" velocity="1"/>
+        <limit lower="${-pi/2}" upper="${pi/2}" effort="${maxeffort_val}" velocity="${maxVel_val}"/>
+        <xacro:if value="$(arg use_URDF_joint_dynamics_coefficients)">
+            <dynamics damping="${damping_val}" friction="${friction_val}"/>
+        </xacro:if>
     </joint>
     <link name="Right_Thigh">
@@ -28,4 +31,5 @@
         </inertial>
     </link>
+    <xacro:if value="$(arg use_gazebo_joint_physics_coefficients)">
     <gazebo reference="RTy">
         <implicitSpringDamper>${Damper_val}</implicitSpringDamper>
@@ -35,13 +39,16 @@
         <stopCfm>${stopCfm_val}</stopCfm>
     </gazebo>
+    </xacro:if>
     <gazebo reference="Right_Thigh">
         <material>Gazebo/Grey</material>
-        <mu1 value="${mu1_val}"/>
-        <mu2 value="${mu2_val}"/>
-        <kp value="${kp_val}" />
-        <kd value="${kd_val}" />
-        <maxVel value="${maxVel_val}"/>
-        <dampingFactor value="${dampigFactor_val}"/>
-        <selfCollide>${selfCollide_val}</selfCollide>
+        <xacro:if value="$(arg use_gazebo_link_physics_coefficients)">
+          <mu1 value="${mu1_val}"/>
+          <mu2 value="${mu2_val}"/>
+          <kp value="${kp_val}" />
+          <kd value="${kd_val}" />
+          <maxVel value="${maxVel_val}"/>
+          <dampingFactor value="${dampigFactor_val}"/>
+          <selfCollide>${selfCollide_val}</selfCollide>
+        </xacro:if>
     </gazebo>
 </robot>

Commit message: Thrown out the links that are not on the real robot and mount those which are in reality

File: description/RobotElements/HeadElems/Head.xacro (robot description, xacro)
@@ -13,7 +13,7 @@
     <link name="Head">
         <visual>
-            <origin xyz="0 0 0" rpy="0 0 0"/>
+            <origin xyz="0 0 0" rpy="-${pi/2} 0 0"/>
             <geometry>
-                <mesh filename="file://$(find ros2_humanoid_virtual_twin)/meshes/Head.stl"/>
+                <mesh filename="file://$(find ros2_humanoid_virtual_twin)/meshes/Head.stl" scale="0.001 0.001 0.001"/>
             </geometry>
             <material name="grey"/>
@@ -26,7 +26,7 @@
         </collision>
         <inertial>
-            <origin xyz="3.387e-3 0.317e-3 11.04e-3" rpy="0 0 0"/>
-            <mass value="0.092"/>
-            <inertia ixx="31.574e-6" iyy="28.238e-6" izz="23.684e-6" ixy="-0.065e-6" ixz="0.362e-6"  iyz="0.693e-6"/>
+            <origin xyz="-0.03e-3 -12.752e-3 1.006e-3" rpy="0 0 0"/>
+            <mass value="0.055"/>
+            <inertia ixx="15.916e-6" iyy="8.790e-6" izz="13.393e-6" ixy="-0.014e-6" ixz="0.002e-6"  iyz="-0.145e-6"/>
         </inertial>
     </link>

File: description/RobotElements/HeadElems/Headmount.xacro (robot description, xacro)
@@ -2,5 +2,5 @@
 <robot xmlns:xacro="http://www.ros.org/wiki/xacro">
     <joint name="Hz" type="revolute">
-        <origin xyz="18.061e-3 0.134e-3 42.5e-3" rpy="0 0 0"/>
+        <origin xyz="18.1e-3 -0.159e-3 38.5e-3" rpy="0 0 0"/>
         <parent link="Trunk"/>
         <child link="Head_Mounting"/>
@@ -15,5 +15,5 @@
             <origin xyz="0 0 0" rpy="0 0 0"/>
             <geometry>
-                <mesh filename="file://$(find ros2_humanoid_virtual_twin)/meshes/HeadMounting.stl"/>
+                <mesh filename="file://$(find ros2_humanoid_virtual_twin)/meshes/HeadMounting.stl" scale="0.001 0.001 0.001"/>
             </geometry>
             <material name="grey"/>
@@ -26,7 +26,7 @@
         </collision>
         <inertial>
-            <origin xyz="0 -3.335e-3 -17.703e-3" rpy="0 0 0"/>
-            <mass value="0.011"/>
-            <inertia ixx="4.859e-6" iyy="2.246e-6" izz="3.894e-6" ixy="0" ixz="0"  iyz="0.637e-6"/>
+            <origin xyz="-0.031e-3 1.68e-3 -12.625e-3" rpy="0 0 0"/>
+            <mass value="0.009"/>
+            <inertia ixx="4.189e-6" iyy="1.569e-6" izz="3.565e-6" ixy="0.005e-6" ixz="0.002e-6"  iyz="-0.185e-6"/>
         </inertial>
     </link>

File: description/RobotElements/head.xacro (robot description, xacro)
@@ -3,3 +3,4 @@
   <xacro:include filename="HeadElems/Headmount.xacro"/>
   <xacro:include filename="HeadElems/Head.xacro"/>
+  <xacro:include filename="HeadElems/camera.xacro"/>
 </robot>

File: description/RobotElements/left_arm.xacro (robot description, xacro)
@@ -3,4 +3,4 @@
   <xacro:include filename="LeftArmElems/Larmmount.xacro"/>
   <xacro:include filename="LeftArmElems/Larm.xacro"/>
-  <xacro:include filename="LeftArmElems/Lforearm.xacro"/>
+  <!-- <xacro:include filename="LeftArmElems/Lforearm.xacro"/> -->
 </robot>

File: description/RobotElements/right_arm.xacro (robot description, xacro)
@@ -3,4 +3,4 @@
   <xacro:include filename="RightArmElems/Rarmmount.xacro"/>
   <xacro:include filename="RightArmElems/Rarm.xacro"/>
-  <xacro:include filename="RightArmElems/Rforearm.xacro"/>
+  <!-- <xacro:include filename="RightArmElems/Rforearm.xacro"/> -->
 </robot>
