Commit message: usunieto bledy zwiazane z brakiem ladowania pliku.stl kolizji lewego uda, oraz dodano komentarze w j.ang

File: description/robot.urdf.xacro (robot description, xacro)
@@ -1,6 +1,6 @@
 <?xml version="1.0"?>
 <robot xmlns:xacro="http://www.ros.org/wiki/xacro"  name="Melman">
-    <!-- Ponizej plik inicjujacy geometrie robota oraz parametry masowo bezwladnosciowe -->
+    <!-- Below is a file which initiates geometry of robot and inertial, dynamic, collision parameters -->
     <xacro:include filename="robot_core.xacro" />
-    <!-- Ponizej znajda sie parametry dotyczace kontroli ruchow Melmana -->
+    <!-- Below is a file which contains parameters controlling movements of a robot -->
 </robot>

File: description/robot_core.xacro (robot description, xacro)
@@ -1,21 +1,22 @@
 <?xml version="1.0"?>
 <robot xmlns:xacro="http://www.ros.org/wiki/xacro" >
-  <!-- Zdefiniowanie czarnego materialu -->
+  <!-- Definition of grey material-->
   <material name="grey">
       <color rgba="0.6 0.6 0.6 1"/>
   </material>
-  <!-- BASE LINK zrobi spawna w 0 0 0-->
+  <!-- BASE LINK spawns in x0 y0 z0-->
   <link name="base_link">
   </link>
-  <!-- KORPUS -->
+  <!-- <xacro:include filename="RobotElements/Trunk.xacro"/> -->
+   <!-- TRUNK -->
   <joint name="Trunk_joint" type="fixed">
       <parent link="base_link"/>
       <child link="Trunk"/>
-      <!--Origin definiuje przesuniecie ukladu child wzgledem ukladu parent w ukladzie parent-->
+      <!--Origin defines translation child frame relative to parent frame. Translation is performed in parent frame.-->
       <origin xyz="0 0 0.5" rpy="0 0 0"/>
   </joint>
   <link name="Trunk">
     <visual>
-		  <!--Origin definiuje jak srodek geometryczny obiektu ma sie znajdowac wzgledem child frame-->
+		  <!--Origin defines geometric center of spawnego object relative to child frame-->
       <origin xyz="0 0 0" rpy="0 0 0"/>
       <geometry>
@@ -30,8 +31,8 @@
     </inertial>
     <collision>
-      <origin xyz="0 0 0" rpy="0 0 0"/>
       <geometry>
         <mesh filename="package://ros2_humanoid_virtual_twin/STLe/Trunk-Collision.stl"/>
       </geometry>
+      <origin xyz="0 0 0" rpy="0 0 0"/>
     </collision>
   </link>
@@ -39,7 +40,7 @@
       <material>Gazebo/Black</material>
   </gazebo>
-  <!-- LEWA NOGA -->
+  <!-- LEFT FOOT -->
   <joint name="LTz" type="revolute">
-		<!--Origin definiuje przesuniecie ukladu child wzgledem ukladu parent w ukladzie parent-->
+    <!--Origin defines translation child frame relative to parent frame. Translation is performed in parent frame.-->
     <origin xyz="0	40e-3	-150.065e-3" rpy="0 0 0"/>
     <parent link="Trunk"/>
@@ -59,5 +60,5 @@
       <origin xyz="0 0 0" rpy="0 0 0"/>
       <geometry>
-        <mesh filename="package://ros2_humanoid_virtual_twin/Left_HipMount_collision"/>
+        <mesh filename="package://ros2_humanoid_virtual_twin/STLe/Rgiht-HipMount-Collision.stl"/>
       </geometry>
     </collision>

Commit message: Added ros2control

File: description/robot.urdf.xacro (robot description, xacro)
@@ -4,9 +4,10 @@
     <xacro:include filename="robot_core.xacro" />
     <!-- If you want the Trunk to be immovable and static at a certain height uncomment lines below -->
-    <!-- <link name="world"/>
+    <link name="world"/>
     <joint name="world-base_link-fixed" type="fixed">
         <parent link="world"/>
         <child link="base_link"/>
-    </joint> -->
+    </joint>
     <!-- Below is a file which contains parameters controlling movements of a robot -->
+     <xacro:include filename="$(find ros2_humanoid_virtual_twin)/description/Melman_ros2control_gazebo.xacro" />
 </robot>
