Commit message: Humanoid Rviz model with trunk and Left leg

File: description/robot_core.xacro (robot description, xacro)
@@ -8,64 +8,5 @@
   <link name="base_link">
   </link>
-  <!-- <xacro:include filename="RobotElements/Trunk.xacro"/> -->
-   <!-- TRUNK -->
-  <joint name="Trunk_joint" type="fixed">
-      <parent link="base_link"/>
-      <child link="Trunk"/>
-      <!--Origin defines translation child frame relative to parent frame. Translation is performed in parent frame.-->
-      <origin xyz="0 0 0.5" rpy="0 0 0"/>
-  </joint>
-  <link name="Trunk">
-    <visual>
-		  <!--Origin defines geometric center of spawnego object relative to child frame-->
-      <origin xyz="0 0 0" rpy="0 0 0"/>
-      <geometry>
-        <mesh filename="package://ros2_humanoid_virtual_twin/STLe/Trunk.stl"/>
-      </geometry>
-      <material name="grey"/>
-    </visual>
-    <inertial>
-      <origin xyz="-7.709e-3	-0.06e-3	-57.629e-3" rpy="0 0 0"/>
-      <mass value="0.691"/>
-      <inertia ixx="1992.6e-6" iyy="1287.385e-6" izz="1142.314e-6" ixy="0.546e-6" ixz="-217.49e-6"  iyz="1.946e-6" />
-    </inertial>
-    <collision>
-      <geometry>
-        <mesh filename="package://ros2_humanoid_virtual_twin/STLe/Trunk-Collision.stl"/>
-      </geometry>
-      <origin xyz="0 0 0" rpy="0 0 0"/>
-    </collision>
-  </link>
-  <gazebo reference="Trunk">
-      <material>Gazebo/Black</material>
-  </gazebo>
-  <!-- LEFT FOOT -->
-  <joint name="LTz" type="revolute">
-    <!--Origin defines translation child frame relative to parent frame. Translation is performed in parent frame.-->
-    <origin xyz="0	40e-3	-150.065e-3" rpy="0 0 0"/>
-    <parent link="Trunk"/>
-    <child link="Left_HipMount"/>
-    <axis xyz="0 0 1.0"/>
-    <limit lower="${-pi}" upper="${pi}" effort="100" velocity="100"/>
-  </joint>
-  <link name="Left_HipMount">
-    <visual>
-      <origin xyz="0 0 0" rpy="0 0 0"/>
-      <geometry>
-        <mesh filename="package://ros2_humanoid_virtual_twin/STLe/Left-HipMount.stl"/>
-      </geometry>
-      <material name="grey"/>
-    </visual>
-    <collision>
-      <origin xyz="0 0 0" rpy="0 0 0"/>
-      <geometry>
-        <mesh filename="package://ros2_humanoid_virtual_twin/STLe/Rgiht-HipMount-Collision.stl"/>
-      </geometry>
-    </collision>
-    <inertial>
-      <origin xyz="-14.306e-3	0	24.769e-3" rpy="0 0 0"/>
-      <mass value="0.038"/>
-      <inertia ixx="11.743e-6" iyy="61.298e-6" izz="58.734e-6" ixy="0" ixz="4.429e-6"  iyz="0" />
-    </inertial>
-  </link>
+  <xacro:include filename="RobotElements/Trunk.xacro"/>
+  <xacro:include filename="RobotElements/left_leg.xacro"/>
 </robot>

Commit message: Gained control over the effort controller. Terminal command to control joints pasted in control_txt_files

File: description/robot_core.xacro (robot description, xacro)
@@ -18,6 +18,6 @@
   <xacro:property name="damping_val" value="1.0"/>
   <xacro:property name="friction_val" value="1.0"/>
-  <xacro:property name="maxVel_val" value="0.0"/>
-  <xacro:property name="maxeffort_val" value="0.0"/>
+  <xacro:property name="maxVel_val" value="5.1"/>
+  <xacro:property name="maxeffort_val" value="5.1"/>
   <!-- Definition of grey material-->
   <material name="grey">
