Commit message: Selected kp, kd, mu1, mu2 coefficients for the robot not to explode in the air

File: description/Melman_ros2control_gazebo.xacro (robot description, xacro)
@@ -10,7 +10,5 @@
             <command_interface name="velocity"/>
             <state_interface name="position"/>
-                <param name="initial_value">0.0</param>
             <state_interface name="velocity"/>
-            <state_interface name="effort"/>
         </joint>
         <!-- Right Thigh X axis rotation control-->
@@ -19,7 +17,5 @@
             <command_interface name="velocity"/>
             <state_interface name="position"/>
-                <param name="initial_value">0.0</param>
             <state_interface name="velocity"/>
-            <state_interface name="effort"/>
         </joint>
         <!-- Right Thigh Y axis rotation control-->
@@ -28,7 +24,5 @@
             <command_interface name="velocity"/>
             <state_interface name="position"/>
-                <param name="initial_value">0.0</param>
             <state_interface name="velocity"/>
-            <state_interface name="effort"/>
         </joint>
         <!-- Right shank Y axis rotation control-->
@@ -37,7 +31,5 @@
             <command_interface name="velocity"/>
             <state_interface name="position"/>
-                <param name="initial_value">0.0</param>
             <state_interface name="velocity"/>
-            <state_interface name="effort"/>
         </joint>
         <!--Right foot Y axis rotation control -->
@@ -46,7 +38,5 @@
             <command_interface name="velocity"/>
             <state_interface name="position"/>
-                <param name="initial_value">0.0</param>
             <state_interface name="velocity"/>
-            <state_interface name="effort"/>
         </joint>
         <!-- Right foot X axis rotation control-->
@@ -55,7 +45,5 @@
             <command_interface name="velocity"/>
             <state_interface name="position"/>
-                <param name="initial_value">0.0</param>
             <state_interface name="velocity"/>
-            <state_interface name="effort"/>
         </joint>
         <!-- Left thigh z axis rotation control-->
@@ -64,7 +52,5 @@
             <command_interface name="velocity"/>
             <state_interface name="position"/>
-                <param name="initial_value">0.0</param>
             <state_interface name="velocity"/>
-            <state_interface name="effort"/>
         </joint>
         <!--Left thigh x axis rotation control -->
@@ -73,7 +59,5 @@
             <command_interface name="velocity"/>
             <state_interface name="position"/>
-                <param name="initial_value">0.0</param>
             <state_interface name="velocity"/>
-            <state_interface name="effort"/>
         </joint>
         <!-- Left thigh y axis rotation control-->
@@ -82,7 +66,5 @@
             <command_interface name="velocity"/>
             <state_interface name="position"/>
-                <param name="initial_value">0.0</param>
             <state_interface name="velocity"/>
-            <state_interface name="effort"/>
         </joint>
         <!-- Left shank y axis rotation control-->
@@ -91,7 +73,5 @@
             <command_interface name="velocity"/>
             <state_interface name="position"/>
-                <param name="initial_value">0.0</param>
             <state_interface name="velocity"/>
-            <state_interface name="effort"/>
         </joint>
         <!-- Left foot y axis rotation control-->
@@ -100,7 +80,5 @@
             <command_interface name="velocity"/>
             <state_interface name="position"/>
-                <param name="initial_value">0.0</param>
             <state_interface name="velocity"/>
-            <state_interface name="effort"/>
         </joint>
         <!--Left foot x axis rotation control -->
@@ -109,7 +87,5 @@
             <command_interface name="velocity"/>
             <state_interface name="position"/>
-                <param name="initial_value">0.0</param>
             <state_interface name="velocity"/>
-            <state_interface name="effort"/>
         </joint>
         <!-- Right arm y axis rotation control -->
@@ -118,7 +94,5 @@
             <command_interface name="velocity"/>
             <state_interface name="position"/>
-                <param name="initial_value">0.0</param>
             <state_interface name="velocity"/>
-            <state_interface name="effort"/>
         </joint>
         <!-- Right arm x axis rotation control-->
@@ -127,7 +101,5 @@
             <command_interface name="velocity"/>
             <state_interface name="position"/>
-                <param name="initial_value">0.0</param>
             <state_interface name="velocity"/>
-            <state_interface name="effort"/>
         </joint>
         <!-- Roght forearm y axis rotation control-->
@@ -136,7 +108,5 @@
             <command_interface name="velocity"/>
             <state_interface name="position"/>
-                <param name="initial_value">0.0</param>
             <state_interface name="velocity"/>
-            <state_interface name="effort"/>
         </joint>
         <!--Left arm y axis rotation control -->
@@ -145,7 +115,5 @@
             <command_interface name="velocity"/>
             <state_interface name="position"/>
-                <param name="initial_value">0.0</param>
             <state_interface name="velocity"/>
-            <state_interface name="effort"/>
         </joint>
         <!-- Left arm x axis rotation control -->
@@ -154,7 +122,5 @@
             <command_interface name="velocity"/>
             <state_interface name="position"/>
-                <param name="initial_value">0.0</param>
             <state_interface name="velocity"/>
-            <state_interface name="effort"/>
         </joint>
         <!-- Left forearm y axis rotation control -->
@@ -165,5 +131,4 @@
               <param name="initial_value">0.0</param>
             <state_interface name="velocity"/>
-            <state_interface name="effort"/>
         </joint>
         <!-- Head z axis rotation control-->
@@ -172,7 +137,5 @@
             <command_interface name="velocity"/>
             <state_interface name="position"/>
-                <param name="initial_value">0.0</param>
             <state_interface name="velocity"/>
-            <state_interface name="effort"/>
         </joint>
         <!-- Head y axis rotation control-->
@@ -181,7 +144,5 @@
             <command_interface name="velocity"/>
             <state_interface name="position"/>
-                <param name="initial_value">0.0</param>
             <state_interface name="velocity"/>
-            <state_interface name="effort"/>
         </joint>
     </ros2_control>

File: description/RobotElements/LeftArmElems/Larm.xacro (robot description, xacro)
@@ -19,5 +19,5 @@
             <origin xyz="0 0 0" rpy="0 0 0"/>
             <geometry>
-                <mesh filename="file://$(find ros2_humanoid_virtual_twin)/meshes/Left-Arm-Collision.stl"/>
+                <mesh filename="file://$(find ros2_humanoid_virtual_twin)/meshes/Left-Arm_Collision.stl" scale="0.001 0.001 0.001"/>
             </geometry>
         </collision>

File: description/RobotElements/LeftLegElems/Lfoot.xacro (robot description, xacro)
@@ -20,5 +20,5 @@
         <origin xyz="0 0 0" rpy="0 0 0"/>
         <geometry>
-			<mesh filename="file://$(find ros2_humanoid_virtual_twin)/meshes/Left-Foot-collision.stl"/>
+			    <mesh filename="file://$(find ros2_humanoid_virtual_twin)/meshes/Left-Foot-collision.stl"/>
         </geometry>
       </collision>
@@ -31,11 +31,7 @@
     <gazebo reference="Left_Foot">
       <material>Gazebo/Grey</material>
-      <mu1 value="200.0"/>
-      <mu2 value="100.0"/>
-      <kp value="10000000.0" />
-      <kd value="1.0" />
-      <selfCollide>true</selfCollide>
-      <dampingFactor>15.0</dampingFactor>
-      <maxVel>0.5</maxVel>
+      <mu1 value="0.002"/>
+      <mu2 value="0.003"/>
+      <kp value="100000.0"/>
     </gazebo>
 </robot>

File: description/RobotElements/RightArmElems/Rarm.xacro (robot description, xacro)
@@ -12,5 +12,5 @@
             <origin xyz="0 0 0" rpy="0 0 0"/>
             <geometry>
-                <mesh filename="file://$(find ros2_humanoid_virtual_twin)/meshes/Left-Arm.stl" scale="0.001 0.001 0.001"/>
+                <mesh filename="file://$(find ros2_humanoid_virtual_twin)/meshes/Right-Arm.stl" scale="0.001 0.001 0.001"/>
             </geometry>
             <material name="grey"/>
@@ -19,5 +19,5 @@
             <origin xyz="0 0 0" rpy="0 0 0"/>
             <geometry>
-                <mesh filename="file://$(find ros2_humanoid_virtual_twin)/meshes/Left-Arm-Collision.stl"/>
+                <mesh filename="file://$(find ros2_humanoid_virtual_twin)/meshes/Right-Arm_Collision.stl" scale="0.001 0.001 0.001"/>
             </geometry>
         </collision>

File: description/RobotElements/RightLegElems/Rfoot.xacro (robot description, xacro)
@@ -30,11 +30,7 @@
     <gazebo reference="Right_Foot">
         <material>Gazebo/Grey</material>
-        <mu1 value="200.0"/>
-        <mu2 value="100.0"/>
-        <kp value="10000000.0" />
-        <kd value="1.0" />
-        <selfCollide>true</selfCollide>
-        <dampingFactor>15.0</dampingFactor>
-        <maxVel>0.5</maxVel>
+        <mu1 value="0.002"/>
+        <mu2 value="0.003"/>
+        <kp value="100000.0"/>
     </gazebo>
 </robot>

File: description/RobotElements/Trunk.xacro (robot description, xacro)
@@ -6,5 +6,5 @@
       <child link="Trunk"/>
       <!--Origin defines translation child frame relative to parent frame. Translation is performed in parent frame.-->
-      <origin xyz="0 0 0.45" rpy="0 0 0"/>
+      <origin xyz="0 0 0.443" rpy="0 0 0"/>
   </joint>
   <link name="Trunk">
@@ -31,9 +31,7 @@
   <gazebo reference="Trunk">
       <material>Gazebo/Grey</material>
-      <must_be_base_link>true</must_be_base_link>
       <mu1 value="200.0"/>
       <mu2 value="100.0"/>
-      <kp value="10000000.0" />
-      <kd value="1.0" />
+      <kp value="100000.0" />
       <selfCollide>true</selfCollide>
   </gazebo>

File: description/robot.urdf.xacro (robot description, xacro)
@@ -4,9 +4,9 @@
     <xacro:include filename="robot_core.xacro" />
     <!-- If you want the Trunk to be immovable and static at a certain height uncomment lines below -->
-    <link name="world"/>
+    <!-- <link name="world"/>
     <joint name="world-base_link-fixed" type="fixed">
         <parent link="world"/>
         <child link="base_link"/>
-    </joint>
+    </joint> -->
     <!-- Below is a file which contains parameters controlling movements of a robot -->
     <xacro:include filename="$(find ros2_humanoid_virtual_twin)/description/Melman_ros2control_gazebo.xacro" />
