Commit message: Added xacro parameters for links to tune their joint and contact physical properties. Robot flies in the air unfortunately

File: description/Melman_ros2control_gazebo.xacro (robot description, xacro)
@@ -7,6 +7,12 @@
         <!-- Right Thigh Z axis rotation control -->
         <joint name="RTz">
-            <command_interface name="position"/>
-            <command_interface name="velocity"/>
+            <command_interface name="position">
+                <param name="min">${-pi/2}</param>
+                <param name="max">${pi/2}</param>
+            </command_interface>
+            <command_interface name="velocity">
+                <param name="min">-5.0</param>
+                <param name="max">5.0</param>
+            </command_interface>
             <state_interface name="position"/>
             <state_interface name="velocity"/>
@@ -14,6 +20,12 @@
         <!-- Right Thigh X axis rotation control-->
         <joint name="RTx">
-            <command_interface name="position"/>
-            <command_interface name="velocity"/>
+            <command_interface name="position">
+                <param name="min">${-pi/2}</param>
+                <param name="max">${pi/2}</param>
+            </command_interface>
+            <command_interface name="velocity">
+                <param name="min">-5.0</param>
+                <param name="max">5.0</param>
+            </command_interface>
             <state_interface name="position"/>
             <state_interface name="velocity"/>
@@ -21,13 +33,27 @@
         <!-- Right Thigh Y axis rotation control-->
         <joint name="RTy">
-            <command_interface name="position"/>
-            <command_interface name="velocity"/>
-            <state_interface name="position"/>
+            <command_interface name="position">
+                <param name="min">${-pi/2}</param>
+                <param name="max">${pi/2}</param>
+            </command_interface>
+            <command_interface name="velocity">
+                <param name="min">-5.0</param>
+                <param name="max">5.0</param>
+            </command_interface>
+            <state_interface name="position">
+                <!-- <param name="initial_value">-0.1</param> -->
+            </state_interface>
             <state_interface name="velocity"/>
         </joint>
         <!-- Right shank Y axis rotation control-->
         <joint name="RSy">
-            <command_interface name="position"/>
-            <command_interface name="velocity"/>
+            <command_interface name="position">
+                <param name="min">${-pi/2}</param>
+                <param name="max">${pi/2}</param>
+            </command_interface>
+            <command_interface name="velocity">
+                <param name="min">-5.0</param>
+                <param name="max">5.0</param>
+            </command_interface>
             <state_interface name="position"/>
             <state_interface name="velocity"/>
@@ -35,6 +61,12 @@
         <!--Right foot Y axis rotation control -->
         <joint name="RFy">
-            <command_interface name="position"/>
-            <command_interface name="velocity"/>
+            <command_interface name="position">
+                <param name="min">${-pi/2}</param>
+                <param name="max">${pi/2}</param>
+            </command_interface>
+            <command_interface name="velocity">
+                <param name="min">-5.0</param>
+                <param name="max">5.0</param>
+            </command_interface>
             <state_interface name="position"/>
             <state_interface name="velocity"/>
@@ -42,6 +74,12 @@
         <!-- Right foot X axis rotation control-->
         <joint name="RFx">
-            <command_interface name="position"/>
-            <command_interface name="velocity"/>
+            <command_interface name="position">
+                <param name="min">${-pi/2}</param>
+                <param name="max">${pi/2}</param>
+            </command_interface>
+            <command_interface name="velocity">
+                <param name="min">-5.0</param>
+                <param name="max">5.0</param>
+            </command_interface>
             <state_interface name="position"/>
             <state_interface name="velocity"/>
@@ -49,6 +87,12 @@
         <!-- Left thigh z axis rotation control-->
         <joint name="LTz">
-            <command_interface name="position"/>
-            <command_interface name="velocity"/>
+            <command_interface name="position">
+                <param name="min">${-pi/2}</param>
+                <param name="max">${pi/2}</param>
+            </command_interface>
+            <command_interface name="velocity">
+                <param name="min">-5.0</param>
+                <param name="max">5.0</param>
+            </command_interface>
             <state_interface name="position"/>
             <state_interface name="velocity"/>
@@ -56,6 +100,12 @@
         <!--Left thigh x axis rotation control -->
         <joint name="LTx">
-            <command_interface name="position"/>
-            <command_interface name="velocity"/>
+            <command_interface name="position">
+                <param name="min">${-pi/2}</param>
+                <param name="max">${pi/2}</param>
+            </command_interface>
+            <command_interface name="velocity">
+                <param name="min">-5.0</param>
+                <param name="max">5.0</param>
+            </command_interface>
             <state_interface name="position"/>
             <state_interface name="velocity"/>
@@ -63,13 +113,27 @@
         <!-- Left thigh y axis rotation control-->
         <joint name="LTy">
-            <command_interface name="position"/>
-            <command_interface name="velocity"/>
-            <state_interface name="position"/>
+            <command_interface name="position">
+                <param name="min">${-pi/2}</param>
+                <param name="max">${pi/2}</param>
+            </command_interface>
+            <command_interface name="velocity">
+                <param name="min">-5.0</param>
+                <param name="max">5.0</param>
+            </command_interface>
+            <state_interface name="position">
+                <!-- <param name="initial_value">-0.1</param> -->
+            </state_interface>
             <state_interface name="velocity"/>
         </joint>
         <!-- Left shank y axis rotation control-->
         <joint name="LSy">
-            <command_interface name="position"/>
-            <command_interface name="velocity"/>
+            <command_interface name="position">
+                <param name="min">${-pi/2}</param>
+                <param name="max">${pi/2}</param>
+            </command_interface>
+            <command_interface name="velocity">
+                <param name="min">-5.0</param>
+                <param name="max">5.0</param>
+            </command_interface>
             <state_interface name="position"/>
             <state_interface name="velocity"/>
@@ -77,6 +141,12 @@
         <!-- Left foot y axis rotation control-->
         <joint name="LFy">
-            <command_interface name="position"/>
-            <command_interface name="velocity"/>
+            <command_interface name="position">
+                <param name="min">${-pi/2}</param>
+                <param name="max">${pi/2}</param>
+            </command_interface>
+            <command_interface name="velocity">
+                <param name="min">-5.0</param>
+                <param name="max">5.0</param>
+            </command_interface>
             <state_interface name="position"/>
             <state_interface name="velocity"/>
@@ -84,6 +154,12 @@
         <!--Left foot x axis rotation control -->
         <joint name="LFx">
-            <command_interface name="position"/>
-            <command_interface name="velocity"/>
+            <command_interface name="position">
+                <param name="min">${-pi/2}</param>
+                <param name="max">${pi/2}</param>
+            </command_interface>
+            <command_interface name="velocity">
+                <param name="min">-5.0</param>
+                <param name="max">5.0</param>
+            </command_interface>
             <state_interface name="position"/>
             <state_interface name="velocity"/>
@@ -91,6 +167,12 @@
         <!-- Right arm y axis rotation control -->
         <joint name="RAy">
-            <command_interface name="position"/>
-            <command_interface name="velocity"/>
+            <command_interface name="position">
+                <param name="min">${-pi/2}</param>
+                <param name="max">${pi/2}</param>
+            </command_interface>
+            <command_interface name="velocity">
+                <param name="min">-5.0</param>
+                <param name="max">5.0</param>
+            </command_interface>
             <state_interface name="position"/>
             <state_interface name="velocity"/>
@@ -98,6 +180,12 @@
         <!-- Right arm x axis rotation control-->
         <joint name="RAx">
-            <command_interface name="position"/>
-            <command_interface name="velocity"/>
+            <command_interface name="position">
+                <param name="min">${-pi/2}</param>
+                <param name="max">${pi/2}</param>
+            </command_interface>
+            <command_interface name="velocity">
+                <param name="min">-5.0</param>
+                <param name="max">5.0</param>
+            </command_interface>
             <state_interface name="position"/>
             <state_interface name="velocity"/>
@@ -105,6 +193,12 @@
         <!-- Roght forearm y axis rotation control-->
         <joint name="RFAy">
-            <command_interface name="position"/>
-            <command_interface name="velocity"/>
+            <command_interface name="position">
+                <param name="min">${-pi/2}</param>
+                <param name="max">${pi/2}</param>
+            </command_interface>
+            <command_interface name="velocity">
+                <param name="min">-5.0</param>
+                <param name="max">5.0</param>
+            </command_interface>
             <state_interface name="position"/>
             <state_interface name="velocity"/>
@@ -112,6 +206,12 @@
         <!--Left arm y axis rotation control -->
         <joint name="LAy">
-            <command_interface name="position"/>
-            <command_interface name="velocity"/>
+            <command_interface name="position">
+                <param name="min">${-pi/2}</param>
+                <param name="max">${pi/2}</param>
+            </command_interface>
+            <command_interface name="velocity">
+              <param name="min">-5.0</param>
+                <param name="max">5.0</param>
+            </command_interface>
             <state_interface name="position"/>
             <state_interface name="velocity"/>
@@ -119,6 +219,12 @@
         <!-- Left arm x axis rotation control -->
         <joint name="LAx">
-            <command_interface name="position"/>
-            <command_interface name="velocity"/>
+            <command_interface name="position">
+                <param name="min">${-pi/2}</param>
+                <param name="max">${pi/2}</param>
+            </command_interface>
+            <command_interface name="velocity">
+                <param name="min">-5.0</param>
+                <param name="max">5.0</param>
+            </command_interface>
             <state_interface name="position"/>
             <state_interface name="velocity"/>
@@ -126,14 +232,25 @@
         <!-- Left forearm y axis rotation control -->
         <joint name="LFAy">
-            <command_interface name="position"/>
-            <command_interface name="velocity"/>
-            <state_interface name="position"/>
-              <param name="initial_value">0.0</param>
+            <command_interface name="position">
+                <param name="min">${-pi/2}</param>
+                <param name="max">${pi/2}</param>
+            </command_interface>
+            <command_interface name="velocity">
+                <param name="min">-5.0</param>
+                <param name="max">5.0</param>
+            </command_interface>
+            <state_interface name="position"/>
             <state_interface name="velocity"/>
         </joint>
         <!-- Head z axis rotation control-->
         <joint name="Hz">
-            <command_interface name="position"/>
-            <command_interface name="velocity"/>
+            <command_interface name="position">
+                <param name="min">${-pi/2}</param>
+                <param name="max">${pi/2}</param>
+            </command_interface>
+            <command_interface name="velocity">
+                <param name="min">-5.0</param>
+                <param name="max">5.0</param>
+            </command_interface>
             <state_interface name="position"/>
             <state_interface name="velocity"/>
@@ -141,6 +258,12 @@
         <!-- Head y axis rotation control-->
         <joint name="Hy">
-            <command_interface name="position"/>
-            <command_interface name="velocity"/>
+            <command_interface name="position">
+                <param name="min">${-pi/2}</param>
+                <param name="max">${pi/2}</param>
+            </command_interface>
+            <command_interface name="velocity">
+                <param name="min">-5.0</param>
+                <param name="max">5.0</param>
+            </command_interface>
             <state_interface name="position"/>
             <state_interface name="velocity"/>

File: description/RobotElements/HeadElems/Head.xacro (robot description, xacro)
@@ -6,5 +6,5 @@
         <child link="Head"/>
         <axis xyz="0 1.0 0"/>
-        <limit lower="${-pi/2}" upper="${pi/2}" effort="100" velocity="100"/>
+        <limit lower="${-pi/2}" upper="${pi/2}" effort="1" velocity="1"/>
     </joint>
     <link name="Head">
@@ -28,4 +28,11 @@
         </inertial>
     </link>
+    <gazebo reference="Hy">
+        <implicitSpringDamper>${Damper_val}</implicitSpringDamper>
+        <springStiffness>${springstiffness_val}</springStiffness>
+        <springReference>${springReference_val}</springReference>
+        <stopErp>${stopErp_val}</stopErp>
+        <stopCfm>${stopCfm_val}</stopCfm>
+    </gazebo>
     <gazebo reference="Head">
         <material>Gazebo/Grey</material>
@@ -35,4 +42,5 @@
         <kd value="${kd_val}" />
         <maxVel value="${maxVel_val}"/>
+        <dampingFactor value="${dampigFactor_val}"/>
         <selfCollide>${selfCollide_val}</selfCollide>
     </gazebo>

File: description/RobotElements/HeadElems/Headmount.xacro (robot description, xacro)
@@ -6,5 +6,5 @@
         <child link="Head_Mounting"/>
         <axis xyz="0 0 1.0"/>
-        <limit lower="${-pi/2}" upper="${pi/2}" effort="100" velocity="100"/>
+        <limit lower="${-pi/2}" upper="${pi/2}" effort="1" velocity="1"/>
     </joint>
     <link name="Head_Mounting">
@@ -28,4 +28,11 @@
         </inertial>
     </link>
+    <gazebo reference="Hz">
+        <implicitSpringDamper>${Damper_val}</implicitSpringDamper>
+        <springStiffness>${springstiffness_val}</springStiffness>
+        <springReference>${springReference_val}</springReference>
+        <stopErp>${stopErp_val}</stopErp>
+        <stopCfm>${stopCfm_val}</stopCfm>
+    </gazebo>
     <gazebo reference="Head_Mounting">
         <material>Gazebo/Grey</material>
@@ -35,4 +42,5 @@
         <kd value="${kd_val}" />
         <maxVel value="${maxVel_val}"/>
+        <dampingFactor value="${dampigFactor_val}"/>
         <selfCollide>${selfCollide_val}</selfCollide>
     </gazebo>

File: description/RobotElements/LeftArmElems/Larm.xacro (robot description, xacro)
@@ -6,5 +6,5 @@
         <child link="Left_Arm"/>
         <axis xyz="1.0 0 0"/>
-        <limit lower="${-pi/2}" upper="${pi/2}" effort="100" velocity="100"/>
+        <limit lower="${-pi/2}" upper="${pi/2}" effort="1" velocity="1"/>
     </joint>
     <link name="Left_Arm">
@@ -28,4 +28,11 @@
         </inertial>
     </link>
+    <gazebo reference="LAx">
+        <implicitSpringDamper>${Damper_val}</implicitSpringDamper>
+        <springStiffness>${springstiffness_val}</springStiffness>
+        <springReference>${springReference_val}</springReference>
+        <stopErp>${stopErp_val}</stopErp>
+        <stopCfm>${stopCfm_val}</stopCfm>
+    </gazebo>
     <gazebo reference="Left_Arm">
         <material>Gazebo/Grey</material>
@@ -35,4 +42,5 @@
         <kd value="${kd_val}" />
         <maxVel value="${maxVel_val}"/>
+        <dampingFactor value="${dampigFactor_val}"/>
         <selfCollide>${selfCollide_val}</selfCollide>
     </gazebo>

File: description/RobotElements/LeftArmElems/Larmmount.xacro (robot description, xacro)
@@ -6,5 +6,5 @@
         <child link="Left_ArmMounting"/>
         <axis xyz="0 1.0 0"/>
-        <limit lower="${-pi/2}" upper="${pi/2}" effort="100" velocity="100"/>
+        <limit lower="${-pi/2}" upper="${pi/2}" effort="1" velocity="1"/>
     </joint>
     <link name="Left_ArmMounting">
@@ -28,4 +28,11 @@
         </inertial>
     </link>
+    <gazebo reference="LAy">
+        <implicitSpringDamper>${Damper_val}</implicitSpringDamper>
+        <springStiffness>${springstiffness_val}</springStiffness>
+        <springReference>${springReference_val}</springReference>
+        <stopErp>${stopErp_val}</stopErp>
+        <stopCfm>${stopCfm_val}</stopCfm>
+    </gazebo>
     <gazebo reference="Left_ArmMounting">
         <material>Gazebo/Grey</material>
@@ -35,4 +42,5 @@
         <kd value="${kd_val}" />
         <maxVel value="${maxVel_val}"/>
+        <dampingFactor value="${dampigFactor_val}"/>
         <selfCollide>${selfCollide_val}</selfCollide>
     </gazebo>

File: description/RobotElements/LeftArmElems/Lforearm.xacro (robot description, xacro)
@@ -6,5 +6,5 @@
         <child link="Left_Forearm"/>
         <axis xyz="0 1.0 0"/>
-        <limit lower="${-pi/2}" upper="${pi/2}" effort="100" velocity="100"/>
+        <limit lower="${-pi/2}" upper="${pi/2}" effort="1" velocity="1"/>
     </joint>
     <link name="Left_Forearm">
@@ -28,4 +28,11 @@
         </inertial>
     </link>
+    <gazebo reference="LFAy">
+        <implicitSpringDamper>${Damper_val}</implicitSpringDamper>
+        <springStiffness>${springstiffness_val}</springStiffness>
+        <springReference>${springReference_val}</springReference>
+        <stopErp>${stopErp_val}</stopErp>
+        <stopCfm>${stopCfm_val}</stopCfm>
+    </gazebo>
     <gazebo reference="Left_Forearm">
         <material>Gazebo/Grey</material>
@@ -35,4 +42,5 @@
         <kd value="${kd_val}" />
         <maxVel value="${maxVel_val}"/>
+        <dampingFactor value="${dampigFactor_val}"/>
         <selfCollide>${selfCollide_val}</selfCollide>
     </gazebo>

File: description/RobotElements/LeftLegElems/Lankle.xacro (robot description, xacro)
@@ -6,5 +6,5 @@
       <child link="Left_Ankle"/>
       <axis xyz="0 1.0 0"/>
-      <limit lower="${-pi/2}" upper="${pi/2}" effort="100" velocity="100"/>
+      <limit lower="${-pi/2}" upper="${pi/2}" effort="1" velocity="1"/>
     </joint>
 	<link name="Left_Ankle">
@@ -28,4 +28,11 @@
       </inertial>
     </link>
+    <gazebo reference="LFy">
+        <implicitSpringDamper>${Damper_val}</implicitSpringDamper>
+        <springStiffness>${springstiffness_val}</springStiffness>
+        <springReference>${springReference_val}</springReference>
+        <stopErp>${stopErp_val}</stopErp>
+        <stopCfm>${stopCfm_val}</stopCfm>
+    </gazebo>
     <gazebo reference="Left_Ankle">
         <material>Gazebo/Grey</material>
@@ -35,4 +42,5 @@
         <kd value="${kd_val}" />
         <maxVel value="${maxVel_val}"/>
+        <dampingFactor value="${dampigFactor_val}"/>
         <selfCollide>${selfCollide_val}</selfCollide>
     </gazebo>

File: description/RobotElements/LeftLegElems/Lfoot.xacro (robot description, xacro)
@@ -6,5 +6,6 @@
       <child link="Left_Foot"/>
       <axis xyz="1.0 0 0"/>
-      <limit lower="${-pi/2}" upper="${pi/2}" effort="100" velocity="100"/>
+      <limit lower="${-pi/2}" upper="${pi/2}" effort="1" velocity="1"/>
+      <dynamics damping="${damping_val}" friction="${friction_val}"/>
     </joint>
     <link name="Left_Foot">
@@ -29,11 +30,19 @@
       </inertial>
     </link>
+  <gazebo reference="LFx">
+    <implicitSpringDamper>${Damper_val}</implicitSpringDamper>
+    <springStiffness>${springstiffness_val}</springStiffness>
+    <springReference>${springReference_val}</springReference>
+    <stopErp>${stopErp_val}</stopErp>
+    <stopCfm>${stopCfm_val}</stopCfm>
+  </gazebo>
     <gazebo reference="Left_Foot">
         <material>Gazebo/Grey</material>
-        <mu1 value="0.02"/>
-        <mu2 value="0.03"/>
+        <mu1 value="${mu1_val}"/>
+        <mu2 value="${mu2_val}"/>
         <kp value="${kp_val}" />
         <kd value="${kd_val}" />
         <maxVel value="${maxVel_val}"/>
+        <dampingFactor value="${dampigFactor_val}"/>
         <selfCollide>${selfCollide_val}</selfCollide>
     </gazebo>

File: description/RobotElements/LeftLegElems/Lhip.xacro (robot description, xacro)
@@ -7,5 +7,5 @@
       <child link="Left_Hip"/>
       <axis xyz="1.0 0 0"/>
-      <limit lower="${-pi/2}" upper="${pi/2}" effort="100" velocity="100"/>
+      <limit lower="${-pi/2}" upper="${pi/2}" effort="1" velocity="1"/>
     </joint>
     <link name="Left_Hip">
@@ -29,4 +29,11 @@
       </inertial>
     </link>
+    <gazebo reference="LTx">
+        <implicitSpringDamper>${Damper_val}</implicitSpringDamper>
+        <springStiffness>${springstiffness_val}</springStiffness>
+        <springReference>${springReference_val}</springReference>
+        <stopErp>${stopErp_val}</stopErp>
+        <stopCfm>${stopCfm_val}</stopCfm>
+    </gazebo>
     <gazebo reference="Left_Hip">
         <material>Gazebo/Grey</material>
@@ -36,4 +43,5 @@
         <kd value="${kd_val}" />
         <maxVel value="${maxVel_val}"/>
+        <dampingFactor value="${dampigFactor_val}"/>
         <selfCollide>${selfCollide_val}</selfCollide>
     </gazebo>
