Commit message: Added xacro parameters for links to tune their joint and contact physical properties. Robot flies in the air unfortunately

File: description/RobotElements/LeftLegElems/Lhipmount.xacro (robot description, xacro)
@@ -8,5 +8,5 @@
     <child link="Left_HipMount"/>
     <axis xyz="0 0 1.0"/>
-    <limit lower="${-pi/2}" upper="${pi/2}" effort="100" velocity="100"/>
+    <limit lower="${-pi/2}" upper="${pi/2}" effort="1" velocity="1"/>
   </joint>
   <link name="Left_HipMount">
@@ -30,4 +30,11 @@
     </inertial>
   </link>
+  <gazebo reference="LTz">
+    <implicitSpringDamper>${Damper_val}</implicitSpringDamper>
+    <springStiffness>${springstiffness_val}</springStiffness>
+    <springReference>${springReference_val}</springReference>
+    <stopErp>${stopErp_val}</stopErp>
+    <stopCfm>${stopCfm_val}</stopCfm>
+  </gazebo>
   <gazebo reference="Left_HipMount">
         <material>Gazebo/Grey</material>
@@ -37,4 +44,5 @@
         <kd value="${kd_val}" />
         <maxVel value="${maxVel_val}"/>
+        <dampingFactor value="${dampigFactor_val}"/>
         <selfCollide>${selfCollide_val}</selfCollide>
   </gazebo>

File: description/RobotElements/LeftLegElems/Lshank.xacro (robot description, xacro)
@@ -6,5 +6,5 @@
       <child link="Left_Shank"/>
       <axis xyz="0 1.0 0"/>
-      <limit lower="${-pi/2}" upper="${pi/2}" effort="100" velocity="100"/>
+      <limit lower="${-pi/2}" upper="${pi/2}" effort="1" velocity="1"/>
     </joint>
 	<link name="Left_Shank">
@@ -28,4 +28,11 @@
       </inertial>
     </link>
+    <gazebo reference="LSy">
+        <implicitSpringDamper>${Damper_val}</implicitSpringDamper>
+        <springStiffness>${springstiffness_val}</springStiffness>
+        <springReference>${springReference_val}</springReference>
+        <stopErp>${stopErp_val}</stopErp>
+        <stopCfm>${stopCfm_val}</stopCfm>
+    </gazebo>
     <gazebo reference="Left_Shank">
         <material>Gazebo/Grey</material>
@@ -35,4 +42,5 @@
         <kd value="${kd_val}" />
         <maxVel value="${maxVel_val}"/>
+        <dampingFactor value="${dampigFactor_val}"/>
         <selfCollide>${selfCollide_val}</selfCollide>
     </gazebo>

File: description/RobotElements/LeftLegElems/Lthigh.xacro (robot description, xacro)
@@ -6,5 +6,5 @@
       <child link="Left_Thigh"/>
       <axis xyz="0 1.0 0"/>
-      <limit lower="${-pi/2}" upper="${pi/2}" effort="100" velocity="100"/>
+      <limit lower="${-pi/2}" upper="${pi/2}" effort="1" velocity="1"/>
     </joint>
     <link name="Left_Thigh">
@@ -28,4 +28,11 @@
       </inertial>
     </link>
+    <gazebo reference="LTy">
+        <implicitSpringDamper>${Damper_val}</implicitSpringDamper>
+        <springStiffness>${springstiffness_val}</springStiffness>
+        <springReference>${springReference_val}</springReference>
+        <stopErp>${stopErp_val}</stopErp>
+        <stopCfm>${stopCfm_val}</stopCfm>
+    </gazebo>
     <gazebo reference="Left_Thigh">
         <material>Gazebo/Grey</material>
@@ -35,4 +42,5 @@
         <kd value="${kd_val}" />
         <maxVel value="${maxVel_val}"/>
+        <dampingFactor value="${dampigFactor_val}"/>
         <selfCollide>${selfCollide_val}</selfCollide>
     </gazebo>

File: description/RobotElements/RightArmElems/Rarm.xacro (robot description, xacro)
@@ -6,5 +6,5 @@
         <child link="Right_Arm"/>
         <axis xyz="1.0 0 0"/>
-        <limit lower="${-pi/2}" upper="${pi/2}" effort="100" velocity="100"/>
+        <limit lower="${-pi/2}" upper="${pi/2}" effort="1" velocity="1"/>
     </joint>
     <link name="Right_Arm">
@@ -28,4 +28,11 @@
         </inertial>
     </link>
+    <gazebo reference="RAx">
+        <implicitSpringDamper>${Damper_val}</implicitSpringDamper>
+        <springStiffness>${springstiffness_val}</springStiffness>
+        <springReference>${springReference_val}</springReference>
+        <stopErp>${stopErp_val}</stopErp>
+        <stopCfm>${stopCfm_val}</stopCfm>
+    </gazebo>
     <gazebo reference="Right_Arm">
         <material>Gazebo/Grey</material>
@@ -35,4 +42,5 @@
         <kd value="${kd_val}" />
         <maxVel value="${maxVel_val}"/>
+        <dampingFactor value="${dampigFactor_val}"/>
         <selfCollide>${selfCollide_val}</selfCollide>
     </gazebo>

File: description/RobotElements/RightArmElems/Rarmmount.xacro (robot description, xacro)
@@ -6,5 +6,5 @@
         <child link="Right_ArmMounting"/>
         <axis xyz="0 1.0 0"/>
-        <limit lower="${-pi/2}" upper="${pi/2}" effort="100" velocity="100"/>
+        <limit lower="${-pi/2}" upper="${pi/2}" effort="1" velocity="1"/>
     </joint>
     <link name="Right_ArmMounting">
@@ -28,4 +28,11 @@
         </inertial>
     </link>
+    <gazebo reference="RAy">
+        <implicitSpringDamper>${Damper_val}</implicitSpringDamper>
+        <springStiffness>${springstiffness_val}</springStiffness>
+        <springReference>${springReference_val}</springReference>
+        <stopErp>${stopErp_val}</stopErp>
+        <stopCfm>${stopCfm_val}</stopCfm>
+    </gazebo>
     <gazebo reference="Right_ArmMounting">
         <material>Gazebo/Grey</material>
@@ -35,4 +42,5 @@
         <kd value="${kd_val}" />
         <maxVel value="${maxVel_val}"/>
+        <dampingFactor value="${dampigFactor_val}"/>
         <selfCollide>${selfCollide_val}</selfCollide>
     </gazebo>

File: description/RobotElements/RightArmElems/Rforearm.xacro (robot description, xacro)
@@ -6,5 +6,5 @@
         <child link="Right_Forearm"/>
         <axis xyz="0 1.0 0"/>
-        <limit lower="${-pi/2}" upper="${pi/2}" effort="100" velocity="100"/>
+        <limit lower="${-pi/2}" upper="${pi/2}" effort="1" velocity="1"/>
     </joint>
     <link name="Right_Forearm">
@@ -28,4 +28,11 @@
         </inertial>
     </link>
+    <gazebo reference="RFAy">
+        <implicitSpringDamper>${Damper_val}</implicitSpringDamper>
+        <springStiffness>${springstiffness_val}</springStiffness>
+        <springReference>${springReference_val}</springReference>
+        <stopErp>${stopErp_val}</stopErp>
+        <stopCfm>${stopCfm_val}</stopCfm>
+    </gazebo>
     <gazebo reference="Right_Forearm">
         <material>Gazebo/Grey</material>
@@ -35,4 +42,5 @@
         <kd value="${kd_val}" />
         <maxVel value="${maxVel_val}"/>
+        <dampingFactor value="${dampigFactor_val}"/>
         <selfCollide>${selfCollide_val}</selfCollide>
     </gazebo>

File: description/RobotElements/RightLegElems/Rankle.xacro (robot description, xacro)
@@ -6,5 +6,5 @@
         <child link="Right_Ankle"/>
         <axis xyz="0 1.0 0"/>
-        <limit lower="${-pi/2}" upper="${pi/2}" effort="100" velocity="100"/>
+        <limit lower="${-pi/2}" upper="${pi/2}" effort="1" velocity="1"/>
     </joint>
     <link name="Right_Ankle">
@@ -30,4 +30,11 @@
         </inertial>
     </link>
+    <gazebo reference="RFy">
+        <implicitSpringDamper>${Damper_val}</implicitSpringDamper>
+        <springStiffness>${springstiffness_val}</springStiffness>
+        <springReference>${springReference_val}</springReference>
+        <stopErp>${stopErp_val}</stopErp>
+        <stopCfm>${stopCfm_val}</stopCfm>
+    </gazebo>
     <gazebo reference="Right_Ankle">
         <material>Gazebo/Grey</material>
@@ -37,4 +44,5 @@
         <kd value="${kd_val}" />
         <maxVel value="${maxVel_val}"/>
+        <dampingFactor value="${dampigFactor_val}"/>
         <selfCollide>${selfCollide_val}</selfCollide>
     </gazebo>

File: description/RobotElements/RightLegElems/Rfoot.xacro (robot description, xacro)
@@ -6,5 +6,7 @@
         <child link="Right_Foot"/>
         <axis xyz="1.0 0 0"/>
-        <limit lower="${-pi/2}" upper="${pi/2}" effort="100" velocity="100"/>
+        <limit lower="${-pi/2}" upper="${pi/2}" effort="1" velocity="1"/>
+        <dynamics damping="0.7" friction="0.5"/>
+        <dynamics damping="${damping_val}" friction="${friction_val}"/>
     </joint>
     <link name="Right_Foot">
@@ -28,11 +30,19 @@
         </inertial>
     </link>
+    <gazebo reference="RFx">
+        <implicitSpringDamper>${Damper_val}</implicitSpringDamper>
+        <springStiffness>${springstiffness_val}</springStiffness>
+        <springReference>${springReference_val}</springReference>
+        <stopErp>${stopErp_val}</stopErp>
+        <stopCfm>${stopCfm_val}</stopCfm>
+    </gazebo>
     <gazebo reference="Right_Foot">
         <material>Gazebo/Grey</material>
-        <mu1 value="0.02"/>
-        <mu2 value="0.03"/>
+        <mu1 value="${mu1_val}"/>
+        <mu2 value="${mu2_val}"/>
         <kp value="${kp_val}" />
         <kd value="${kd_val}" />
         <maxVel value="${maxVel_val}"/>
+        <dampingFactor value="${dampigFactor_val}"/>
         <selfCollide>${selfCollide_val}</selfCollide>
     </gazebo>

File: description/RobotElements/RightLegElems/Rhip.xacro (robot description, xacro)
@@ -6,5 +6,5 @@
         <child link="Right_Hip"/>
         <axis xyz="1.0 0 0"/>
-        <limit lower="${-pi/2}" upper="${pi/2}" effort="100" velocity="100"/>
+        <limit lower="${-pi/2}" upper="${pi/2}" effort="1" velocity="1"/>
     </joint>
     <link name="Right_Hip">
@@ -28,4 +28,11 @@
         </inertial>
     </link>
+    <gazebo reference="RTx">
+        <implicitSpringDamper>${Damper_val}</implicitSpringDamper>
+        <springStiffness>${springstiffness_val}</springStiffness>
+        <springReference>${springReference_val}</springReference>
+        <stopErp>${stopErp_val}</stopErp>
+        <stopCfm>${stopCfm_val}</stopCfm>
+    </gazebo>
     <gazebo reference="Right_Hip">
         <material>Gazebo/Grey</material>
@@ -35,4 +42,5 @@
         <kd value="${kd_val}" />
         <maxVel value="${maxVel_val}"/>
+        <dampingFactor value="${dampigFactor_val}"/>
         <selfCollide>${selfCollide_val}</selfCollide>
     </gazebo>

File: description/RobotElements/RightLegElems/Rhipmount.xacro (robot description, xacro)
@@ -6,5 +6,5 @@
         <child link="Right_HipMount"/>
         <axis xyz="0 0 1.0"/>
-        <limit lower="${-pi/2}" upper="${pi/2}" effort="100" velocity="100"/>
+        <limit lower="${-pi/2}" upper="${pi/2}" effort="1" velocity="1"/>
     </joint>
     <link name="Right_HipMount">
@@ -28,4 +28,11 @@
         </inertial>
     </link>
+    <gazebo reference="RTz">
+        <implicitSpringDamper>${Damper_val}</implicitSpringDamper>
+        <springStiffness>${springstiffness_val}</springStiffness>
+        <springReference>${springReference_val}</springReference>
+        <stopErp>${stopErp_val}</stopErp>
+        <stopCfm>${stopCfm_val}</stopCfm>
+    </gazebo>
     <gazebo reference="Right_HipMount">
         <material>Gazebo/Grey</material>
@@ -35,4 +42,5 @@
         <kd value="${kd_val}" />
         <maxVel value="${maxVel_val}"/>
+        <dampingFactor value="${dampigFactor_val}"/>
         <selfCollide>${selfCollide_val}</selfCollide>
     </gazebo>

File: description/RobotElements/RightLegElems/Rshank.xacro (robot description, xacro)
@@ -6,5 +6,5 @@
       <child link="Right_Shank"/>
       <axis xyz="0 1.0 0"/>
-      <limit lower="${-pi/2}" upper="${pi/2}" effort="100" velocity="100"/>
+      <limit lower="${-pi/2}" upper="${pi/2}" effort="1" velocity="1"/>
     </joint>
     <link name="Right_Shank">
@@ -28,4 +28,11 @@
         </inertial>
     </link>
+    <gazebo reference="RSy">
+        <implicitSpringDamper>${Damper_val}</implicitSpringDamper>
+        <springStiffness>${springstiffness_val}</springStiffness>
+        <springReference>${springReference_val}</springReference>
+        <stopErp>${stopErp_val}</stopErp>
+        <stopCfm>${stopCfm_val}</stopCfm>
+    </gazebo>
     <gazebo reference="Right_Shank">
         <material>Gazebo/Grey</material>
@@ -35,4 +42,5 @@
         <kd value="${kd_val}" />
         <maxVel value="${maxVel_val}"/>
+        <dampingFactor value="${dampigFactor_val}"/>
         <selfCollide>${selfCollide_val}</selfCollide>
     </gazebo>

Commit message: Created launchfile that segregates launchproceses in time. Robot description topics and other parameters are passed in the way that doens't cause errors. Velocity controller and joint trajectory controllers active

File: description/Melman_ros2control_gazebo.xacro (robot description, xacro)
@@ -4,4 +4,5 @@
         <hardware>
             <plugin>gazebo_ros2_control/GazeboSystem</plugin>
+            <!-- <plugin>dynamixel_hardware/DynamixelHardware</plugin> -->
         </hardware>
         <!-- Right Thigh Z axis rotation control -->
@@ -272,5 +273,9 @@
     <gazebo>
       <plugin filename="libgazebo_ros2_control.so" name="gazebo_ros2_control">
+            <robot_param>robot_description</robot_param>
+            <robot_param_node>robot_state_publisher</robot_param_node>
             <parameters>$(find ros2_humanoid_virtual_twin)/controllers/controllers.yaml</parameters>
+            <hold_joints>true</hold_joints>
+            <controller_manager_name>controller_manager</controller_manager_name>
       </plugin>
     </gazebo>

File: description/RobotElements/LeftArmElems/Lforearm.xacro (robot description, xacro)
@@ -16,10 +16,10 @@
             <material name="grey"/>
         </visual>
-        <collision>
+        <!-- <collision>
             <origin xyz="0 0 0" rpy="0 0 0"/>
             <geometry>
                 <mesh filename="file://$(find ros2_humanoid_virtual_twin)/meshes/Right_Forearm.stl" scale="0.001 0.001 0.001"/>
             </geometry>
-        </collision>
+        </collision> -->
         <inertial>
             <origin xyz="0 0 -93.816e-3" rpy="0 0 0"/>
@@ -37,5 +37,5 @@
     <gazebo reference="Left_Forearm">
         <material>Gazebo/Grey</material>
-        <mu1 value="${mu1_val}"/>
+        <!-- <mu1 value="${mu1_val}"/>
         <mu2 value="${mu2_val}"/>
         <kp value="${kp_val}" />
@@ -43,5 +43,5 @@
         <maxVel value="${maxVel_val}"/>
         <dampingFactor value="${dampigFactor_val}"/>
-        <selfCollide>${selfCollide_val}</selfCollide>
+        <selfCollide>${selfCollide_val}</selfCollide>   -->
     </gazebo>
 </robot>

File: description/RobotElements/RightArmElems/Rforearm.xacro (robot description, xacro)
@@ -16,10 +16,10 @@
             <material name="grey"/>
         </visual>
-        <collision>
+        <!-- <collision>
             <origin xyz="0 0 0" rpy="0 0 0"/>
             <geometry>
                 <mesh filename="file://$(find ros2_humanoid_virtual_twin)/meshes/Right_Forearm.stl" scale="0.001 0.001 0.001"/>
             </geometry>
-        </collision>
+        </collision> -->
         <inertial>
             <origin xyz="0 0 -93.816e-3" rpy="0 0 0"/>
@@ -37,5 +37,5 @@
     <gazebo reference="Right_Forearm">
         <material>Gazebo/Grey</material>
-        <mu1 value="${mu1_val}"/>
+        <!-- <mu1 value="${mu1_val}"/>
         <mu2 value="${mu2_val}"/>
         <kp value="${kp_val}" />
@@ -43,5 +43,5 @@
         <maxVel value="${maxVel_val}"/>
         <dampingFactor value="${dampigFactor_val}"/>
-        <selfCollide>${selfCollide_val}</selfCollide>
+        <selfCollide>${selfCollide_val}</selfCollide>    -->
     </gazebo>
 </robot>

File: description/robot.urdf.xacro (robot description, xacro)
@@ -2,5 +2,5 @@
 <robot xmlns:xacro="http://www.ros.org/wiki/xacro"  name="Melman">
     <!-- Below is a file which initiates geometry of robot and inertial, dynamic, collision parameters -->
-    <xacro:include filename="robot_core.xacro" />
+    <xacro:include filename="$(find ros2_humanoid_virtual_twin)/description/robot_core.xacro" />
     <!-- If you want the Trunk to be immovable and static at a certain height uncomment lines below -->
     <!-- <link name="world"/>
