Commit message: Reparation of main branch

File: description/Melman_ros2control_gazebo.xacro (robot description, xacro)
@@ -6,4 +6,97 @@
             <!-- <plugin>dynamixel_hardware/DynamixelHardware</plugin> -->
         </hardware>
+        <!-- Right Thigh Z axis rotation control -->
+        <joint name="RTz">
+            <command_interface name="position">
+                <param name="min">${-pi/2}</param>
+                <param name="max">${pi/2}</param>
+            </command_interface>
+            <command_interface name="velocity">
+                <param name="min">-5.0</param>
+                <param name="max">5.0</param>
+            </command_interface>
+            <state_interface name="position"/>
+            <state_interface name="velocity"/>
+        </joint>
+        <!-- Right Thigh X axis rotation control-->
+        <joint name="RTx">
+            <command_interface name="position">
+                <param name="min">${-pi/2}</param>
+                <param name="max">${pi/2}</param>
+            </command_interface>
+            <command_interface name="velocity">
+                <param name="min">-5.0</param>
+                <param name="max">5.0</param>
+            </command_interface>
+            <state_interface name="position"/>
+            <state_interface name="velocity"/>
+        </joint>
+        <!-- Right Thigh Y axis rotation control-->
+        <joint name="RTy">
+            <command_interface name="position">
+                <param name="min">${-pi/2}</param>
+                <param name="max">${pi/2}</param>
+            </command_interface>
+            <command_interface name="velocity">
+                <param name="min">-5.0</param>
+                <param name="max">5.0</param>
+            </command_interface>
+            <state_interface name="position">
+                <!-- <param name="initial_value">-0.1</param> -->
+            </state_interface>
+            <state_interface name="velocity"/>
+        </joint>
+        <!-- Right shank Y axis rotation control-->
+        <joint name="RSy">
+            <command_interface name="position">
+                <param name="min">${-pi/2}</param>
+                <param name="max">${pi/2}</param>
+            </command_interface>
+            <command_interface name="velocity">
+                <param name="min">-5.0</param>
+                <param name="max">5.0</param>
+            </command_interface>
+            <state_interface name="position"/>
+            <state_interface name="velocity"/>
+        </joint>
+        <!--Right foot Y axis rotation control -->
+        <joint name="RFy">
+            <command_interface name="position">
+                <param name="min">${-pi/2}</param>
+                <param name="max">${pi/2}</param>
+            </command_interface>
+            <command_interface name="velocity">
+                <param name="min">-5.0</param>
+                <param name="max">5.0</param>
+            </command_interface>
+            <state_interface name="position"/>
+            <state_interface name="velocity"/>
+        </joint>
+        <!-- Right foot X axis rotation control-->
+        <joint name="RFx">
+            <command_interface name="position">
+                <param name="min">${-pi/2}</param>
+                <param name="max">${pi/2}</param>
+            </command_interface>
+            <command_interface name="velocity">
+                <param name="min">-5.0</param>
+                <param name="max">5.0</param>
+            </command_interface>
+            <state_interface name="position"/>
+            <state_interface name="velocity"/>
+        </joint>
+        <!-- Left thigh z axis rotation control-->
+        <joint name="LTz">
+            <command_interface name="position">
+                <param name="min">${-pi/2}</param>
+                <param name="max">${pi/2}</param>
+            </command_interface>
+            <command_interface name="velocity">
+                <param name="min">-5.0</param>
+                <param name="max">5.0</param>
+            </command_interface>
+            <state_interface name="position"/>
+            <state_interface name="velocity"/>
+        </joint>
         <!--Left thigh x axis rotation control -->
         <joint name="LTx">
@@ -16,8 +109,6 @@
                 <param name="max">5.0</param>
             </command_interface>
-            <command_interface name="effort"/>
-            <state_interface name="position"/>
-            <state_interface name="velocity"/>
-            <state_interface name="effort"/>
+            <state_interface name="position"/>
+            <state_interface name="velocity"/>
         </joint>
         <!-- Left thigh y axis rotation control-->
@@ -31,8 +122,6 @@
                 <param name="max">5.0</param>
             </command_interface>
-            <command_interface name="effort"/>
             <state_interface name="position">
-                <!-- <param name="initial_valu
-                <state_interface name="effort"/>e">-0.1</param> -->
+                <!-- <param name="initial_value">-0.1</param> -->
             </state_interface>
             <state_interface name="velocity"/>
@@ -48,8 +137,6 @@
                 <param name="max">5.0</param>
             </command_interface>
-            <command_interface name="effort"/>
-            <state_interface name="position"/>
-            <state_interface name="velocity"/>
-            <state_interface name="effort"/>
+            <state_interface name="position"/>
+            <state_interface name="velocity"/>
         </joint>
         <!-- Left foot y axis rotation control-->
@@ -63,8 +150,6 @@
                 <param name="max">5.0</param>
             </command_interface>
-            <command_interface name="effort"/>
-            <state_interface name="position"/>
-            <state_interface name="velocity"/>
-            <state_interface name="effort"/>
+            <state_interface name="position"/>
+            <state_interface name="velocity"/>
         </joint>
         <!--Left foot x axis rotation control -->
@@ -78,8 +163,110 @@
                 <param name="max">5.0</param>
             </command_interface>
-            <command_interface name="effort"/>
-            <state_interface name="position"/>
-            <state_interface name="velocity"/>
-            <state_interface name="effort"/>
+            <state_interface name="position"/>
+            <state_interface name="velocity"/>
+        </joint>
+        <!-- Right arm y axis rotation control -->
+        <joint name="RAy">
+            <command_interface name="position">
+                <param name="min">${-pi/2}</param>
+                <param name="max">${pi/2}</param>
+            </command_interface>
+            <command_interface name="velocity">
+                <param name="min">-5.0</param>
+                <param name="max">5.0</param>
+            </command_interface>
+            <state_interface name="position"/>
+            <state_interface name="velocity"/>
+        </joint>
+        <!-- Right arm x axis rotation control-->
+        <joint name="RAx">
+            <command_interface name="position">
+                <param name="min">${-pi/2}</param>
+                <param name="max">${pi/2}</param>
+            </command_interface>
+            <command_interface name="velocity">
+                <param name="min">-5.0</param>
+                <param name="max">5.0</param>
+            </command_interface>
+            <state_interface name="position"/>
+            <state_interface name="velocity"/>
+        </joint>
+        <!-- Roght forearm y axis rotation control-->
+        <joint name="RFAy">
+            <command_interface name="position">
+                <param name="min">${-pi/2}</param>
+                <param name="max">${pi/2}</param>
+            </command_interface>
+            <command_interface name="velocity">
+                <param name="min">-5.0</param>
+                <param name="max">5.0</param>
+            </command_interface>
+            <state_interface name="position"/>
+            <state_interface name="velocity"/>
+        </joint>
+        <!--Left arm y axis rotation control -->
+        <joint name="LAy">
+            <command_interface name="position">
+                <param name="min">${-pi/2}</param>
+                <param name="max">${pi/2}</param>
+            </command_interface>
+            <command_interface name="velocity">
+              <param name="min">-5.0</param>
+                <param name="max">5.0</param>
+            </command_interface>
+            <state_interface name="position"/>
+            <state_interface name="velocity"/>
+        </joint>
+        <!-- Left arm x axis rotation control -->
+        <joint name="LAx">
+            <command_interface name="position">
+                <param name="min">${-pi/2}</param>
+                <param name="max">${pi/2}</param>
+            </command_interface>
+            <command_interface name="velocity">
+                <param name="min">-5.0</param>
+                <param name="max">5.0</param>
+            </command_interface>
+            <state_interface name="position"/>
+            <state_interface name="velocity"/>
+        </joint>
+        <!-- Left forearm y axis rotation control -->
+        <joint name="LFAy">
+            <command_interface name="position">
+                <param name="min">${-pi/2}</param>
+                <param name="max">${pi/2}</param>
+            </command_interface>
+            <command_interface name="velocity">
+                <param name="min">-5.0</param>
+                <param name="max">5.0</param>
+            </command_interface>
+            <state_interface name="position"/>
+            <state_interface name="velocity"/>
+        </joint>
+        <!-- Head z axis rotation control-->
+        <joint name="Hz">
+            <command_interface name="position">
+                <param name="min">${-pi/2}</param>
+                <param name="max">${pi/2}</param>
+            </command_interface>
+            <command_interface name="velocity">
+                <param name="min">-5.0</param>
+                <param name="max">5.0</param>
+            </command_interface>
+            <state_interface name="position"/>
+            <state_interface name="velocity"/>
+        </joint>
+        <!-- Head y axis rotation control-->
+        <joint name="Hy">
+            <command_interface name="position">
+                <param name="min">${-pi/2}</param>
+                <param name="max">${pi/2}</param>
+            </command_interface>
+            <command_interface name="velocity">
+                <param name="min">-5.0</param>
+                <param name="max">5.0</param>
+            </command_interface>
+            <state_interface name="position"/>
+            <state_interface name="velocity"/>
         </joint>
     </ros2_control>
@@ -89,5 +276,5 @@
             <robot_param_node>robot_state_publisher</robot_param_node>
             <parameters>$(find ros2_humanoid_virtual_twin)/controllers/controllers.yaml</parameters>
-            <hold_joints>true</hold_joints>
+            <hold_joints>false</hold_joints>
             <controller_manager_name>controller_manager</controller_manager_name>
       </plugin>

File: description/RobotElements/LeftLegElems/Lhipmount.xacro (robot description, xacro)
@@ -1,14 +1,8 @@
 <?xml version="1.0"?>
 <robot xmlns:xacro="http://www.ros.org/wiki/xacro" >
-  <joint name="Trunk_joint" type="fixed">
-      <parent link="base_link"/>
-      <child link="Left_HipMount"/>
-      <!--Origin defines translation child frame relative to parent frame. Translation is performed in parent frame.-->
-      <origin xyz="0 0 0.3" rpy="0 0 0"/>
-  </joint>
   <!-- LEFT HIP MOUNT-->
-  <!-- <joint name="LTz" type="revolute"> -->
+  <joint name="LTz" type="revolute">
     <!--Origin defines translation child frame relative to parent frame. Translation is performed in parent frame.-->
-    <!-- <origin xyz="0	40e-3	-150.065e-3" rpy="0 0 0"/>
+    <origin xyz="0	40e-3	-150.065e-3" rpy="0 0 0"/>
     <parent link="Trunk"/>
     <child link="Left_HipMount"/>
@@ -18,5 +12,5 @@
         <dynamics damping="${damping_val}" friction="${friction_val}"/>
     </xacro:if>
-  </joint>   -->
+  </joint>
   <link name="Left_HipMount">
     <visual>

File: description/robot_core.xacro (robot description, xacro)
@@ -2,8 +2,8 @@
 <robot xmlns:xacro="http://www.ros.org/wiki/xacro" >
   <!-- Definition of GAZEBO physics coefficients for LINKS -->
-	<xacro:property name="kp_val" value="1000000000.0"/>
-  <xacro:property name="kd_val" value="1"/>
-  <xacro:property name="mu1_val" value="300"/>
-  <xacro:property name="mu2_val" value="300"/>
+	<xacro:property name="kp_val" value="25000.0"/>
+  <xacro:property name="kd_val" value="0.05"/>
+  <xacro:property name="mu1_val" value="50"/>
+  <xacro:property name="mu2_val" value="25"/>
   <xacro:property name="maxVel_val" value="0.1"/>
   <xacro:property name="dampigFactor_val" value="0.004"/>
@@ -27,9 +27,9 @@
   <link name="base_link">
   </link>
-  <!-- <xacro:include filename="RobotElements/Trunk.xacro"/> -->
+  <xacro:include filename="RobotElements/Trunk.xacro"/>
   <xacro:include filename="RobotElements/left_leg.xacro"/>
-  <!-- <xacro:include filename="RobotElements/right_leg.xacro"/>
+  <xacro:include filename="RobotElements/right_leg.xacro"/>
   <xacro:include filename="RobotElements/left_arm.xacro"/>
   <xacro:include filename="RobotElements/right_arm.xacro"/>
-  <xacro:include filename="RobotElements/head.xacro"/> -->
+  <xacro:include filename="RobotElements/head.xacro"/>
 </robot>
