Commit message: Added ros2control rviz connection

File: description/Melman_ros2control_gazebo.xacro (robot description, xacro)
@@ -3,35 +3,47 @@
     <ros2_control name="Melman_ros2control_gazebo" type="system">
         <hardware>
-            <plugin>gazebo_ros2_control/GazeboSystem</plugin>
-            <!-- <plugin>dynamixel_hardware/DynamixelHardware</plugin> -->
+            <xacro:if value="$(arg use_gazebo)">
+                <plugin>gazebo_ros2_control/GazeboSystem</plugin>
+            </xacro:if>
+            <xacro:unless value="$(arg use_gazebo)">
+                <plugin>dynamixel_hardware/DynamixelHardware</plugin>
+                <param name="usb_port">/dev/ttyUSB0</param>
+                <param name="baud_rate">57600</param>
+                <param name="use_dummy">true</param>
+            </xacro:unless>
         </hardware>
         <!-- Right Thigh Z axis rotation control -->
         <joint name="RTz">
-            <command_interface name="position">
-                <param name="min">${-pi/2}</param>
-                <param name="max">${pi/2}</param>
-            </command_interface>
-            <command_interface name="velocity">
-                <param name="min">-5.0</param>
-                <param name="max">5.0</param>
-            </command_interface>
-            <state_interface name="position"/>
-            <state_interface name="velocity"/>
+            <param name="id">1</param>
+            <command_interface name="position">
+                <param name="min">${-pi/2}</param>
+                <param name="max">${pi/2}</param>
+            </command_interface>
+            <command_interface name="velocity">
+                <param name="min">-5.0</param>
+                <param name="max">5.0</param>
+            </command_interface>
+            <state_interface name="position"/>
+            <state_interface name="velocity"/>
+            <state_interface name="effort"/>
         </joint>
         <!-- Right Thigh X axis rotation control-->
         <joint name="RTx">
-            <command_interface name="position">
-                <param name="min">${-pi/2}</param>
-                <param name="max">${pi/2}</param>
-            </command_interface>
-            <command_interface name="velocity">
-                <param name="min">-5.0</param>
-                <param name="max">5.0</param>
-            </command_interface>
-            <state_interface name="position"/>
-            <state_interface name="velocity"/>
+            <param name="id">2</param>
+            <command_interface name="position">
+                <param name="min">${-pi/2}</param>
+                <param name="max">${pi/2}</param>
+            </command_interface>
+            <command_interface name="velocity">
+                <param name="min">-5.0</param>
+                <param name="max">5.0</param>
+            </command_interface>
+            <state_interface name="position"/>
+            <state_interface name="velocity"/>
+            <state_interface name="effort"/>
         </joint>
         <!-- Right Thigh Y axis rotation control-->
         <joint name="RTy">
+            <param name="id">3</param>
             <command_interface name="position">
                 <param name="min">${-pi/2}</param>
@@ -46,72 +58,84 @@
             </state_interface>
             <state_interface name="velocity"/>
+            <state_interface name="effort"/>
         </joint>
         <!-- Right shank Y axis rotation control-->
         <joint name="RSy">
-            <command_interface name="position">
-                <param name="min">${-pi/2}</param>
-                <param name="max">${pi/2}</param>
-            </command_interface>
-            <command_interface name="velocity">
-                <param name="min">-5.0</param>
-                <param name="max">5.0</param>
-            </command_interface>
-            <state_interface name="position"/>
-            <state_interface name="velocity"/>
+            <param name="id">4</param>
+            <command_interface name="position">
+                <param name="min">${-pi/2}</param>
+                <param name="max">${pi/2}</param>
+            </command_interface>
+            <command_interface name="velocity">
+                <param name="min">-5.0</param>
+                <param name="max">5.0</param>
+            </command_interface>
+            <state_interface name="position"/>
+            <state_interface name="velocity"/>
+            <state_interface name="effort"/>
         </joint>
         <!--Right foot Y axis rotation control -->
         <joint name="RFy">
-            <command_interface name="position">
-                <param name="min">${-pi/2}</param>
-                <param name="max">${pi/2}</param>
-            </command_interface>
-            <command_interface name="velocity">
-                <param name="min">-5.0</param>
-                <param name="max">5.0</param>
-            </command_interface>
-            <state_interface name="position"/>
-            <state_interface name="velocity"/>
+            <param name="id">5</param>
+            <command_interface name="position">
+                <param name="min">${-pi/2}</param>
+                <param name="max">${pi/2}</param>
+            </command_interface>
+            <command_interface name="velocity">
+                <param name="min">-5.0</param>
+                <param name="max">5.0</param>
+            </command_interface>
+            <state_interface name="position"/>
+            <state_interface name="velocity"/>
+            <state_interface name="effort"/>
         </joint>
         <!-- Right foot X axis rotation control-->
         <joint name="RFx">
-            <command_interface name="position">
-                <param name="min">${-pi/2}</param>
-                <param name="max">${pi/2}</param>
-            </command_interface>
-            <command_interface name="velocity">
-                <param name="min">-5.0</param>
-                <param name="max">5.0</param>
-            </command_interface>
-            <state_interface name="position"/>
-            <state_interface name="velocity"/>
+            <param name="id">6</param>
+            <command_interface name="position">
+                <param name="min">${-pi/2}</param>
+                <param name="max">${pi/2}</param>
+            </command_interface>
+            <command_interface name="velocity">
+                <param name="min">-5.0</param>
+                <param name="max">5.0</param>
+            </command_interface>
+            <state_interface name="position"/>
+            <state_interface name="velocity"/>
+            <state_interface name="effort"/>
         </joint>
         <!-- Left thigh z axis rotation control-->
         <joint name="LTz">
-            <command_interface name="position">
-                <param name="min">${-pi/2}</param>
-                <param name="max">${pi/2}</param>
-            </command_interface>
-            <command_interface name="velocity">
-                <param name="min">-5.0</param>
-                <param name="max">5.0</param>
-            </command_interface>
-            <state_interface name="position"/>
-            <state_interface name="velocity"/>
+            <param name="id">7</param>
+            <command_interface name="position">
+                <param name="min">${-pi/2}</param>
+                <param name="max">${pi/2}</param>
+            </command_interface>
+            <command_interface name="velocity">
+                <param name="min">-5.0</param>
+                <param name="max">5.0</param>
+            </command_interface>
+            <state_interface name="position"/>
+            <state_interface name="velocity"/>
+            <state_interface name="effort"/>
         </joint>
         <!--Left thigh x axis rotation control -->
         <joint name="LTx">
-            <command_interface name="position">
-                <param name="min">${-pi/2}</param>
-                <param name="max">${pi/2}</param>
-            </command_interface>
-            <command_interface name="velocity">
-                <param name="min">-5.0</param>
-                <param name="max">5.0</param>
-            </command_interface>
-            <state_interface name="position"/>
-            <state_interface name="velocity"/>
+            <param name="id">8</param>
+            <command_interface name="position">
+                <param name="min">${-pi/2}</param>
+                <param name="max">${pi/2}</param>
+            </command_interface>
+            <command_interface name="velocity">
+                <param name="min">-5.0</param>
+                <param name="max">5.0</param>
+            </command_interface>
+            <state_interface name="position"/>
+            <state_interface name="velocity"/>
+            <state_interface name="effort"/>
         </joint>
         <!-- Left thigh y axis rotation control-->
         <joint name="LTy">
+            <param name="id">9</param>
             <command_interface name="position">
                 <param name="min">${-pi/2}</param>
@@ -126,85 +150,99 @@
             </state_interface>
             <state_interface name="velocity"/>
+            <state_interface name="effort"/>
         </joint>
         <!-- Left shank y axis rotation control-->
         <joint name="LSy">
-            <command_interface name="position">
-                <param name="min">${-pi/2}</param>
-                <param name="max">${pi/2}</param>
-            </command_interface>
-            <command_interface name="velocity">
-                <param name="min">-5.0</param>
-                <param name="max">5.0</param>
-            </command_interface>
-            <state_interface name="position"/>
-            <state_interface name="velocity"/>
+            <param name="id">10</param>
+            <command_interface name="position">
+                <param name="min">${-pi/2}</param>
+                <param name="max">${pi/2}</param>
+            </command_interface>
+            <command_interface name="velocity">
+                <param name="min">-5.0</param>
+                <param name="max">5.0</param>
+            </command_interface>
+            <state_interface name="position"/>
+            <state_interface name="velocity"/>
+            <state_interface name="effort"/>
         </joint>
         <!-- Left foot y axis rotation control-->
         <joint name="LFy">
-            <command_interface name="position">
-                <param name="min">${-pi/2}</param>
-                <param name="max">${pi/2}</param>
-            </command_interface>
-            <command_interface name="velocity">
-                <param name="min">-5.0</param>
-                <param name="max">5.0</param>
-            </command_interface>
-            <state_interface name="position"/>
-            <state_interface name="velocity"/>
+            <param name="id">11</param>
+            <command_interface name="position">
+                <param name="min">${-pi/2}</param>
+                <param name="max">${pi/2}</param>
+            </command_interface>
+            <command_interface name="velocity">
+                <param name="min">-5.0</param>
+                <param name="max">5.0</param>
+            </command_interface>
+            <state_interface name="position"/>
+            <state_interface name="velocity"/>
+            <state_interface name="effort"/>
         </joint>
         <!--Left foot x axis rotation control -->
         <joint name="LFx">
-            <command_interface name="position">
-                <param name="min">${-pi/2}</param>
-                <param name="max">${pi/2}</param>
-            </command_interface>
-            <command_interface name="velocity">
-                <param name="min">-5.0</param>
-                <param name="max">5.0</param>
-            </command_interface>
-            <state_interface name="position"/>
-            <state_interface name="velocity"/>
+            <param name="id">12</param>
+            <command_interface name="position">
+                <param name="min">${-pi/2}</param>
+                <param name="max">${pi/2}</param>
+            </command_interface>
+            <command_interface name="velocity">
+                <param name="min">-5.0</param>
+                <param name="max">5.0</param>
+            </command_interface>
+            <state_interface name="position"/>
+            <state_interface name="velocity"/>
+            <state_interface name="effort"/>
         </joint>
         <!-- Right arm y axis rotation control -->
         <joint name="RAy">
-            <command_interface name="position">
-                <param name="min">${-pi/2}</param>
-                <param name="max">${pi/2}</param>
-            </command_interface>
-            <command_interface name="velocity">
-                <param name="min">-5.0</param>
-                <param name="max">5.0</param>
-            </command_interface>
-            <state_interface name="position"/>
-            <state_interface name="velocity"/>
+            <param name="id">13</param>
+            <command_interface name="position">
+                <param name="min">${-pi/2}</param>
+                <param name="max">${pi/2}</param>
+            </command_interface>
+            <command_interface name="velocity">
+                <param name="min">-5.0</param>
+                <param name="max">5.0</param>
+            </command_interface>
+            <state_interface name="position"/>
+            <state_interface name="velocity"/>
+            <state_interface name="effort"/>
         </joint>
         <!-- Right arm x axis rotation control-->
         <joint name="RAx">
-            <command_interface name="position">
-                <param name="min">${-pi/2}</param>
-                <param name="max">${pi/2}</param>
-            </command_interface>
-            <command_interface name="velocity">
-                <param name="min">-5.0</param>
-                <param name="max">5.0</param>
-            </command_interface>
-            <state_interface name="position"/>
-            <state_interface name="velocity"/>
+            <param name="id">14</param>
+            <command_interface name="position">
+                <param name="min">${-pi/2}</param>
+                <param name="max">${pi/2}</param>
+            </command_interface>
+            <command_interface name="velocity">
+                <param name="min">-5.0</param>
+                <param name="max">5.0</param>
+            </command_interface>
+            <state_interface name="position"/>
+            <state_interface name="velocity"/>
+            <state_interface name="effort"/>
         </joint>
         <!-- Roght forearm y axis rotation control-->
         <joint name="RFAy">
-            <command_interface name="position">
-                <param name="min">${-pi/2}</param>
-                <param name="max">${pi/2}</param>
-            </command_interface>
-            <command_interface name="velocity">
-                <param name="min">-5.0</param>
-                <param name="max">5.0</param>
-            </command_interface>
-            <state_interface name="position"/>
-            <state_interface name="velocity"/>
+            <param name="id">15</param>
+            <command_interface name="position">
+                <param name="min">${-pi/2}</param>
+                <param name="max">${pi/2}</param>
+            </command_interface>
+            <command_interface name="velocity">
+                <param name="min">-5.0</param>
+                <param name="max">5.0</param>
+            </command_interface>
+            <state_interface name="position"/>
+            <state_interface name="velocity"/>
+            <state_interface name="effort"/>
         </joint>
         <!--Left arm y axis rotation control -->
         <joint name="LAy">
+            <param name="id">16</param>
             <command_interface name="position">
                 <param name="min">${-pi/2}</param>
@@ -217,58 +255,68 @@
             <state_interface name="position"/>
             <state_interface name="velocity"/>
+            <state_interface name="effort"/>
         </joint>
         <!-- Left arm x axis rotation control -->
         <joint name="LAx">
-            <command_interface name="position">
-                <param name="min">${-pi/2}</param>
-                <param name="max">${pi/2}</param>
-            </command_interface>
-            <command_interface name="velocity">
-                <param name="min">-5.0</param>
-                <param name="max">5.0</param>
-            </command_interface>
-            <state_interface name="position"/>
-            <state_interface name="velocity"/>
+            <param name="id">17</param>
+            <command_interface name="position">
+                <param name="min">${-pi/2}</param>
+                <param name="max">${pi/2}</param>
+            </command_interface>
+            <command_interface name="velocity">
+                <param name="min">-5.0</param>
+                <param name="max">5.0</param>
+            </command_interface>
+            <state_interface name="position"/>
+            <state_interface name="velocity"/>
+            <state_interface name="effort"/>
         </joint>
         <!-- Left forearm y axis rotation control -->
         <joint name="LFAy">
-            <command_interface name="position">
-                <param name="min">${-pi/2}</param>
-                <param name="max">${pi/2}</param>
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
File: description/robot_core.xacro (robot description, xacro)
@@ -18,6 +18,6 @@
   <xacro:property name="damping_val" value="1.0"/>
   <xacro:property name="friction_val" value="1.0"/>
-  <xacro:property name="maxVel_val" value="0.0"/>
-  <xacro:property name="maxeffort_val" value="0.0"/>
+  <xacro:property name="maxVel_val" value="0.01"/>
+  <xacro:property name="maxeffort_val" value="0.01"/>
   <!-- Definition of grey material-->
   <material name="grey">
