Commit message: Melman finally not flying in gazebo with effort controller joint trajectory controller. PID is not set correctly

File: description/Melman_ros2control_gazebo.xacro (robot description, xacro)
@@ -24,4 +24,5 @@
                 <param name="max">5.0</param>
             </command_interface>
+            <command_interface name="effort"/>
             <state_interface name="position"/>
             <state_interface name="velocity"/>
@@ -39,4 +40,5 @@
                 <param name="max">5.0</param>
             </command_interface>
+            <command_interface name="effort"/>
             <state_interface name="position"/>
             <state_interface name="velocity"/>
@@ -54,4 +56,5 @@
                 <param name="max">5.0</param>
             </command_interface>
+            <command_interface name="effort"/>
             <state_interface name="position">
                 <!-- <param name="initial_value">-0.1</param> -->
@@ -71,4 +74,5 @@
                 <param name="max">5.0</param>
             </command_interface>
+            <command_interface name="effort"/>
             <state_interface name="position"/>
             <state_interface name="velocity"/>
@@ -86,4 +90,5 @@
                 <param name="max">5.0</param>
             </command_interface>
+            <command_interface name="effort"/>
             <state_interface name="position"/>
             <state_interface name="velocity"/>
@@ -101,4 +106,5 @@
                 <param name="max">5.0</param>
             </command_interface>
+            <command_interface name="effort"/>
             <state_interface name="position"/>
             <state_interface name="velocity"/>
@@ -116,4 +122,5 @@
                 <param name="max">5.0</param>
             </command_interface>
+            <command_interface name="effort"/>
             <state_interface name="position"/>
             <state_interface name="velocity"/>
@@ -131,4 +138,5 @@
                 <param name="max">5.0</param>
             </command_interface>
+            <command_interface name="effort"/>
             <state_interface name="position"/>
             <state_interface name="velocity"/>
@@ -146,4 +154,5 @@
                 <param name="max">5.0</param>
             </command_interface>
+            <command_interface name="effort"/>
             <state_interface name="position">
                 <!-- <param name="initial_value">-0.1</param> -->
@@ -163,4 +172,5 @@
                 <param name="max">5.0</param>
             </command_interface>
+            <command_interface name="effort"/>
             <state_interface name="position"/>
             <state_interface name="velocity"/>
@@ -178,4 +188,5 @@
                 <param name="max">5.0</param>
             </command_interface>
+            <command_interface name="effort"/>
             <state_interface name="position"/>
             <state_interface name="velocity"/>
@@ -193,4 +204,5 @@
                 <param name="max">5.0</param>
             </command_interface>
+            <command_interface name="effort"/>
             <state_interface name="position"/>
             <state_interface name="velocity"/>
@@ -208,4 +220,5 @@
                 <param name="max">5.0</param>
             </command_interface>
+            <command_interface name="effort"/>
             <state_interface name="position"/>
             <state_interface name="velocity"/>
@@ -223,4 +236,5 @@
                 <param name="max">5.0</param>
             </command_interface>
+            <command_interface name="effort"/>
             <state_interface name="position"/>
             <state_interface name="velocity"/>
@@ -238,4 +252,5 @@
                 <param name="max">5.0</param>
             </command_interface>
+            <command_interface name="effort"/>
             <state_interface name="position"/>
             <state_interface name="velocity"/>
@@ -253,4 +268,5 @@
                 <param name="max">5.0</param>
             </command_interface>
+            <command_interface name="effort"/>
             <state_interface name="position"/>
             <state_interface name="velocity"/>
@@ -268,4 +284,5 @@
                 <param name="max">5.0</param>
             </command_interface>
+            <command_interface name="effort"/>
             <state_interface name="position"/>
             <state_interface name="velocity"/>
@@ -283,4 +300,5 @@
                 <param name="max">5.0</param>
             </command_interface>
+            <command_interface name="effort"/>
             <state_interface name="position"/>
             <state_interface name="velocity"/>
@@ -298,4 +316,5 @@
                 <param name="max">5.0</param>
             </command_interface>
+            <command_interface name="effort"/>
             <state_interface name="position"/>
             <state_interface name="velocity"/>
@@ -313,4 +332,5 @@
                 <param name="max">5.0</param>
             </command_interface>
+            <command_interface name="effort"/>
             <state_interface name="position"/>
             <state_interface name="velocity"/>

File: description/robot_core.xacro (robot description, xacro)
@@ -18,6 +18,6 @@
   <xacro:property name="damping_val" value="1.0"/>
   <xacro:property name="friction_val" value="1.0"/>
-  <xacro:property name="maxVel_val" value="0.01"/>
-  <xacro:property name="maxeffort_val" value="0.01"/>
+  <xacro:property name="maxVel_val" value="5.1"/>
+  <xacro:property name="maxeffort_val" value="5.1"/>
   <!-- Definition of grey material-->
   <material name="grey">
