Commit message: Added realistic limits of servomechanisms - speed and torque. Tuned PID a bit. Added transmissions- but they propably dont work

File: description/Melman_ros2control_gazebo.xacro (robot description, xacro)
@@ -46,4 +46,11 @@
             <state_interface name="effort"/>
         </joint>
+        <transmission name="transmissionRTz">
+            <plugin>transmission_interface/SimpleTransmission</plugin>
+            <joint name="RTz" role="joint1">
+                <mechanical_reduction>200.0</mechanical_reduction>
+                <offset>0.0</offset>
+            </joint>
+        </transmission>
         <!-- Right Thigh X axis rotation control-->
         <joint name="RTx">
@@ -64,4 +71,11 @@
             <state_interface name="effort"/>
         </joint>
+        <transmission name="transmissionRTx">
+            <plugin>transmission_interface/SimpleTransmission</plugin>
+            <joint name="RTx" role="joint2">
+                <mechanical_reduction>200.0</mechanical_reduction>
+                <offset>0.0</offset>
+            </joint>
+        </transmission>
         <!-- Right Thigh Y axis rotation control-->
         <joint name="RTy">
@@ -84,4 +98,11 @@
             <state_interface name="effort"/>
         </joint>
+        <transmission name="transmissionRTy">
+            <plugin>transmission_interface/SimpleTransmission</plugin>
+            <joint name="RTy" role="joint3">
+                <mechanical_reduction>200.0</mechanical_reduction>
+                <offset>0.0</offset>
+            </joint>
+        </transmission>
         <!-- Right shank Y axis rotation control-->
         <joint name="RSy">
@@ -102,4 +123,11 @@
             <state_interface name="effort"/>
         </joint>
+        <transmission name="transmissionRSy">
+            <plugin>transmission_interface/SimpleTransmission</plugin>
+            <joint name="RSy" role="joint4">
+                <mechanical_reduction>200.0</mechanical_reduction>
+                <offset>0.0</offset>
+            </joint>
+        </transmission>
         <!--Right foot Y axis rotation control -->
         <joint name="RFy">
@@ -120,4 +148,11 @@
             <state_interface name="effort"/>
         </joint>
+        <transmission name="transmissionRFy">
+            <plugin>transmission_interface/SimpleTransmission</plugin>
+            <joint name="RFy" role="joint5">
+                <mechanical_reduction>200.0</mechanical_reduction>
+                <offset>0.0</offset>
+            </joint>
+        </transmission>
         <!-- Right foot X axis rotation control-->
         <joint name="RFx">
@@ -138,4 +173,11 @@
             <state_interface name="effort"/>
         </joint>
+        <transmission name="transmissionRFx">
+            <plugin>transmission_interface/SimpleTransmission</plugin>
+            <joint name="RFx" role="joint6">
+                <mechanical_reduction>200.0</mechanical_reduction>
+                <offset>0.0</offset>
+            </joint>
+        </transmission>
         <!-- Left thigh z axis rotation control-->
         <joint name="LTz">
@@ -156,4 +198,11 @@
             <state_interface name="effort"/>
         </joint>
+        <transmission name="transmissionLTz">
+            <plugin>transmission_interface/SimpleTransmission</plugin>
+            <joint name="LTz" role="joint7">
+                <mechanical_reduction>200.0</mechanical_reduction>
+                <offset>0.0</offset>
+            </joint>
+        </transmission>
         <!--Left thigh x axis rotation control -->
         <joint name="LTx">
@@ -174,4 +223,11 @@
             <state_interface name="effort"/>
         </joint>
+        <transmission name="transmissionLTx">
+            <plugin>transmission_interface/SimpleTransmission</plugin>
+            <joint name="LTx" role="joint8">
+                <mechanical_reduction>200.0</mechanical_reduction>
+                <offset>0.0</offset>
+            </joint>
+        </transmission>
         <!-- Left thigh y axis rotation control-->
         <joint name="LTy">
@@ -194,4 +250,11 @@
             <state_interface name="effort"/>
         </joint>
+        <transmission name="transmissionLTy">
+            <plugin>transmission_interface/SimpleTransmission</plugin>
+            <joint name="LTy" role="joint9">
+                <mechanical_reduction>200.0</mechanical_reduction>
+                <offset>0.0</offset>
+            </joint>
+        </transmission>
         <!-- Left shank y axis rotation control-->
         <joint name="LSy">
@@ -212,4 +275,11 @@
             <state_interface name="effort"/>
         </joint>
+        <transmission name="transmissionLSy">
+            <plugin>transmission_interface/SimpleTransmission</plugin>
+            <joint name="LSy" role="joint10">
+                <mechanical_reduction>200.0</mechanical_reduction>
+                <offset>0.0</offset>
+            </joint>
+        </transmission>
         <!-- Left foot y axis rotation control-->
         <joint name="LFy">
@@ -230,4 +300,11 @@
             <state_interface name="effort"/>
         </joint>
+        <transmission name="transmissionLFy">
+            <plugin>transmission_interface/SimpleTransmission</plugin>
+            <joint name="LFy" role="joint11">
+                <mechanical_reduction>200.0</mechanical_reduction>
+                <offset>0.0</offset>
+            </joint>
+        </transmission>
         <!--Left foot x axis rotation control -->
         <joint name="LFx">
@@ -248,4 +325,11 @@
             <state_interface name="effort"/>
         </joint>
+        <transmission name="transmissionLFx">
+            <plugin>transmission_interface/SimpleTransmission</plugin>
+            <joint name="LFx" role="joint12">
+                <mechanical_reduction>200.0</mechanical_reduction>
+                <offset>0.0</offset>
+            </joint>
+        </transmission>
         <!-- Right arm y axis rotation control -->
         <joint name="RAy">
@@ -266,4 +350,11 @@
             <state_interface name="effort"/>
         </joint>
+        <transmission name="transmissionRAy">
+            <plugin>transmission_interface/SimpleTransmission</plugin>
+            <joint name="RAy" role="joint16">
+            <mechanical_reduction>193.0</mechanical_reduction>
+            <offset>0.0</offset>
+            </joint>
+        </transmission>
         <!-- Right arm x axis rotation control-->
         <joint name="RAx">
@@ -284,4 +375,11 @@
             <state_interface name="effort"/>
         </joint>
+        <transmission name="transmissionRAx">
+            <plugin>transmission_interface/SimpleTransmission</plugin>
+            <joint name="RAx" role="joint17">
+            <mechanical_reduction>193.0</mechanical_reduction>
+            <offset>0.0</offset>
+            </joint>
+        </transmission>
         <!-- Roght forearm y axis rotation control-->
         <joint name="RFAy">
@@ -302,4 +400,11 @@
             <state_interface name="effort"/>
         </joint>
+        <transmission name="transmissionRFAy">
+            <plugin>transmission_interface/SimpleTransmission</plugin>
+            <joint name="RFAy" role="joint18">
+            <mechanical_reduction>193.0</mechanical_reduction>
+            <offset>0.0</offset>
+            </joint>
+        </transmission>
         <!--Left arm y axis rotation control -->
         <joint name="LAy">
@@ -320,4 +425,11 @@
             <state_interface name="effort"/>
         </joint>
+        <transmission name="transmissionLAy">
+            <plugin>transmission_interface/SimpleTransmission</plugin>
+            <joint name="LAy" role="joint13">
+            <mechanical_reduction>193.0</mechanical_reduction>
+            <offset>0.0</offset>
+            </joint>
+        </transmission>
         <!-- Left arm x axis rotation control -->
         <joint name="LAx">
@@ -338,4 +450,11 @@
             <state_interface name="effort"/>
         </joint>
+        <transmission name="transmissionLAx">
+            <plugin>transmission_interface/SimpleTransmission</plugin>
+            <joint name="LAx" role="joint14">
+            <mechanical_reduction>193.0</mechanical_reduction>
+            <offset>0.0</offset>
+            </joint>
+        </transmission>
         <!-- Left forearm y axis rotation control -->
         <joint name="LFAy">
@@ -356,4 +475,11 @@
             <state_interface name="effort"/>
         </joint>
+        <transmission name="transmissionLFAy">
+            <plugin>transmission_interface/SimpleTransmission</plugin>
+            <joint name="LFAy" role="joint15">
+            <mechanical_reduction>193.0</mechanical_reduction>
+            <offset>0.0</offset>
+            </joint>
+        </transmission>
         <!-- Head z axis rotation control-->
         <xacro:if value="$(arg use_gazebo)">

File: description/RobotElements/HeadElems/Head.xacro (robot description, xacro)
@@ -26,7 +26,7 @@
         </collision>
         <inertial>
-            <origin xyz="0.022e-3 0.28e-3 11.283e-3" rpy="0 0 0"/>
-            <mass value="0.077"/>
-            <inertia ixx="22.035e-6" iyy="18.242e-6" izz="13.649e-6" ixy="-0.008e-6" ixz="-0.02e-6"  iyz="0.689e-6"/>
+            <origin xyz="3.387e-3 0.317e-3 11.04e-3" rpy="0 0 0"/>
+            <mass value="0.092"/>
+            <inertia ixx="31.574e-6" iyy="28.238e-6" izz="23.684e-6" ixy="-0.065e-6" ixz="0.362e-6"  iyz="0.693e-6"/>
         </inertial>
     </link>

File: description/RobotElements/LeftArmElems/Larm.xacro (robot description, xacro)
@@ -6,5 +6,5 @@
         <child link="Left_Arm"/>
         <axis xyz="1.0 0 0"/>
-        <limit lower="${-pi/2}" upper="${pi/2}" effort="${maxeffort_val}" velocity="${maxVel_val}"/>
+        <limit lower="${-pi/2}" upper="${pi/2}" effort="${MX28maxeffort_val}" velocity="${MX28maxVel_val}"/>
         <xacro:if value="$(arg use_URDF_joint_dynamics_coefficients)">
             <dynamics damping="${damping_val}" friction="${friction_val}"/>
@@ -26,7 +26,7 @@
         </collision>
         <inertial>
-            <origin xyz="0.152e-3 -0.087e-3 -49.855e-3" rpy="0 0 0"/>
-            <mass value="0.165"/>
-            <inertia ixx="269.772e-6" iyy="269.138e-6" izz="29.837e-6" ixy="-0.02e-6" ixz="-1.454e-6"  iyz="-0.269e-6"/>
+            <origin xyz="0.144e-3 -0.082e-3 -57.405e-3" rpy="0 0 0"/>
+            <mass value="0.174"/>
+            <inertia ixx="371.391e-6" iyy="370.895e-6" izz="31.634e-6" ixy="-0.019e-6" ixz="-1.591e-6"  iyz="-0.374e-6"/>
         </inertial>
     </link>

File: description/RobotElements/LeftArmElems/Larmmount.xacro (robot description, xacro)
@@ -6,5 +6,5 @@
         <child link="Left_ArmMounting"/>
         <axis xyz="0 1.0 0"/>
-        <limit lower="${-pi/2}" upper="${pi/2}" effort="${maxeffort_val}" velocity="${maxVel_val}"/>
+        <limit lower="${-pi/2}" upper="${pi/2}" effort="${MX28maxeffort_val}" velocity="${MX28maxVel_val}"/>
         <xacro:if value="$(arg use_URDF_joint_dynamics_coefficients)">
             <dynamics damping="${damping_val}" friction="${friction_val}"/>

File: description/RobotElements/LeftArmElems/Lforearm.xacro (robot description, xacro)
@@ -6,5 +6,5 @@
         <child link="Left_Forearm"/>
         <axis xyz="0 1.0 0"/>
-        <limit lower="${-pi/2}" upper="${pi/2}" effort="${maxeffort_val}" velocity="${maxVel_val}"/>
+        <limit lower="${-pi/2}" upper="${pi/2}" effort="${MX28maxeffort_val}" velocity="${MX28maxVel_val}"/>
         <xacro:if value="$(arg use_URDF_joint_dynamics_coefficients)">
             <dynamics damping="${damping_val}" friction="${friction_val}"/>
@@ -26,7 +26,7 @@
         </collision>
         <inertial>
-            <origin xyz="0 0 -93.816e-3" rpy="0 0 0"/>
-            <mass value="0.094"/>
-            <inertia ixx="228.969e-6" iyy="231.48e-6" izz="16.247e-6" ixy="0" ixz="0"  iyz="0.002e-6"/>
+            <origin xyz="0 0.058e-3 -72.17e-3" rpy="0 0 0"/>
+            <mass value="0.057"/>
+            <inertia ixx="82.13e-6" iyy="83.135e-6" izz="11.456e-6" ixy="0" ixz="0"  iyz="-0.113e-6"/>
         </inertial>
     </link>

File: description/RobotElements/LeftLegElems/Lankle.xacro (robot description, xacro)
@@ -26,7 +26,7 @@
       </collision>
       <inertial>
-        <origin xyz="-21.137e-3	0.17e-3	14.739e-3" rpy="0 0 0"/>
-        <mass value="0.351"/>
-        <inertia ixx="135.823e-6" iyy="317.524e-6" izz="266.663e-6" ixy="-1.265e-6" ixz="4.25e-6"  iyz="2.029e-6" />
+        <origin xyz="-20.881e-3	0.167e-3	14.849e-3" rpy="0 0 0"/>
+        <mass value="0.294"/>
+        <inertia ixx="115.377e-6" iyy="266.21e-6" izz="222.99e-6" ixy="-1.023e-6" ixz="4.663e-6"  iyz="1.655e-6" />
       </inertial>
     </link>

File: description/RobotElements/LeftLegElems/Lfoot.xacro (robot description, xacro)
@@ -27,7 +27,7 @@
       </collision>
       <inertial>
-        <origin xyz="-4.442e-3	0	-30.98e-3" rpy="0 0 0"/>
-        <mass value="0.088"/>
-        <inertia ixx="42.902e-6" iyy="138.102e-6" izz="160.902e-6" ixy="0" ixz="-0.647e-6"  iyz="0" />
+        <origin xyz="-5.077e-3	0	-30.402e-3" rpy="0 0 0"/>
+        <mass value="0.075"/>
+        <inertia ixx="35.802e-6" iyy="118.503e-6" izz="135.531e-6" ixy="0" ixz="-1.108e-6"  iyz="0" />
       </inertial>
     </link>

File: description/RobotElements/LeftLegElems/Lhip.xacro (robot description, xacro)
@@ -27,7 +27,7 @@
       </collision>
       <inertial>
-        <origin xyz="-21.137e-3	0.17e-3	14.739e-3" rpy="0 0 0"/>
-        <mass value="0.351"/>
-        <inertia ixx="135.823e-6" iyy="317.524e-6" izz="266.663e-6" ixy="-1.265e-6" ixz="4.25e-6"  iyz="2.029e-6" />
+        <origin xyz="-20.881e-3	-0.167e-3	-14.849e-3" rpy="0 0 0"/>
+        <mass value="0.294"/>
+        <inertia ixx="115.377e-6" iyy="266.21e-6" izz="222.99e-6" ixy="1.023e-6" ixz="-4.663e-6"  iyz="1.655e-6" />
       </inertial>
     </link>

File: description/RobotElements/LeftLegElems/Lhipmount.xacro (robot description, xacro)
@@ -28,7 +28,7 @@
     </collision>
     <inertial>
-      <origin xyz="-14.306e-3	0	24.769e-3" rpy="0 0 0"/>
-      <mass value="0.038"/>
-      <inertia ixx="11.743e-6" iyy="61.298e-6" izz="58.734e-6" ixy="0" ixz="4.429e-6"  iyz="0" />
+      <origin xyz="-13.999e-3	0	24.592e-3" rpy="0 0 0"/>
+      <mass value="0.036"/>
+      <inertia ixx="11.125e-6" iyy="57.759e-6" izz="55.215e-6" ixy="0" ixz="4.397e-6"  iyz="0" />
     </inertial>
   </link>

File: description/RobotElements/LeftLegElems/Lthigh.xacro (robot description, xacro)
@@ -26,7 +26,7 @@
       </collision>
       <inertial>
-        <origin xyz="2.335e-3	0.65e-3	-99.757e-3" rpy="0 0 0"/>
-        <mass value="0.22"/>
-        <inertia ixx="275.661e-6" iyy="250.206e-6" izz="77.57e-6" ixy="0.334e-6" ixz="-7.878e-6"  iyz="-5.455e-6" />
+        <origin xyz="2.704e-3	0.696e-3 -97.695e-3" rpy="0 0 0"/>
+        <mass value="0.19"/>
+        <inertia ixx="257.406e-6" iyy="233.803e-6" izz="70.376e-6" ixy="0.357e-6" ixz="-6.819e-6"  iyz="-5.699e-6" />
       </inertial>
     </link>

File: description/RobotElements/RightArmElems/Rarm.xacro (robot description, xacro)
@@ -6,5 +6,5 @@
         <child link="Right_Arm"/>
         <axis xyz="1.0 0 0"/>
-        <limit lower="${-pi/2}" upper="${pi/2}" effort="${maxeffort_val}" velocity="${maxVel_val}"/>
+        <limit lower="${-pi/2}" upper="${pi/2}" effort="${MX28maxeffort_val}" velocity="${MX28maxVel_val}"/>
         <xacro:if value="$(arg use_URDF_joint_dynamics_coefficients)">
             <dynamics damping="${damping_val}" friction="${friction_val}"/>
@@ -26,7 +26,7 @@
         </collision>
         <inertial>
-            <origin xyz="0.152e-3 -0.087e-3 -49.855e-3" rpy="0 0 0"/>
-            <mass value="0.165"/>
-            <inertia ixx="269.772e-6" iyy="269.138e-6" izz="29.837e-6" ixy="-0.02e-6" ixz="-1.454e-6"  iyz="-0.269e-6"/>
+            <origin xyz="0.144e-3 -0.082e-3 -57.405e-3" rpy="0 0 0"/>
+            <mass value="0.174"/>
+            <inertia ixx="371.391e-6" iyy="370.895e-6" izz="31.634e-6" ixy="-0.019e-6" ixz="-1.591e-6"  iyz="-0.374e-6"/>
         </inertial>
     </link>

File: description/RobotElements/RightArmElems/Rarmmount.xacro (robot description, xacro)
@@ -6,5 +6,5 @@
         <child link="Right_ArmMounting"/>
         <axis xyz="0 1.0 0"/>
-        <limit lower="${-pi/2}" upper="${pi/2}" effort="${maxeffort_val}" velocity="${maxVel_val}"/>
+        <limit lower="${-pi/2}" upper="${pi/2}" effort="${MX28maxeffort_val}" velocity="${MX28maxVel_val}"/>
         <xacro:if value="$(arg use_URDF_joint_dynamics_coefficients)">
             <dynamics damping="${damping_val}" friction="${friction_val}"/>

File: description/RobotElements/RightArmElems/Rforearm.xacro (robot description, xacro)
@@ -6,5 +6,5 @@
         <child link="Right_Forearm"/>
         <axis xyz="0 1.0 0"/>
-        <limit lower="${-pi/2}" upper="${pi/2}" effort="${maxeffort_val}" velocity="${maxVel_val}"/>
+        <limit lower="${-pi/2}" upper="${pi/2}" effort="${MX28maxeffort_val}" velocity="${MX28maxVel_val}"/>
         <xacro:if value="$(arg use_URDF_joint_dynamics_coefficients)">
             <dynamics damping="${damping_val}" friction="${friction_val}"/>
@@ -26,7 +26,7 @@
         </collision>
         <inertial>
-            <origin xyz="0 0 -93.816e-3" rpy="0 0 0"/>
-            <mass value="0.094"/>
-            <inertia ixx="228.969e-6" iyy="231.48e-6" izz="16.247e-6" ixy="0" ixz="0"  iyz="0.002e-6"/>
+            <origin xyz="0 -0.059e-3 -72.17e-3" rpy="0 0 0"/>
+            <mass value="0.057"/>
+            <inertia ixx="82.13e-6" iyy="83.135e-6" izz="11.456e-6" ixy="0" ixz="0"  iyz="0.116e-6"/>
         </inertial>
     </link>

File: description/RobotElements/RightLegElems/Rankle.xacro (robot description, xacro)
@@ -28,7 +28,7 @@
         </collision>
         <inertial>
-            <origin xyz="-21.137e-3	0.17e-3	14.739e-3" rpy="0 0 0"/>
-            <mass value="0.351"/>
-            <inertia ixx="135.823e-6" iyy="317.524e-6" izz="266.663e-6" ixy="-1.265e-6" ixz="4.25e-6"  iyz="2.029e-6" />
+            <origin xyz="-20.881e-3	0.167e-3 14.849e-3" rpy="0 0 0"/>
+            <mass value="0.294"/>
+            <inertia ixx="115.377e-6" iyy="266.21e-6" izz="222.99e-6" ixy="-1.023e-6" ixz="4.663e-6"  iyz="1.655e-6" />
         </inertial>
     </link>

File: description/RobotElements/RightLegElems/Rfoot.xacro (robot description, xacro)
@@ -26,7 +26,7 @@
         </collision>
         <inertial>
-            <origin xyz="-4.442e-3	0	-30.98e-3" rpy="0 0 0"/>
-            <mass value="0.088"/>
-            <inertia ixx="42.902e-6" iyy="138.102e-6" izz="160.902e-6" ixy="0" ixz="-0.647e-6"  iyz="0" />
+            <origin xyz="-5.077e-3	0	-30.402e-3" rpy="0 0 0"/>
+            <mass value="0.075"/>
+            <inertia ixx="35.802e-6" iyy="118.503e-6" izz="135.531e-6" ixy="0" ixz="-1.108e-6"  iyz="0" />
         </inertial>
     </link>

File: description/RobotElements/RightLegElems/Rhip.xacro (robot description, xacro)
@@ -26,7 +26,7 @@
         </collision>
         <inertial>
-            <origin xyz="-21.137e-06 0.17e-03 14.739e-03" rpy="0 0 0"/>
-            <mass value="0.351"/>
-            <inertia ixx="135.823e-6" iyy="317.524e-6" izz="266.663e-6" ixy="-1.265e-6" ixz="4.25e-6"  iyz="2.029e-6" />
+            <origin xyz="-20.881e-3	-0.167e-3	-14.849e-3" rpy="0 0 0"/>
+            <mass value="0.294"/>
+            <inertia ixx="115.377e-6" iyy="266.21e-6" izz="222.99e-6" ixy="1.023e-6" ixz="-4.663e-6"  iyz="1.655e-6" />
         </inertial>
     </link>

File: description/RobotElements/RightLegElems/Rhipmount.xacro (robot description, xacro)
@@ -26,7 +26,7 @@
         </collision>
         <inertial>
-            <origin xyz="-14.306e-03 0 24.769e-03" rpy="0 0 0"/>
-            <mass value="0.038"/>
-            <inertia ixx="11.743e-6" iyy="61.298e-6" izz="58.734e-6" ixy="0" ixz="4.429e-6" iyz="0"/>
+            <origin xyz="-13.999e-3	0	24.592e-3" rpy="0 0 0"/>
+            <mass value="0.036"/>
+            <inertia ixx="11.125e-6" iyy="57.759e-6" izz="55.215e-6" ixy="0" ixz="4.397e-6"  iyz="0" />
         </inertial>
     </link>

File: description/RobotElements/RightLegElems/Rthigh.xacro (robot description, xacro)
@@ -26,7 +26,7 @@
         </collision>
         <inertial>
-            <origin xyz="2.335e-3	0.65e-3	-99.757e-3" rpy="0 0 0"/>
-            <mass value="0.22"/>
-            <inertia ixx="275.661e-6" iyy="250.206e-6" izz="77.57e-6" ixy="0.334e-6" ixz="-7.878e-6"  iyz="-5.455e-6" />
+            <origin xyz="2.704e-3	0.696e-3 -97.695e-3" rpy="0 0 0"/>
+            <mass value="0.19"/>
+            <inertia ixx="257.406e-6" iyy="233.803e-6" izz="70.376e-6" ixy="0.357e-6" ixz="-6.819e-6"  iyz="-5.699e-6" />
         </inertial>
     </link>

File: description/RobotElements/Trunk.xacro (robot description, xacro)
@@ -18,7 +18,7 @@
     </visual>
     <inertial>
-      <origin xyz="-7.709e-3	-0.06e-3	-57.629e-3" rpy="0 0 0"/>
-      <mass value="0.691"/>
-      <inertia ixx="1992.6e-6" iyy="1287.385e-6" izz="1142.314e-6" ixy="0.546e-6" ixz="-217.49e-6"  iyz="1.946e-6" />
+      <origin xyz="-25.163e-3	-1.006e-3	-39.233e-3" rpy="0 0 0"/>
+      <mass value="1.282"/>
+      <inertia ixx="3554.642e-6" iyy="3113.534e-6" izz="2635.241e-6" ixy="-52.803e-6" ixz="364.587e-6"  iyz="16.6e-6" />
     </inertial>
     <collision>

File: description/imu.xacro (robot description, xacro)
@@ -22,5 +22,5 @@
             <mass value="0.009" />
             <origin xyz="0 0 0" rpy="0 0 0"/>
-            <inertia ixx="16.401e-6" ixy="0" ixz="0" iyy="36.818e-6" iyz="0" izz="53.083e-6" />
+            <inertia ixx="147.609e-9" ixy="0" ixz="0" iyy="331.362e-9" iyz="0" izz="477.747e-9" />
         </inertial>
     </link>
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