Commit message: Finished project. Melman Moves in gazebo gracefully wih trajectories given from txt files. Servomechanisms simulated properly

File: description/Melman_ros2control_gazebo.xacro (robot description, xacro)
@@ -383,5 +383,5 @@
         </transmission>
         <!-- Roght forearm y axis rotation control-->
-        <joint name="RFAy">
+        <!-- <joint name="RFAy">
             <param name="id">18</param>
             <command_interface name="position">
@@ -406,5 +406,5 @@
             <offset>0.0</offset>
             </joint>
-        </transmission>
+        </transmission> -->
         <!--Left arm y axis rotation control -->
         <joint name="LAy">
@@ -458,5 +458,5 @@
         </transmission>
         <!-- Left forearm y axis rotation control -->
-        <joint name="LFAy">
+        <!-- <joint name="LFAy">
             <param name="id">15</param>
             <command_interface name="position">
@@ -481,7 +481,7 @@
             <offset>0.0</offset>
             </joint>
-        </transmission>
+        </transmission> -->
         <!-- Head z axis rotation control-->
-        <xacro:if value="$(arg use_gazebo)">
+        <!-- <xacro:if value="$(arg use_gazebo)">
         <joint name="Hz">
             <param name="id">19</param>
@@ -501,7 +501,7 @@
             <state_interface name="effort"/>
         </joint>
-        </xacro:if>
+        </xacro:if> -->
         <!-- Head y axis rotation control-->
-        <xacro:if value="$(arg use_gazebo)">
+        <!-- <xacro:if value="$(arg use_gazebo)">
         <joint name="Hy">
             <param name="id">20</param>
@@ -521,5 +521,5 @@
             <state_interface name="effort"/>
         </joint>
-        </xacro:if>
+        </xacro:if> -->
     </ros2_control>
     <xacro:if value="$(arg use_gazebo)">

File: description/RobotElements/HeadElems/Head.xacro (robot description, xacro)
@@ -1,5 +1,5 @@
 <?xml version = "1.0"?>
 <robot xmlns:xacro="http://www.ros.org/wiki/xacro">
-    <joint name="Hy" type="revolute">
+    <joint name="Hy" type="fixed">
         <origin xyz="0 0 0" rpy="0 0 0"/>
         <parent link="Head_Mounting"/>

File: description/RobotElements/HeadElems/Headmount.xacro (robot description, xacro)
@@ -1,5 +1,5 @@
 <?xml version="1.0"?>
 <robot xmlns:xacro="http://www.ros.org/wiki/xacro">
-    <joint name="Hz" type="revolute">
+    <joint name="Hz" type="fixed">
         <origin xyz="18.1e-3 -0.159e-3 38.5e-3" rpy="0 0 0"/>
         <parent link="Trunk"/>

File: description/RobotElements/LeftArmElems/Larm.xacro (robot description, xacro)
@@ -6,7 +6,7 @@
         <child link="Left_Arm"/>
         <axis xyz="-1.0 0 0"/>
-        <limit lower="${-pi/2}" upper="${pi/2}" effort="${MX28maxeffort_val}" velocity="${MX28maxVel_val}"/>
+        <limit lower="${-pi}" upper="${pi}" effort="${MX28maxeffort_val}" velocity="${MX28maxVel_val}"/>
         <xacro:if value="$(arg use_URDF_joint_dynamics_coefficients)">
-            <dynamics damping="${damping_val}" friction="${friction_val}"/>
+            <dynamics damping="${damping_valMX28}" friction="${friction_valMX28}"/>
         </xacro:if>
     </joint>
@@ -33,9 +33,9 @@
     <xacro:if value="$(arg use_gazebo_joint_physics_coefficients)">
     <gazebo reference="LAx">
-        <implicitSpringDamper>${Damper_val}</implicitSpringDamper>
-        <springStiffness>${springstiffness_val}</springStiffness>
-        <springReference>${springReference_val}</springReference>
-        <stopErp>${stopErp_val}</stopErp>
-        <stopCfm>${stopCfm_val}</stopCfm>
+        <implicitSpringDamper>${Damper_valMX28}</implicitSpringDamper>
+        <springStiffness>${springstiffness_valMX28}</springStiffness>
+        <springReference>${springReference_valMX28}</springReference>
+        <stopErp>${stopErp_valMX28}</stopErp>
+        <stopCfm>${stopCfm_valMX28}</stopCfm>
     </gazebo>
     </xacro:if>

File: description/RobotElements/LeftArmElems/Larmmount.xacro (robot description, xacro)
@@ -6,7 +6,7 @@
         <child link="Left_ArmMounting"/>
         <axis xyz="0 1.0 0"/>
-        <limit lower="${-pi/2}" upper="${pi/2}" effort="${MX28maxeffort_val}" velocity="${MX28maxVel_val}"/>
+        <limit lower="${-pi}" upper="${pi}" effort="${MX28maxeffort_val}" velocity="${MX28maxVel_val}"/>
         <xacro:if value="$(arg use_URDF_joint_dynamics_coefficients)">
-            <dynamics damping="${damping_val}" friction="${friction_val}"/>
+            <dynamics damping="${damping_valMX28}" friction="${friction_valMX28}"/>
         </xacro:if>
     </joint>
@@ -33,9 +33,9 @@
     <xacro:if value="$(arg use_gazebo_joint_physics_coefficients)">
     <gazebo reference="LAy">
-        <implicitSpringDamper>${Damper_val}</implicitSpringDamper>
-        <springStiffness>${springstiffness_val}</springStiffness>
-        <springReference>${springReference_val}</springReference>
-        <stopErp>${stopErp_val}</stopErp>
-        <stopCfm>${stopCfm_val}</stopCfm>
+        <implicitSpringDamper>${Damper_valMX28}</implicitSpringDamper>
+        <springStiffness>${springstiffness_valMX28}</springStiffness>
+        <springReference>${springReference_valMX28}</springReference>
+        <stopErp>${stopErp_valMX28}</stopErp>
+        <stopCfm>${stopCfm_valMX28}</stopCfm>
     </gazebo>
     </xacro:if>

File: description/RobotElements/LeftArmElems/Lforearm.xacro (robot description, xacro)
@@ -8,5 +8,5 @@
         <limit lower="${-pi/2}" upper="${pi/2}" effort="${MX28maxeffort_val}" velocity="${MX28maxVel_val}"/>
         <xacro:if value="$(arg use_URDF_joint_dynamics_coefficients)">
-            <dynamics damping="${damping_val}" friction="${friction_val}"/>
+            <dynamics damping="${damping_valMX28}" friction="${friction_valMX28}"/>
         </xacro:if>
     </joint>
@@ -33,9 +33,9 @@
     <xacro:if value="$(arg use_gazebo_joint_physics_coefficients)">
     <gazebo reference="LFAy">
-        <implicitSpringDamper>${Damper_val}</implicitSpringDamper>
-        <springStiffness>${springstiffness_val}</springStiffness>
-        <springReference>${springReference_val}</springReference>
-        <stopErp>${stopErp_val}</stopErp>
-        <stopCfm>${stopCfm_val}</stopCfm>
+        <implicitSpringDamper>${Damper_valMX28}</implicitSpringDamper>
+        <springStiffness>${springstiffness_valMX28}</springStiffness>
+        <springReference>${springReference_valMX28}</springReference>
+        <stopErp>${stopErp_valMX28}</stopErp>
+        <stopCfm>${stopCfm_valMX28}</stopCfm>
     </gazebo>
     </xacro:if>

File: description/RobotElements/RightArmElems/Rarm.xacro (robot description, xacro)
@@ -6,7 +6,7 @@
         <child link="Right_Arm"/>
         <axis xyz="-1.0 0 0"/>
-        <limit lower="${-pi/2}" upper="${pi/2}" effort="${MX28maxeffort_val}" velocity="${MX28maxVel_val}"/>
+        <limit lower="${-pi}" upper="${pi}" effort="${MX28maxeffort_val}" velocity="${MX28maxVel_val}"/>
         <xacro:if value="$(arg use_URDF_joint_dynamics_coefficients)">
-            <dynamics damping="${damping_val}" friction="${friction_val}"/>
+            <dynamics damping="${damping_valMX28}" friction="${friction_valMX28}"/>
         </xacro:if>
     </joint>
@@ -33,9 +33,9 @@
     <xacro:if value="$(arg use_gazebo_joint_physics_coefficients)">
     <gazebo reference="RAx">
-        <implicitSpringDamper>${Damper_val}</implicitSpringDamper>
-        <springStiffness>${springstiffness_val}</springStiffness>
-        <springReference>${springReference_val}</springReference>
-        <stopErp>${stopErp_val}</stopErp>
-        <stopCfm>${stopCfm_val}</stopCfm>
+        <implicitSpringDamper>${Damper_valMX28}</implicitSpringDamper>
+        <springStiffness>${springstiffness_valMX28}</springStiffness>
+        <springReference>${springReference_valMX28}</springReference>
+        <stopErp>${stopErp_valMX28}</stopErp>
+        <stopCfm>${stopCfm_valMX28}</stopCfm>
     </gazebo>
     </xacro:if>

File: description/RobotElements/RightArmElems/Rarmmount.xacro (robot description, xacro)
@@ -6,7 +6,7 @@
         <child link="Right_ArmMounting"/>
         <axis xyz="0 1.0 0"/>
-        <limit lower="${-pi/2}" upper="${pi/2}" effort="${MX28maxeffort_val}" velocity="${MX28maxVel_val}"/>
+        <limit lower="${-pi}" upper="${pi}" effort="${MX28maxeffort_val}" velocity="${MX28maxVel_val}"/>
         <xacro:if value="$(arg use_URDF_joint_dynamics_coefficients)">
-            <dynamics damping="${damping_val}" friction="${friction_val}"/>
+            <dynamics damping="${damping_valMX28}" friction="${friction_valMX28}"/>
         </xacro:if>
     </joint>
@@ -33,9 +33,9 @@
     <xacro:if value="$(arg use_gazebo_joint_physics_coefficients)">
     <gazebo reference="RAy">
-        <implicitSpringDamper>${Damper_val}</implicitSpringDamper>
-        <springStiffness>${springstiffness_val}</springStiffness>
-        <springReference>${springReference_val}</springReference>
-        <stopErp>${stopErp_val}</stopErp>
-        <stopCfm>${stopCfm_val}</stopCfm>
+        <implicitSpringDamper>${Damper_valMX28}</implicitSpringDamper>
+        <springStiffness>${springstiffness_valMX28}</springStiffness>
+        <springReference>${springReference_valMX28}</springReference>
+        <stopErp>${stopErp_valMX28}</stopErp>
+        <stopCfm>${stopCfm_valMX28}</stopCfm>
     </gazebo>
     </xacro:if>

File: description/RobotElements/RightArmElems/Rforearm.xacro (robot description, xacro)
@@ -8,5 +8,5 @@
         <limit lower="${-pi/2}" upper="${pi/2}" effort="${MX28maxeffort_val}" velocity="${MX28maxVel_val}"/>
         <xacro:if value="$(arg use_URDF_joint_dynamics_coefficients)">
-            <dynamics damping="${damping_val}" friction="${friction_val}"/>
+            <dynamics damping="${damping_valMX28}" friction="${friction_valMX28}"/>
         </xacro:if>
     </joint>
@@ -33,9 +33,9 @@
     <xacro:if value="$(arg use_gazebo_joint_physics_coefficients)">
     <gazebo reference="RFAy">
-        <implicitSpringDamper>${Damper_val}</implicitSpringDamper>
-        <springStiffness>${springstiffness_val}</springStiffness>
-        <springReference>${springReference_val}</springReference>
-        <stopErp>${stopErp_val}</stopErp>
-        <stopCfm>${stopCfm_val}</stopCfm>
+        <implicitSpringDamper>${Damper_valMX28}</implicitSpringDamper>
+        <springStiffness>${springstiffness_valMX28}</springStiffness>
+        <springReference>${springReference_valMX28}</springReference>
+        <stopErp>${stopErp_valMX28}</stopErp>
+        <stopCfm>${stopCfm_valMX28}</stopCfm>
     </gazebo>
     </xacro:if>

File: description/RobotElements/Trunk.xacro (robot description, xacro)
@@ -19,5 +19,5 @@
     <inertial>
       <origin xyz="-25.163e-3	-1.006e-3	-39.233e-3" rpy="0 0 0"/>
-      <mass value="1.282"/>
+      <mass value="1.569"/>
       <inertia ixx="3554.642e-6" iyy="3113.534e-6" izz="2635.241e-6" ixy="-52.803e-6" ixz="364.587e-6"  iyz="16.6e-6" />
     </inertial>

File: description/imu.xacro (robot description, xacro)
@@ -2,6 +2,9 @@
 <robot xmlns:xacro="http://www.ros.org/wiki/xacro">
     <joint name="imu_sensor_joint" type="fixed">
-        <origin xyz="0.0 -0.016 -0.057" rpy="${pi/2} ${pi/2} 0"/>
-        <parent link="Right_Arm"/>
+        <origin xyz="${31.505-0.790}e-3 ${-40.249+39.898}e-3 ${-231.798+278.063-128}e-3" rpy="${pi/2} ${(pi/2-0.99)-pi/2} ${pi/2}"/>
+        <!-- BEBECH <origin xyz="28e-3 -0.048e-3 -47.018e-3" rpy="${pi/2} ${pi/2} 0"/> -->
+        <!-- ARM RANDOM LOCALIZATION<origin xyz="0.0 -0.016 -0.057" rpy="${pi/2} ${pi/2} 0"/> -->
+        <!-- ARM Precise localization<origin xyz="${-1*(0-0.353)}e-3 ${-1*(88.341-105.341)}e-3 ${-1*(0+57.104)}e-3" rpy="${-pi/2} ${pi/4} 0"/> -->
+        <parent link="Right_Thigh"/>
         <child link="imu"/>
     </joint>

File: description/robot_core.xacro (robot description, xacro)
@@ -9,13 +9,22 @@
   <xacro:property name="dampigFactor_val" value="0.004"/>
   <xacro:property name="selfCollide_val" value="true"/>
-  <!-- Definition of GAZEBO physics coefficients for all JOINTS -->
+  <!-- Definition of GAZEBO physics coefficients for JOINTS powered by MX64AR servos-->
   <xacro:property name="Damper_val" value="true"/>
-  <xacro:property name="springstiffness_val" value="6.0"/>
-  <xacro:property name="springReference_val" value="0.01"/>
+  <xacro:property name="springstiffness_val" value="0.5"/>
+  <xacro:property name="springReference_val" value="0.061"/>
   <xacro:property name="stopErp_val" value="0.2"/>
-  <xacro:property name="stopCfm_val" value="0.2"/>
-  <!-- Definition of URDF physics coefficients for all JOINTS -->
-  <xacro:property name="damping_val" value="1.0"/>
-  <xacro:property name="friction_val" value="1.0"/>
+  <xacro:property name="stopCfm_val" value="0.45"/>
+  <!-- Definition of GAZEBO physics coefficients for JOINTS powered by MX28AR servos-->
+  <xacro:property name="Damper_valMX28" value="true"/>
+  <xacro:property name="springstiffness_valMX28" value="0.5"/>
+  <xacro:property name="springReference_valMX28" value="0.061"/>
+  <xacro:property name="stopErp_valMX28" value="0.7"/>
+  <xacro:property name="stopCfm_valMX28" value="0.45"/>
+  <!-- Definition of URDF physics coefficients for JOINTS powered by MX64AR servos-->
+  <xacro:property name="damping_val" value="0.5"/>
+  <xacro:property name="friction_val" value="1.788"/>
+  <!-- Definition of URDF physics coefficients for JOINTS powered by MX28AR servos-->
+  <xacro:property name="damping_valMX28" value="0.5"/>
+  <xacro:property name="friction_valMX28" value="1.288"/>
   <!-- Definition of URDF physics coefficients for JOINTS powered by MX64AR servos-->
   <xacro:property name="maxVel_val" value="6.597"/>
