Commit message: Changed the .stl files to fresh ones, and scaled them properly

File: description/RobotElements/Trunk.xacro (robot description, xacro)
@@ -13,5 +13,5 @@
       <origin xyz="0 0 0" rpy="0 0 0"/>
       <geometry>
-        <mesh filename="file://$(find ros2_humanoid_virtual_twin)/meshes/Trunk.stl"/>
+        <mesh filename="file://$(find ros2_humanoid_virtual_twin)/meshes/Trunk.stl" scale="0.001 0.001 0.001"/>
       </geometry>
       <material name="grey"/>
@@ -25,5 +25,5 @@
       <origin xyz="0 0 0" rpy="0 0 0"/>
       <geometry>
-        <mesh filename="file://$(find ros2_humanoid_virtual_twin)/meshes/Trunk-Collision.stl"/>
+        <mesh filename="file://$(find ros2_humanoid_virtual_twin)/meshes/Trunk-Collision.stl" scale="0.001 0.001 0.001"/>
       </geometry>
     </collision>

Commit message: Added new collision mesh for trunk and acutalized the rviz launchfile for new URDF

File: description/RobotElements/Trunk.xacro (robot description, xacro)
@@ -23,8 +23,7 @@
     </inertial>
     <collision>
-      <origin xyz="0 0 -45e-3" rpy="0 0 0"/>
+      <origin xyz="0 0 0" rpy="0 0 0"/>
       <geometry>
-        <!-- <mesh filename="file://$(find ros2_humanoid_virtual_twin)/meshes/Trunk-Collision.stl" scale="0.001 0.001 0.001"/> -->
-        <box size="0.14 0.1 0.1"/>
+        <mesh filename="file://$(find ros2_humanoid_virtual_twin)/meshes/Trunk_Collision.stl" scale="0.001 0.001 0.001"/>
       </geometry>
     </collision>
