Commit message: added collisions back to forearms and more gyroscopic paramters

File: description/RobotElements/LeftArmElems/Lforearm.xacro (robot description, xacro)
@@ -19,10 +19,10 @@
             <material name="grey"/>
         </visual>
-        <!-- <collision>
+        <collision>
             <origin xyz="0 0 0" rpy="0 0 0"/>
             <geometry>
                 <mesh filename="file://$(find ros2_humanoid_virtual_twin)/meshes/Right_Forearm.stl" scale="0.001 0.001 0.001"/>
             </geometry>
-        </collision> -->
+        </collision>
         <inertial>
             <origin xyz="0 0 -93.816e-3" rpy="0 0 0"/>
@@ -42,5 +42,5 @@
     <gazebo reference="Left_Forearm">
         <material>Gazebo/Grey</material>
-        <!-- <xacro:if value="$(arg use_gazebo_link_physics_coefficients)">
+        <xacro:if value="$(arg use_gazebo_link_physics_coefficients)">
           <mu1 value="${mu1_val}"/>
           <mu2 value="${mu2_val}"/>
@@ -50,5 +50,5 @@
           <dampingFactor value="${dampigFactor_val}"/>
           <selfCollide>${selfCollide_val}</selfCollide>
-        </xacro:if> -->
+        </xacro:if>
     </gazebo>
 </robot>

File: description/RobotElements/RightArmElems/Rforearm.xacro (robot description, xacro)
@@ -19,10 +19,10 @@
             <material name="grey"/>
         </visual>
-        <!-- <collision>
+        <collision>
             <origin xyz="0 0 0" rpy="0 0 0"/>
             <geometry>
                 <mesh filename="file://$(find ros2_humanoid_virtual_twin)/meshes/Right_Forearm.stl" scale="0.001 0.001 0.001"/>
             </geometry>
-        </collision> -->
+        </collision>
         <inertial>
             <origin xyz="0 0 -93.816e-3" rpy="0 0 0"/>
@@ -42,5 +42,5 @@
     <gazebo reference="Right_Forearm">
         <material>Gazebo/Grey</material>
-        <!-- <xacro:if value="$(arg use_gazebo_link_physics_coefficients)">
+        <xacro:if value="$(arg use_gazebo_link_physics_coefficients)">
           <mu1 value="${mu1_val}"/>
           <mu2 value="${mu2_val}"/>
@@ -50,5 +50,5 @@
           <dampingFactor value="${dampigFactor_val}"/>
           <selfCollide>${selfCollide_val}</selfCollide>
-        </xacro:if> -->
+        </xacro:if>
     </gazebo>
 </robot>

File: description/imu.xacro (robot description, xacro)
@@ -5,5 +5,4 @@
         <parent link="Right_Arm"/>
         <child link="imu"/>
-        <dynamics damping="0.0" friction="0.0"/>
     </joint>
     <link name="imu">
@@ -27,7 +26,9 @@
     </link>
     <gazebo reference="imu">
+        <!-- <gravity>true</gravity> -->
         <sensor name="MPU6050sensor" type="imu">
             <always_on>1</always_on>
-            <update_rate>10.0</update_rate>
+            <update_rate>40.0</update_rate>
+            <!-- <visualize>true</visualize> -->
         </sensor>
     </gazebo>
