Commit message: Solved collision problems

File: description/RobotElements/LeftArmElems/Larm.xacro (robot description, xacro)
@@ -19,5 +19,5 @@
             <origin xyz="0 0 0" rpy="0 0 0"/>
             <geometry>
-                <mesh filename="file://$(find ros2_humanoid_virtual_twin)/meshes/Left-Arm-Collision.stl" scale="0.001 0.001 0.001"/>
+                <mesh filename="file://$(find ros2_humanoid_virtual_twin)/meshes/Left-Arm-Collision.stl"/>
             </geometry>
         </collision>

File: description/RobotElements/LeftArmElems/Lforearm.xacro (robot description, xacro)
@@ -19,5 +19,5 @@
             <origin xyz="0 0 0" rpy="0 0 0"/>
             <geometry>
-                <mesh filename="file://$(find ros2_humanoid_virtual_twin)/meshes/Left-Forearm-collision.stl" scale="0.001 0.001 0.001"/>
+                <mesh filename="file://$(find ros2_humanoid_virtual_twin)/meshes/Right_Forearm.stl" scale="0.001 0.001 0.001"/>
             </geometry>
         </collision>

File: description/RobotElements/RightArmElems/Rarm.xacro (robot description, xacro)
@@ -19,5 +19,5 @@
             <origin xyz="0 0 0" rpy="0 0 0"/>
             <geometry>
-                <mesh filename="file://$(find ros2_humanoid_virtual_twin)/meshes/Left-Arm-Collision.stl" scale="0.001 0.001 0.001"/>
+                <mesh filename="file://$(find ros2_humanoid_virtual_twin)/meshes/Left-Arm-Collision.stl"/>
             </geometry>
         </collision>

File: description/RobotElements/RightArmElems/Rforearm.xacro (robot description, xacro)
@@ -19,5 +19,5 @@
             <origin xyz="0 0 0" rpy="0 0 0"/>
             <geometry>
-                <mesh filename="file://$(find ros2_humanoid_virtual_twin)/meshes/Left-Forearm-collision.stl" scale="0.001 0.001 0.001"/>
+                <mesh filename="file://$(find ros2_humanoid_virtual_twin)/meshes/Right_Forearm.stl" scale="0.001 0.001 0.001"/>
             </geometry>
         </collision>

Commit message: Corrected axis orientation to the real robot and deleted old trajectories

File: description/RobotElements/LeftArmElems/Larm.xacro (robot description, xacro)
@@ -5,5 +5,5 @@
         <parent link="Left_ArmMounting"/>
         <child link="Left_Arm"/>
-        <axis xyz="1.0 0 0"/>
+        <axis xyz="-1.0 0 0"/>
         <limit lower="${-pi/2}" upper="${pi/2}" effort="${MX28maxeffort_val}" velocity="${MX28maxVel_val}"/>
         <xacro:if value="$(arg use_URDF_joint_dynamics_coefficients)">

File: description/RobotElements/LeftArmElems/Lforearm.xacro (robot description, xacro)
@@ -5,5 +5,5 @@
         <parent link="Left_Arm"/>
         <child link="Left_Forearm"/>
-        <axis xyz="0 1.0 0"/>
+        <axis xyz="0 -1.0 0"/>
         <limit lower="${-pi/2}" upper="${pi/2}" effort="${MX28maxeffort_val}" velocity="${MX28maxVel_val}"/>
         <xacro:if value="$(arg use_URDF_joint_dynamics_coefficients)">

File: description/RobotElements/LeftLegElems/Lankle.xacro (robot description, xacro)
@@ -5,5 +5,5 @@
       <parent link="Left_Shank"/>
       <child link="Left_Ankle"/>
-      <axis xyz="0 1.0 0"/>
+      <axis xyz="0 -1.0 0"/>
       <limit lower="${-pi/2}" upper="${pi/2}" effort="${maxeffort_val}" velocity="${maxVel_val}"/>
       <xacro:if value="$(arg use_URDF_joint_dynamics_coefficients)">

File: description/RobotElements/LeftLegElems/Lfoot.xacro (robot description, xacro)
@@ -5,5 +5,5 @@
       <parent link="Left_Ankle"/>
       <child link="Left_Foot"/>
-      <axis xyz="1.0 0 0"/>
+      <axis xyz="-1.0 0 0"/>
       <limit lower="${-pi/2}" upper="${pi/2}" effort="${maxeffort_val}" velocity="${maxVel_val}"/>
       <xacro:if value="$(arg use_URDF_joint_dynamics_coefficients)">

File: description/RobotElements/LeftLegElems/Lhip.xacro (robot description, xacro)
@@ -6,5 +6,5 @@
       <parent link="Left_HipMount"/>
       <child link="Left_Hip"/>
-      <axis xyz="1.0 0 0"/>
+      <axis xyz="-1.0 0 0"/>
       <limit lower="${-pi/2}" upper="${pi/2}" effort="${maxeffort_val}" velocity="${maxVel_val}"/>
       <xacro:if value="$(arg use_URDF_joint_dynamics_coefficients)">

File: description/RobotElements/LeftLegElems/Lshank.xacro (robot description, xacro)
@@ -5,5 +5,5 @@
       <parent link="Left_Thigh"/>
       <child link="Left_Shank"/>
-      <axis xyz="0 1.0 0"/>
+      <axis xyz="0 -1.0 0"/>
       <limit lower="${-pi/2}" upper="${pi/2}" effort="${maxeffort_val}" velocity="${maxVel_val}"/>
       <xacro:if value="$(arg use_URDF_joint_dynamics_coefficients)">

File: description/RobotElements/LeftLegElems/Lthigh.xacro (robot description, xacro)
@@ -5,5 +5,5 @@
       <parent link="Left_Hip"/>
       <child link="Left_Thigh"/>
-      <axis xyz="0 1.0 0"/>
+      <axis xyz="0 -1.0 0"/>
       <limit lower="${-pi/2}" upper="${pi/2}" effort="${maxeffort_val}" velocity="${maxVel_val}"/>
       <xacro:if value="$(arg use_URDF_joint_dynamics_coefficients)">

File: description/RobotElements/RightArmElems/Rarm.xacro (robot description, xacro)
@@ -5,5 +5,5 @@
         <parent link="Right_ArmMounting"/>
         <child link="Right_Arm"/>
-        <axis xyz="1.0 0 0"/>
+        <axis xyz="-1.0 0 0"/>
         <limit lower="${-pi/2}" upper="${pi/2}" effort="${MX28maxeffort_val}" velocity="${MX28maxVel_val}"/>
         <xacro:if value="$(arg use_URDF_joint_dynamics_coefficients)">

File: description/RobotElements/RightArmElems/Rforearm.xacro (robot description, xacro)
@@ -5,5 +5,5 @@
         <parent link="Right_Arm"/>
         <child link="Right_Forearm"/>
-        <axis xyz="0 1.0 0"/>
+        <axis xyz="0 -1.0 0"/>
         <limit lower="${-pi/2}" upper="${pi/2}" effort="${MX28maxeffort_val}" velocity="${MX28maxVel_val}"/>
         <xacro:if value="$(arg use_URDF_joint_dynamics_coefficients)">

File: description/RobotElements/RightLegElems/Rankle.xacro (robot description, xacro)
@@ -5,5 +5,5 @@
         <parent link="Right_Shank"/>
         <child link="Right_Ankle"/>
-        <axis xyz="0 1.0 0"/>
+        <axis xyz="0 -1.0 0"/>
         <limit lower="${-pi/2}" upper="${pi/2}" effort="${maxeffort_val}" velocity="${maxVel_val}"/>
         <xacro:if value="$(arg use_URDF_joint_dynamics_coefficients)">

File: description/RobotElements/RightLegElems/Rfoot.xacro (robot description, xacro)
@@ -5,5 +5,5 @@
         <parent link="Right_Ankle"/>
         <child link="Right_Foot"/>
-        <axis xyz="1.0 0 0"/>
+        <axis xyz="-1.0 0 0"/>
         <limit lower="${-pi/2}" upper="${pi/2}" effort="${maxeffort_val}" velocity="${maxVel_val}"/>
         <xacro:if value="$(arg use_URDF_joint_dynamics_coefficients)">

File: description/RobotElements/RightLegElems/Rhip.xacro (robot description, xacro)
@@ -5,5 +5,5 @@
         <parent link="Right_HipMount"/>
         <child link="Right_Hip"/>
-        <axis xyz="1.0 0 0"/>
+        <axis xyz="-1.0 0 0"/>
         <limit lower="${-pi/2}" upper="${pi/2}" effort="${maxeffort_val}" velocity="${maxVel_val}"/>
         <xacro:if value="$(arg use_URDF_joint_dynamics_coefficients)">

File: description/RobotElements/RightLegElems/Rshank.xacro (robot description, xacro)
@@ -5,5 +5,5 @@
       <parent link="Right_Thigh"/>
       <child link="Right_Shank"/>
-      <axis xyz="0 1.0 0"/>
+      <axis xyz="0 -1.0 0"/>
         <limit lower="${-pi/2}" upper="${pi/2}" effort="${maxeffort_val}" velocity="${maxVel_val}"/>
         <xacro:if value="$(arg use_URDF_joint_dynamics_coefficients)">

File: description/RobotElements/RightLegElems/Rthigh.xacro (robot description, xacro)
@@ -5,5 +5,5 @@
       <parent link="Right_Hip"/>
       <child link="Right_Thigh"/>
-      <axis xyz="0 1.0 0"/>
+      <axis xyz="0 -1.0 0"/>
         <limit lower="${-pi/2}" upper="${pi/2}" effort="${maxeffort_val}" velocity="${maxVel_val}"/>
         <xacro:if value="$(arg use_URDF_joint_dynamics_coefficients)">
